File: schematics/board/SP1.brd (EAGLE design)
At the start: 30 x 46 mm, 12 parts

Commit message: ПЛАТЫ, АААААААААААААААААААААААААААА
Parts:
- removed D3, D4: MBR0520LT, diode:SOD123
- removed U$4: SOLAR-2_0, CanCubeSat:SOLAR_0-2
- added D5, D6, D7, D8: MBR0520LT, diode:SOD123
- added U$5, U$6, U$7, U$8: SOLAR-2_0, CanCubeSat:SOLAR_0-2
- U$3: value SOLAR-2_0 -> Плата СП1; device CanCubeSat:SOLAR_0-2 -> UNKNOWN-2024:LOGO
- moved U$3 110.4 mm to (-2.50, -75.0), turned to 0 degrees
Connections:
- removed net N$2: D2.C, D3.A, U$2.OUT, U$3.IN-2
- removed net N$3: D3.C, D4.A, U$3.OUT-2, U$3.OUT-21, U$4.IN-2
- new net N$6: D5.C, D6.A, U$5.OUT-2, U$5.OUT-21, U$6.IN-2
- new net N$8: D7.C, D8.A, U$7.OUT-2, U$7.OUT-21, U$8.IN-2
- net SP+: now also D5.A, D7.A, U$5.IN-2, U$7.IN-2
- net SP-: now also D2.C, D6.C, D8.C, U$2.OUT, U$6.OUT-2, U$6.OUT-21, U$8.OUT-2, U$8.OUT-21; no longer D4.C, U$4.OUT-2, U$4.OUT-21
Routing:
- net N$3: track 31.0 -> 0.00 mm, vias 1 -> 0
- net N$2: track 21.2 -> 0.00 mm, vias 1 -> 0
- net SP-: track 17.8 -> 25.5 mm, vias 0 -> 1
- net SP+: track 33.7 -> 31.9 mm
