File: schematics/board/SP2.brd (EAGLE design)
At the start: 30 x 46 mm, 15 parts

Commit message: ПЛАТЫ, АААААААААААААААААААААААААААА
Parts:
- removed D1, D2, D3, D4: MBR0520LT, diode:SOD123
- removed U$2: SOLAR-2_1, KNPN-2023:SOLAR_1-2
- removed U$3, U$4: SOLAR-2_0, KNPN-2023:SOLAR_0-2
- added D10, D5, D6, D7, D8, D9: MBR0520LT, diode:SOD123
- added U$10, U$11, U$8, U$9: SOLAR-2_0, CanCubeSat:SOLAR_0-2
- added U$5, U$6: SOLAR-2_1, CanCubeSat:SOLAR_1-2
- U$1: value SOLAR-2_1 -> Плата СП2; device KNPN-2023:SOLAR_1-2 -> UNKNOWN-2024:LOGO
- moved U$1 91.7 mm to (1.00, -59.0), turned to 0 degrees
Connections:
- removed net N$1: D1.C, D2.A, U$1.OUT, U$2.IN-2
- removed net N$2: D2.C, D3.A, U$2.OUT, U$3.IN-2
- removed net N$3: D3.C, D4.A, U$3.OUT-2, U$3.OUT-21, U$4.IN-2
- new net N$5: D5.C, D6.A, U$5.OUT, U$6.IN-2
- new net N$7: D7.C, D8.A, U$8.OUT-2, U$8.OUT-21, U$9.IN-2
- new net N$8: D10.A, D9.C, U$10.OUT-2, U$10.OUT-21, U$11.IN-2
- net SP+: now also D5.A, D7.A, D9.A, U$10.IN-2, U$5.IN-2, U$8.IN-2; no longer D1.A, U$1.IN-2
- net SP+-: now also D10.C, D6.C, D8.C, U$11.OUT-2, U$11.OUT-21, U$6.OUT, U$9.OUT-2, U$9.OUT-21; no longer D4.C, U$4.OUT-2, U$4.OUT-21
Routing:
- net N$1: track 40.7 -> 0.00 mm, vias 2 -> 0
- net N$3: track 39.9 -> 0.00 mm, vias 2 -> 0
- net SP+-: track 57.0 -> 34.0 mm
- net N$2: track 15.0 -> 0.00 mm, vias 1 -> 0
