File: schematics/board/GERMO.brd (EAGLE design)
At the start: 100 x 80 mm, 8 parts

Commit message: схемы плат
Parts:
- added R11, R12, R13, R8: 10k, rcl:R0603
- added R39, R41, R43, R45: 100k, rcl:R0603
- added R40, R42, R44, R46: 1M, rcl:R0603
- added U$10, U$11, U$12, U$5, U$6, U$7, U$8, U$9: CONNECT_3, UNKNOWN-2024:CONNECT_3
Connections:
- new net 3V3: R40.1, R42.1, R44.1, R46.1, U$10.1, U$11.1, U$12.1, U$5.1, U$6.1, U$7.1, U$8.1, U$9.1
- new net N$1: R39.2, U$5.3
- new net N$10: R12.1, U$9.2
- new net N$11: R44.2, U$10.3
- new net N$12: R43.1, U$10.2
- new net N$13: R45.2, U$11.3
- new net N$14: R13.1, U$11.2
- new net N$15: R46.2, U$12.3
- new net N$16: R45.1, U$12.2
- new net N$2: R8.1, U$5.2
- new net N$3: R40.2, U$6.3
- new net N$4: R39.1, U$6.2
- new net N$5: R41.2, U$7.3
- new net N$6: R11.1, U$7.2
- new net N$7: R42.2, U$8.3
- new net N$8: R41.1, U$8.2
- new net N$9: R43.2, U$9.3
- net CO: now also R8.2
- net MICS: now also R13.2
- net NH3: now also R12.2
- net NO2: now also R11.2

Commit message: подготовлены файлы для зимней сессии
Parts:
- renumbered U$1 to MICS-6814, U$3 to MICS-5524
Changed lines of the file:
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@@
 <attribute name="VALUE" x="-34.29" y="38.735" size="1.27" layer="27"/>
 </element>
-<element name="U$1" library="CanCubeSat" package="MICS-6814" value="MICS-6814" x="-34.29" y="8.89" smashed="yes">
+<element name="MICS-6814" library="CanCubeSat" package="MICS-6814" value="MICS-6814" x="-34.29" y="8.89" smashed="yes">
 <attribute name="NAME" x="-39.37" y="17.78" size="1.27" layer="25"/>
 </element>
@@
 <attribute name="VALUE" x="-24.9" y="46.76" size="1" layer="21" font="vector" ratio="15"/>
 </element>
-<element name="U$3" library="UNKNOWN-2024" package="MICS-5524" value="MICS_5524" x="-3.81" y="-4.42" smashed="yes">
+<element name="MICS-5524" library="UNKNOWN-2024" package="MICS-5524" value="MICS_5524" x="-3.81" y="-4.42" smashed="yes">
 <attribute name="NAME" x="-7.39" y="6.47" size="1.27" layer="25"/>
 </element>
@@
 <contactref element="JP2" pad="5"/>
 <contactref element="BME280" pad="P$3"/>
-<contactref element="U$1" pad="P$2"/>
-<contactref element="U$3" pad="P$3"/>
+<contactref element="MICS-6814" pad="P$2"/>
+<contactref element="MICS-5524" pad="P$3"/>
 <contactref element="R17" pad="2"/>
 <contactref element="U$4" pad="P$2"/>
@@
 <contactref element="JP2" pad="6"/>
 <contactref element="BME280" pad="P$4"/>
-<contactref element="U$1" pad="P$1"/>
-<contactref element="U$3" pad="P$4"/>
+<contactref element="MICS-6814" pad="P$1"/>
+<contactref element="MICS-5524" pad="P$4"/>
 <contactref element="U$4" pad="P$1"/>
 <wire x1="-39.37" y1="16.07" x2="-43.3" y2="-16.51" width="0" layer="19" extent="1-1"/>
@@
 <signal name="NO2">
 <contactref element="JP2" pad="2"/>
-<contactref element="U$1" pad="P$3"/>
+<contactref element="MICS-6814" pad="P$3"/>
 <contactref element="R11" pad="2"/>
 <wire x1="-34.29" y1="16.07" x2="-53.76" y2="-26.67" width="0" layer="19" extent="1-1"/>
@@
 <signal name="NH3">
 <contactref element="JP2" pad="3"/>
-<contactref element="U$1" pad="P$4"/>
+<contactref element="MICS-6814" pad="P$4"/>
 <contactref element="R12" pad="2"/>
 <wire x1="-31.75" y1="16.07" x2="-48.68" y2="-26.67" width="0" layer="19" extent="1-1"/>
@@
 <signal name="MICS">
 <contactref element="JP2" pad="4"/>
-<contactref element="U$3" pad="P$2"/>
+<contactref element="MICS-5524" pad="P$2"/>
 <contactref element="R13" pad="2"/>
 <wire x1="-5.08" y1="3.86" x2="-43.6" y2="-26.67" width="0" layer="19" extent="1-1"/>
@@
 </signal>
 <signal name="CO">
-<contactref element="U$1" pad="P$5"/>
+<contactref element="MICS-6814" pad="P$5"/>
 <contactref element="JP2" pad="1"/>
 <contactref element="R8" pad="2"/>
@@
 </signal>
 <signal name="EN">
-<contactref element="U$3" pad="P$1"/>
+<contactref element="MICS-5524" pad="P$1"/>
 <contactref element="R17" pad="1"/>
 <wire x1="-7.62" y1="3.86" x2="-40.22" y2="-16.51" width="0" layer="19" extent="1-1"/>
