File: schematics/board/GERMO.brd (EAGLE design)
At the start: 72.1 x 32 mm, 35 parts

Commit message: фцыувкаепнргошщз
Other:
- board text added: "5V"
- board text added: "FOTO0"
- board text added: "FOTO1"
- board text added: "GND"
- board text added: "SCL"
- board text added: "SDA"

Commit message: проверка плат
Changed lines of the file:
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@@
 <?xml version="1.0" encoding="utf-8"?>
 <!DOCTYPE eagle SYSTEM "eagle.dtd">
-<eagle version="9.6.2">
+<eagle version="9.4.2">
 <drawing>
 <settings>
-<setting alwaysvectorfont="no"/>
+<setting alwaysvectorfont="yes"/>
 <setting verticaltext="up"/>
 </settings>
@@
 <attribute name="VALUE" x="56.435" y="9.905" size="1.27" layer="27" font="vector" ratio="15" rot="R180"/>
 </element>
-<element name="JP2" library="pinhead" library_urn="urn:adsk.eagle:library:325" package="1X02" package3d_urn="urn:adsk.eagle:package:22435/2" value="" x="47.46" y="9.5" smashed="yes" rot="R180">
-<attribute name="POPULARITY" value="98" x="47.46" y="9.5" size="1.778" layer="27" rot="R180" display="off"/>
-<attribute name="VALUE" x="50" y="12.675" size="1.27" layer="27" rot="R180"/>
+<element name="JP2" library="pinhead" library_urn="urn:adsk.eagle:library:325" package="1X02" package3d_urn="urn:adsk.eagle:package:22435/2" value="" x="47.5" y="9.5" smashed="yes" rot="R180">
+<attribute name="POPULARITY" value="98" x="47.5" y="9.5" size="1.778" layer="27" rot="R180" display="off"/>
+<attribute name="VALUE" x="50.04" y="12.675" size="1.27" layer="27" rot="R180"/>
 </element>
 </elements>
@@
 <wire x1="55.9" y1="14.675" x2="54.6821125" y2="14.675" width="0.3" layer="1"/>
 <wire x1="54.6821125" y1="14.675" x2="51.5071125" y2="11.5" width="0.3" layer="1"/>
-<wire x1="48.73" y1="11.03" x2="48.73" y2="9.5" width="0.3" layer="1"/>
+<wire x1="48.73" y1="11.03" x2="48.77" y2="9.5" width="0.3" layer="1"/>
 <wire x1="51.5071125" y1="11.5" x2="49.2" y2="11.5" width="0.3" layer="1"/>
 <wire x1="49.2" y1="11.5" x2="48.73" y2="11.03" width="0.3" layer="1"/>
@@
 <contactref element="JP2" pad="2"/>
 <wire x1="55.9" y1="15.325" x2="54.625" y2="15.325" width="0.3" layer="1"/>
-<wire x1="46.19" y1="11.09" x2="46.19" y2="9.5" width="0.3" layer="1"/>
+<wire x1="46.19" y1="11.09" x2="46.23" y2="9.5" width="0.3" layer="1"/>
 <wire x1="54.625" y1="15.325" x2="51.3" y2="12" width="0.3" layer="1"/>
 <wire x1="51.3" y1="12" x2="47.1" y2="12" width="0.3" layer="1"/>

Commit message: Платы готовы
Parts:
- U$2: value Плата ГЕРМО -> Плата Гермообъема
- renumbered U$4 to CCS811
Other:
- board text added: "FOT0"
- board text added: "FOT1"
- board text removed: "FOTO0"
- board text removed: "FOTO1"
Changed lines of the file:
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@@
 <circle x="18.627309375" y="14.52901875" radius="1.1" width="0.001" layer="20"/>
 <circle x="61.372690625" y="14.52901875" radius="1.1" width="0.001" layer="20"/>
-<text x="45" y="7.3" size="1" layer="25" font="vector" ratio="15" rot="R90">FOTO0</text>
-<text x="51.3" y="7.2" size="1" layer="25" font="vector" ratio="15" rot="R90">FOTO1</text>
+<text x="46.7" y="11.2" size="1" layer="25" font="vector" ratio="15" rot="R90">FOT0</text>
+<text x="49.2" y="11.2" size="1" layer="25" font="vector" ratio="15" rot="R90">FOT1</text>
 <text x="34.3" y="11.2" size="1" layer="25" font="vector" ratio="15" rot="R90">SCL</text>
 <text x="31.8" y="11.2" size="1" layer="25" font="vector" ratio="15" rot="R90">SDA</text>
@@
 <element name="U$11" library="UNKNOWN-2024" package="CONNECT_3" value="CONNECT_3" x="37.17" y="22.69" smashed="yes"/>
 <element name="U$12" library="UNKNOWN-2024" package="CONNECT_3" value="CONNECT_3" x="38.19" y="26.15" smashed="yes" rot="R270"/>
-<element name="U$2" library="UNKNOWN-2024" package="LOGO" value="Плата ГЕРМО" x="14.8" y="28.53" smashed="yes">
+<element name="U$2" library="UNKNOWN-2024" package="LOGO" value="Плата Гермообъема" x="14.8" y="28.53" smashed="yes">
 <attribute name="VALUE" x="15.3" y="27.03" size="1" layer="21" font="vector" ratio="15"/>
 </element>
-<element name="U$4" library="UNKNOWN-2024" package="CSS811" value="CCS811" x="21" y="27.82" smashed="yes" rot="MR270"/>
+<element name="CCS811" library="UNKNOWN-2024" package="CSS811" value="CCS811" x="21" y="27.82" smashed="yes" rot="MR270">
+<attribute name="NAME" x="11.8" y="19.91" size="1" layer="26" ratio="15" rot="MR180"/>
+</element>
 <element name="U$5" library="UNKNOWN-2024" package="CONNECT_3" value="CONNECT_3" x="62.09" y="27.41" smashed="yes"/>
 <element name="U$6" library="UNKNOWN-2024" package="CONNECT_3" value="CONNECT_3" x="63.11" y="30.83" smashed="yes" rot="R270"/>
@@
 <attribute name="POPULARITY" value="73" x="46.9" y="16.2" size="1.778" layer="27" display="off"/>
 <attribute name="SPICEPREFIX" value="C" x="46.9" y="16.2" size="1.778" layer="27" display="off"/>
-<attribute name="VALUE" x="60.265" y="17.395" size="1.27" layer="27" font="vector" ratio="15"/>
+<attribute name="VALUE" x="60.265" y="17.395" size="1" layer="27" font="vector" ratio="15"/>
 </element>
 <element name="C3" library="rcl" library_urn="urn:adsk.eagle:library:334" package="C0603" package3d_urn="urn:adsk.eagle:package:23616/2" value="100nF" x="58.4" y="14.1" smashed="yes">
 <attribute name="POPULARITY" value="73" x="52.9" y="17.6" size="1.778" layer="27" display="off"/>
 <attribute name="SPICEPREFIX" value="C" x="52.9" y="17.6" size="1.778" layer="27" display="off"/>
-<attribute name="VALUE" x="60.265" y="15.795" size="1.27" layer="27" font="vector" ratio="15"/>
+<attribute name="VALUE" x="60.265" y="15.795" size="1" layer="27" font="vector" ratio="15"/>
 </element>
 <element name="C4" library="rcl" library_urn="urn:adsk.eagle:library:334" package="C0603" package3d_urn="urn:adsk.eagle:package:23616/2" value="100nF" x="47.8" y="17.1" smashed="yes" rot="R180">
 <attribute name="POPULARITY" value="73" x="59.8" y="18.6" size="1.778" layer="27" rot="R180" display="off"/>
 <attribute name="SPICEPREFIX" value="C" x="59.8" y="18.6" size="1.778" layer="27" rot="R180" display="off"/>
-<attribute name="VALUE" x="49.335" y="16.005" size="1.27" layer="27" font="vector" ratio="15" rot="R180"/>
+<attribute name="VALUE" x="49.335" y="16.005" size="1" layer="27" font="vector" ratio="15" rot="R180"/>
 </element>
 <element name="R16" library="rcl" library_urn="urn:adsk.eagle:library:334" package="R0603" package3d_urn="urn:adsk.eagle:package:23555/3" value="5k1" x="58.4" y="11.9" smashed="yes">
 <attribute name="POPULARITY" value="77" x="52.9" y="10.4" size="1.778" layer="27" display="off"/>
 <attribute name="SPICEPREFIX" value="R" x="52.9" y="10.4" size="1.778" layer="27" display="off"/>
-<attribute name="VALUE" x="59.965" y="11.995" size="1.27" layer="27" font="vector" ratio="15"/>
+<attribute name="VALUE" x="60.165" y="11.995" size="1" layer="27" font="vector" ratio="15"/>
 </element>
 <element name="R2" library="rcl" library_urn="urn:adsk.eagle:library:334" package="R0603" package3d_urn="urn:adsk.eagle:package:23555/3" value="5k1" x="55" y="11.2" smashed="yes" rot="R180">
 <attribute name="POPULARITY" value="77" x="65" y="17.7" size="1.778" layer="27" rot="R180" display="off"/>
 <attribute name="SPICEPREFIX" value="R" x="65" y="17.7" size="1.778" layer="27" rot="R180" display="off"/>
-<attribute name="VALUE" x="56.435" y="9.905" size="1.27" layer="27" font="vector" ratio="15" rot="R180"/>
+<attribute name="VALUE" x="56.335" y="10.105" size="1" layer="27" font="vector" ratio="15" rot="R180"/>
 </element>
 <element name="JP2" library="pinhead" library_urn="urn:adsk.eagle:library:325" package="1X02" package3d_urn="urn:adsk.eagle:package:22435/2" value="" x="47.5" y="9.5" smashed="yes" rot="R180">
@@
 <contactref element="MICS-5524" pad="P$3"/>
 <contactref element="R17" pad="2"/>
-<contactref element="U$4" pad="P$2"/>
+<contactref element="CCS811" pad="P$2"/>
 <contactref element="R1" pad="2"/>
 <contactref element="JP1" pad="1"/>
@@
 <contactref element="MICS-6814" pad="P$1"/>
 <contactref element="MICS-5524" pad="P$4"/>
-<contactref element="U$4" pad="P$1"/>
+<contactref element="CCS811" pad="P$1"/>
 <contactref element="JP1" pad="2"/>
 <wire x1="29.89" y1="21.59" x2="29.89" y2="15.2" width="0.5" layer="16"/>
@@
 <signal name="SDA">
 <contactref element="BME280" pad="P$1"/>
-<contactref element="U$4" pad="P$4"/>
+<contactref element="CCS811" pad="P$4"/>
 <contactref element="JP1" pad="3"/>
 <contactref element="U$14" pad="P$15"/>
@@
 <signal name="SCL">
 <contactref element="BME280" pad="P$2"/>
-<contactref element="U$4" pad="P$3"/>
+<contactref element="CCS811" pad="P$3"/>
 <contactref element="JP1" pad="4"/>
 <contactref element="U$14" pad="P$16"/>
@@
 </signal>
 <signal name="WAC">
-<contactref element="U$4" pad="P$5"/>
+<contactref element="CCS811" pad="P$5"/>
 <contactref element="R1" pad="1"/>
 <wire x1="19.73" y1="21.59" x2="19.73" y2="24" width="0.3" layer="1"/>
