File: schematics/board/SP1.sch (EAGLE design)
At the start: 12 parts

Commit message: ПЛАТЫ, АААААААААААААААААААААААААААА
Parts:
- removed D3, D4: MBR0520LT, diode:MBR0520LT
- removed U$4: SOLAR-2_0, CanCubeSat:SOLAR-2_0
- added D5, D6, D7, D8: MBR0520LT, diode:MBR0520LT
- added U$5, U$6, U$7, U$8: SOLAR-2_0, CanCubeSat:SOLAR-2_0
- U$3: value SOLAR-2_0 -> Плата СП1; device CanCubeSat:SOLAR-2_0 -> UNKNOWN-2024:LOGOPCB-""
Connections:
- removed net N$2: D2.C, D3.A, U$2.OUT, U$3.IN
- removed net N$3: D3.C, D4.A, U$3.OUT, U$4.IN
- new net N$6: D5.C, D6.A, U$5.OUT, U$6.IN
- new net N$8: D7.C, D8.A, U$7.OUT, U$8.IN
- net SP+: now also D5.A, D7.A, U$5.IN, U$7.IN
- net SP-: now also D2.C, D6.C, D8.C, U$2.OUT, U$6.OUT, U$8.OUT; no longer D4.C, U$4.OUT
Other:
- moved on the sheet: C1, JP1, LED1, R1

Commit message: подготовлены файлы для зимней сессии
Changed lines of the file:
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@@
 <attribute name="VALUE" x="33.02" y="78.9686" size="1.778" layer="96"/>
 </instance>
-<instance part="U$3" gate="G$1" x="-76.2" y="111.76" smashed="yes">
-<attribute name="VALUE" x="27.94" y="111.76" size="12.7" layer="96"/>
+<instance part="U$3" gate="G$1" x="-63.5" y="111.76" smashed="yes">
+<attribute name="VALUE" x="40.64" y="111.76" size="12.7" layer="96"/>
 </instance>
 </instances>
