File: schematics/board/MK.brd (EAGLE design)
At the start: 68.9 x 68.9 mm, 19 parts

Commit message: ifdhv
Parts:
- added C2, C3, C4, C5: 100nF, rcl:C0603
- added R0, R11, R12, R13, R14, R15, R16, R17, R18, R19, R22, R23, R24, R25, R7, R8: 5k1, rcl:R0603
- added R20: (no value), rcl:R2512
- added R21: (no value), rcl:0207/15
- added U$0, U$10, U$11, U$12, U$5, U$7, U$8, U$9: VT93N1, KNPN-2023:VT93N1
- added U$13, U$15: 74HC595, CanCubeSat:TSSOP16
- added U$14: AD5593, UNKNOWN-2024:AD5593
- added U$16: INA219AID, CanCubeSat:SOT23-8
- added U$17: IRF7905PBF, UNKNOWN-2024:SO8
- added U$18, U$19, U$20: MOLEX-2-1.25, UNKNOWN-2024:53047-02
- added U$3: BOARD_SHAPE, UNKNOWN-2024:BOARD_SHAPE
- added X1, X2: JST-2-2.5, UNKNOWN-2024:JST-2-2.5
Connections:
- new net BUS+: X1.1, X2.1
- new net FOTO0: U$20.2
- new net INA_SP+: R19.1, R20.1, R21.1
- new net LATCH: U$13.12, U$15.12
- new net MOSI: U$13.14
- new net MOTOR1+: U$13.4, U$18.1
- new net MOTOR1-: U$13.5, U$18.2
- new net MOTOR2+: U$13.2, U$19.1
- new net MOTOR2-: U$13.3, U$19.2
- new net N$10: R14.2, U$11.P$1, U$14.P$12
- new net N$11: C2.1, U$14.P$8
- new net N$12: R15.2, U$12.P$1, U$14.P$13
- new net N$15: C5.2, R19.2, U$16.7
- new net N$16: C3.1, C4.1, U$14.P$3, U$14.P$9
- new net N$17: R16.1, U$14.P$2
- new net N$18: C5.1, R18.2, U$16.8
- new net N$19: R17.1, U$14.P$1
- new net N$20: U$17.7, U$17.8, X1.2
- new net N$21: U$17.5, U$17.6, X2.2
- new net N$22: R22.1, R23.2, U$17.2
- new net N$23: R24.1, R25.2, U$17.4
- new net N$35: U$13.9, U$15.14
- new net N$4: R0.2, U$0.P$1, U$14.P$4
- new net N$5: R8.2, U$14.P$6, U$7.P$1
- new net N$6: R7.2, U$14.P$5, U$5.P$1
- new net N$7: R11.2, U$14.P$7, U$8.P$1
- new net N$8: R12.2, U$14.P$10, U$9.P$1
- new net N$9: R13.2, U$10.P$1, U$14.P$11
- new net PERE1: R23.1, U$13.6
- new net PERE2: R25.1, U$13.7
- new net SCK: U$13.11, U$15.11
- new net SHIFT3: U$15.9
- new net SP+: R18.1, R20.2
- new net SP-: R21.2
- net 3V3: now also R0.1, R11.1, R12.1, R13.1, R14.1, R15.1, R17.2, R7.1, R8.1, U$13.10, U$13.16, U$15.10, U$15.16, U$16.5
- net BUZZER: now also U$13.1
- net GND: now also C2.2, C3.2, C4.2, R16.2, R22.2, R24.2, U$0.P$2, U$10.P$2, U$11.P$2, U$12.P$2, U$13.13, U$13.8, U$14.P$14, U$15.13, U$15.8, U$16.1, U$16.2, U$16.6, U$17.1, U$17.3, U$20.1, U$5.P$2, U$7.P$2, U$8.P$2, U$9.P$2
- net SCL: now also U$14.P$16, U$16.4
- net SDA: now also U$14.P$15, U$16.3
Other:
- board size 68.9 x 68.9 mm -> 76 x 76 mm

Commit message: пам пам тидам
Parts:
- added R26, R27, R28, R29, R30, R31, R32, R33, R34, R35, R36, R37: 5k1, rcl:R0603
- added U$21: MOSFET_2P+2N_AP9930GM, UNKNOWN-2024:SO8
- added U$22, U$23: NDC7002N, UNKNOWN-2024:SOT23-6
- U$15: value 74HC595 -> MOSFET_2P+2N_AP9930GM; device CanCubeSat:TSSOP16 -> UNKNOWN-2024:SO8
- moved U$14 285.3 mm to (-2.27, -278.6)
- moved C5 236.9 mm to (92.6, 23.1), flipped to the bottom
- moved R20 236.1 mm to (92.7, 17.9), flipped to the bottom, turned to 180 degrees
- moved R21 235.3 mm to (86.1, 20.8), flipped to the bottom, turned to 90 degrees
- moved R18 231.2 mm to (95.6, 22.2), flipped to the bottom, turned to 90 degrees
- moved R19 230.8 mm to (89.8, 22.3), flipped to the bottom, turned to 90 degrees
- moved U$16 229.5 mm to (92.4, 27.5), flipped to the bottom, turned to 270 degrees
- moved R8 146.7 mm to (35.2, 73.9)
- moved R0 146.0 mm to (73.8, 35.7)
- moved U$7 145.7 mm to (40.0, 75.5)
- moved U$9 141.5 mm to (14.6, 65.1), turned to 45 degrees
- moved R11 122.0 mm to (45.0, 5.40)
- moved U$8 113.0 mm to (40.0, 4.50), turned to 180 degrees
- moved U$0 92.5 mm to (75.5, 40.0), turned to 270 degrees
- moved R7 89.3 mm to (4.10, 36.0)
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Connections:
- removed net SHIFT3: U$15.9
- new net MK_MOTOR1+: R37.1
- new net MK_MOTOR1-: R36.1
- new net MK_MOTOR2+: R31.1
- new net MK_MOTOR2-: R30.1
- new net N$24: R32.2, R34.1, U$21.1, U$21.8, U$23.6
- new net N$25: R26.2, R28.1, U$15.1, U$15.8, U$22.6
- new net N$26: R27.2, R29.1, U$15.4, U$15.5, U$22.4
- new net N$27: R33.2, R35.1, U$21.4, U$21.5, U$23.4
- new net N$28: R34.2, R36.2, U$23.1
- new net N$29: R35.2, R37.2, U$23.3
- new net N$32: R28.2, R30.2, U$22.1
- new net SHIFT2: U$13.9
- net 3V3: no longer U$15.10, U$15.16
- net 5V: now also R26.1, R27.1, R32.1, R33.1, U$15.7, U$21.7
- net GND: now also U$15.3, U$21.3, U$22.2, U$22.5, U$23.2, U$23.5; no longer U$15.13, U$15.8
- net LATCH: no longer U$15.12
- net MOTOR1+: now also U$21.6
- net MOTOR1-: now also U$21.2
- net MOTOR2+: now also U$15.6
- net MOTOR2-: now also U$15.2
- net N$35: now also R29.2, R31.2, U$22.3; no longer U$13.9, U$15.14
- net SCK: no longer U$15.11
Routing:
- net GND: track 171.4 -> 235.2 mm, vias 5 -> 8
- net SP+: track 0.00 -> 19.4 mm
- net SP-: track 0.00 -> 17.6 mm
- net INA_SP+: track 0.00 -> 10.1 mm
- net N$15: track 0.00 -> 8.27 mm
- net 3V3: track 153.2 -> 160.3 mm
- net N$18: track 0.00 -> 6.11 mm
- net MISO_RADIO: track 99.9 -> 104.8 mm
- net SCK_RADIO: track 79.1 -> 84.0 mm
- net SCL: track 47.9 -> 52.0 mm
- net SD_CK: track 52.6 -> 56.7 mm
- net SDA: track 54.3 -> 58.3 mm

Commit message: iyrd
Parts:
- moved U$10 183.9 mm to (65.2, 65.2), turned to 315 degrees
- moved U$12 167.4 mm to (65.2, 14.8), turned to 225 degrees
- moved U$11 122.2 mm to (14.8, 14.8), turned to 135 degrees
- moved U$9 0.21 mm to (14.8, 65.2)
Changed lines of the file:
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@@
 <attribute name="VALUE" x="44.365" y="3.495" size="1.27" layer="27"/>
 </element>
-<element name="U$9" library="KNPN-2023" package="VT93N1" value="VT93N1" x="14.6" y="65.1" smashed="yes" rot="R45">
-<attribute name="NAME" x="10.35735625" y="65.1" size="1.27" layer="25" rot="R45"/>
+<element name="U$9" library="KNPN-2023" package="VT93N1" value="VT93N1" x="14.772" y="65.228" smashed="yes" rot="R45">
+<attribute name="NAME" x="10.52935625" y="65.228" size="1.27" layer="25" rot="R45"/>
 </element>
 <element name="R12" library="rcl" library_urn="urn:adsk.eagle:library:334" package="R0603" package3d_urn="urn:adsk.eagle:package:23555/3" value="5k1" x="-66" y="-58.3" smashed="yes">
@@
 <attribute name="VALUE" x="-66.635" y="-60.205" size="1.27" layer="27"/>
 </element>
-<element name="U$10" library="KNPN-2023" package="VT93N1" value="VT93N1" x="-64" y="-65.6" smashed="yes">
-<attribute name="NAME" x="-67" y="-62.6" size="1.27" layer="25"/>
+<element name="U$10" library="KNPN-2023" package="VT93N1" value="VT93N1" x="65.228" y="65.228" smashed="yes" rot="R315">
+<attribute name="NAME" x="65.228" y="69.470640625" size="1.27" layer="25" rot="R315"/>
 </element>
 <element name="R13" library="rcl" library_urn="urn:adsk.eagle:library:334" package="R0603" package3d_urn="urn:adsk.eagle:package:23555/3" value="5k1" x="-66" y="-71.3" smashed="yes">
@@
 <attribute name="VALUE" x="-66.635" y="-73.205" size="1.27" layer="27"/>
 </element>
-<element name="U$11" library="KNPN-2023" package="VT93N1" value="VT93N1" x="-64" y="-78.6" smashed="yes">
-<attribute name="NAME" x="-67" y="-75.6" size="1.27" layer="25"/>
+<element name="U$11" library="KNPN-2023" package="VT93N1" value="VT93N1" x="14.772" y="14.772" smashed="yes" rot="R135">
+<attribute name="NAME" x="14.772" y="10.52935625" size="1.27" layer="25" rot="R135"/>
 </element>
 <element name="R14" library="rcl" library_urn="urn:adsk.eagle:library:334" package="R0603" package3d_urn="urn:adsk.eagle:package:23555/3" value="5k1" x="-66" y="-84.3" smashed="yes">
@@
 <attribute name="VALUE" x="-66.635" y="-86.205" size="1.27" layer="27"/>
 </element>
-<element name="U$12" library="KNPN-2023" package="VT93N1" value="VT93N1" x="-64" y="-91.6" smashed="yes">
-<attribute name="NAME" x="-67" y="-88.6" size="1.27" layer="25"/>
+<element name="U$12" library="KNPN-2023" package="VT93N1" value="VT93N1" x="65.228" y="14.772" smashed="yes" rot="R225">
+<attribute name="NAME" x="69.47064375" y="14.772" size="1.27" layer="25" rot="R225"/>
 </element>
 <element name="R15" library="rcl" library_urn="urn:adsk.eagle:library:334" package="R0603" package3d_urn="urn:adsk.eagle:package:23555/3" value="5k1" x="-66" y="-97.3" smashed="yes">
@@
 <wire x1="-65.15" y1="-107.1" x2="-65.15" y2="-112" width="0" layer="19" extent="1-1"/>
 <wire x1="-65.15" y1="-102.2" x2="-65.15" y2="-107.1" width="0" layer="19" extent="1-1"/>
-<wire x1="-62.75" y1="-93.4" x2="-65.15" y2="-102.2" width="0" layer="19" extent="1-1"/>
-<wire x1="-62.75" y1="-80.4" x2="-62.75" y2="-93.4" width="0" layer="19" extent="1-1"/>
-<wire x1="-62.75" y1="-67.4" x2="-62.75" y2="-80.4" width="0" layer="19" extent="1-1"/>
 <wire x1="-3.25" y1="-275.7" x2="-89.9" y2="-250.6" width="0" layer="19" extent="1-1"/>
-<wire x1="23.6" y1="21.8" x2="-62.75" y2="-67.4" width="0" layer="19" extent="1-1"/>
+<wire x1="15.16090625" y1="16.928675" x2="-65.15" y2="-102.2" width="0" layer="19" extent="1-1"/>
+<wire x1="23.6" y1="21.8" x2="15.16090625" y2="16.928675" width="0" layer="19" extent="1-1"/>
+<wire x1="63.071321875" y1="15.16090625" x2="57.99895625" y2="11.501040625" width="0" layer="19" extent="1-1"/>
+<wire x1="64.839090625" y1="63.071321875" x2="67.35" y2="55.7" width="0" layer="19" extent="1-16"/>
 <wire x1="41.25" y1="73.7" x2="34.879" y2="67.021" width="0" layer="19" extent="1-1"/>
 <wire x1="6.3" y1="41.25" x2="15.6" y2="37.5" width="0" layer="19" extent="1-1"/>
 <wire x1="38.75" y1="6.3" x2="41.9" y2="20.01" width="0" layer="19" extent="1-1"/>
-<wire x1="16.756675" y1="64.711090625" x2="29.87" y2="58.73" width="0" layer="19" extent="1-1"/>
+<wire x1="16.928675" y1="64.839090625" x2="29.87" y2="58.73" width="0" layer="19" extent="1-1"/>
 <wire x1="87.771753125" y1="15.328246875" x2="70.56966875" y2="16.06966875" width="0" layer="19" extent="1-16"/>
 <wire x1="73.7" y1="38.75" x2="67.35" y2="55.7" width="0" layer="19" extent="1-16"/>
@@
 <contactref element="R12" pad="2"/>
 <contactref element="U$14" pad="P$10"/>
-<wire x1="14.98890625" y1="62.943321875" x2="-65.15" y2="-58.3" width="0" layer="19" extent="1-1"/>
+<wire x1="15.16090625" y1="63.071321875" x2="-65.15" y2="-58.3" width="0" layer="19" extent="1-1"/>
 <wire x1="-0.65" y1="-275.7" x2="-65.15" y2="-58.3" width="0" layer="19" extent="1-1"/>
 </signal>
@@
 <contactref element="U$10" pad="P$1"/>
 <contactref element="R13" pad="2"/>
-<wire x1="-65.25" y1="-67.4" x2="-65.15" y2="-71.3" width="0" layer="19" extent="1-1"/>
+<wire x1="63.071321875" y1="64.839090625" x2="-65.15" y2="-71.3" width="0" layer="19" extent="1-1"/>
 <wire x1="-1.3" y1="-275.7" x2="-65.15" y2="-71.3" width="0" layer="19" extent="1-1"/>
 </signal>
@@
 <contactref element="U$11" pad="P$1"/>
 <contactref element="U$14" pad="P$12"/>
-<wire x1="-65.25" y1="-80.4" x2="-65.15" y2="-84.3" width="0" layer="19" extent="1-1"/>
+<wire x1="16.928675" y1="15.16090625" x2="-65.15" y2="-84.3" width="0" layer="19" extent="1-1"/>
 <wire x1="-1.95" y1="-275.7" x2="-65.15" y2="-84.3" width="0" layer="19" extent="1-1"/>
 </signal>
@@
 <contactref element="U$12" pad="P$1"/>
 <contactref element="U$14" pad="P$13"/>
-<wire x1="-65.25" y1="-93.4" x2="-65.15" y2="-97.3" width="0" layer="19" extent="1-1"/>
+<wire x1="64.839090625" y1="16.928675" x2="-65.15" y2="-97.3" width="0" layer="19" extent="1-1"/>
 <wire x1="-2.6" y1="-275.7" x2="-65.15" y2="-97.3" width="0" layer="19" extent="1-1"/>
 </signal>

Commit message: Платки там
Parts:
- removed R15: 5k1, rcl:R0603
- removed U$10, U$11, U$12, U$5, U$7, U$8, U$9: VT93N1, KNPN-2023:VT93N1
- added JP1: (no value), pinhead:1X10
- added JP2: (no value), pinhead:1X16
- added R39, R40, R41, R42, R43, R44, R45, R46: 5k1, rcl:R0603
- R20: value (none) -> R05
- moved R21 358.9 mm to (-92.8, -290.3), flipped to the top, turned to 0 degrees
- moved R14 203.1 mm to (-99.7, -284.6)
Connections:
- net SD_CK renamed CK_SD
- removed net N$10: R14.2, U$11.P$1, U$14.P$12
- removed net N$12: R15.2, U$12.P$1, U$14.P$13
- removed net N$5: R8.2, U$14.P$6, U$7.P$1
- new net CO: R8.2, U$14.P$6
- new net CS_LIS: STM.27
- new net CS_LSM: STM.26
- new net H3: R12.2, U$14.P$10
- new net M0_RADIO: STM.15
- new net M1_RADIO: STM.17
- new net MICS: R13.2, U$14.P$11
- new net MISO_SENS: STM.32
- new net MOSI_SENS: STM.33
- new net N$34: R13.1, R45.2
- new net N$36: R12.1, R43.2
- new net N$37: R11.1, R41.2
- new net NO2: R11.2, U$14.P$7
- new net RX_GPS: STM.9
- new net RX_LIDAR: STM.29
- new net RX_RADIO: STM.31
- new net SCK_SENS: STM.11
- new net TX_GPS: STM.8
- new net TX_LIDAR: STM.28
- new net TX_RADIO: STM.30
- net 3V3: now also R40.1, R42.1, R44.1, R46.1; no longer R11.1, R12.1, R13.1, R14.1, R15.1, R8.1
- net 5V: now also R39.2, R8.1
- net ADC_FOTO: no longer STM.6
- net CE_RADIO: no longer STM.2
- net CS_RADIO: no longer STM.3
- net DIR_DRIVER: no longer STM.27
- net FOTO0: now also R7.2, U$14.P$5
- net GND: now also R14.1; no longer U$10.P$2, U$11.P$2, U$12.P$2, U$13.13, U$5.P$2, U$7.P$2, U$8.P$2, U$9.P$2
- net IRQ_RADIO: no longer STM.4
- net MISO_RADIO: no longer STM.28
- net MISO_SR: no longer STM.32
- net MOSI_RADIO: no longer STM.7
- net MOSI_SR: no longer STM.33
- net N$6: now also R39.1, R40.2; no longer R7.2, U$14.P$5, U$5.P$1
- net N$7: now also R41.1, R42.2; no longer R11.2, U$14.P$7, U$8.P$1
- net N$8: now also R43.1, R44.2; no longer R12.2, U$14.P$10, U$9.P$1
- net N$9: now also R45.1, R46.2; no longer R13.2, U$10.P$1, U$14.P$11
- net OE_SR: now also R14.2, U$13.13
- net RX1_BLE: no longer STM.31
- net RX2_GPS: no longer STM.9
- net SCK_RADIO: no longer STM.22
- net SCK_SR: no longer STM.11
- net STEP_DRIVER: no longer STM.26
- net SW_AMP: no longer STM.10
- net TX1_BLE: no longer STM.30
- net TX2_GPS: no longer STM.8
Routing:
- net SP-: track 17.6 -> 0.00 mm
- net MISO_SR: track 10.5 -> 0.18 mm
- net ADC_FOTO: track 26.5 -> 18.2 mm
- net SCK_SR: track 23.9 -> 19.9 mm
- net SCK_RADIO: track 84.0 -> 80.0 mm
- net IRQ_RADIO: track 23.6 -> 20.0 mm
- net MOSI_RADIO: track 27.3 -> 23.8 mm
- net SW_AMP: track 24.6 -> 21.1 mm
- net INA_SP+: track 10.1 -> 7.00 mm
- net MISO_RADIO: track 104.8 -> 102.6 mm
- net DIR_DRIVER: track 11.4 -> 9.26 mm
- net RX2_GPS: track 26.1 -> 24.7 mm
- net STEP_DRIVER: track 8.75 -> 7.42 mm
- net RX1_BLE: track 14.9 -> 13.8 mm
- net TX1_BLE: track 12.3 -> 11.3 mm

Commit message: ПЛАТЫ, АААААААААААААААААААААААААААА
Parts:
- JP2: device pinhead:1X16 -> pinhead:1X18
- moved JP2 65.3 mm to (-78.0, -365.8)
- moved JP1 65.2 mm to (-88.2, -360.4)
Connections:
- removed net BUS+: X1.1, X2.1
- new net 4V: JP1.10, X1.1, X2.1
- new net AUX_RADIO: JP2.10, STM.2
- new net C0: JP2.1
- new net GERMO: JP2.18, U$13.15
- new net NH3: JP2.3
- new net OE: JP1.4
- new net SHIFT_2: JP2.17
- net 3V3: now also JP2.6
- net 5V: now also JP2.7
- net BUZZER: no longer STM.14
- net CS_LIS: now also JP1.8
- net CS_LSM: now also JP1.9
- net GND: now also JP2.5
- net LATCH: now also JP1.5
- net M0_RADIO: now also JP2.12, STM.4; no longer STM.15
- net M1_RADIO: now also JP2.11, STM.3; no longer STM.17
- net MICS: now also JP2.4
- net MISO_SENS: now also JP1.2
- net MOSI_SENS: now also JP1.1
- net NO2: now also JP2.2
- net RX_GPS: now also JP2.14
- net RX_LIDAR: now also JP2.15
- net RX_RADIO: now also JP1.6
- net SCK_SENS: now also JP1.3
- net SCL: now also JP2.9
- net SDA: now also JP2.8
- net TX_GPS: now also JP2.13
- net TX_LIDAR: now also JP2.16
- net TX_RADIO: now also JP1.7

Commit message: схемы плат
Parts:
- removed R11, R12, R13, R39, R40, R41, R42, R43, R44, R45, R46, R8: 5k1, rcl:R0603
- R0, R7: value 5k1 -> 2k2
- renumbered STM to STM32F411, U$18 to MOTOR_SP_V, U$19 to MOTOR_SP_G, U$20 to FOTO0, X1 to PERE1, X2 to PERE2
Connections:
- removed net H3: R12.2, U$14.P$10
- removed net N$34: R13.1, R45.2
- removed net N$36: R12.1, R43.2
- removed net N$37: R11.1, R41.2
- removed net N$6: R39.1, R40.2
- removed net N$7: R41.1, R42.2
- removed net N$8: R43.1, R44.2
- removed net N$9: R45.1, R46.2
- net 3V3: no longer R40.1, R42.1, R44.1, R46.1
- net 5V: no longer R39.2, R8.1
- net CO: no longer R8.2
- net MICS: no longer R13.2
- net NH3: now also U$14.P$10
- net NO2: no longer R11.2

Commit message: подготовлены файлы для зимней сессии
Connections:
- removed net LATCH: JP1.5, U$13.12
- removed net OE: JP1.4
- removed net SHIFT2: U$13.9
- removed net SHIFT_2: JP2.17
- new net SHIFT: JP2.17, U$13.9
- net LATCH_SR: now also JP1.5, U$13.12
- net OE_SR: now also JP1.4
Changed lines of the file:
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@@
 <contactref element="U$13" pad="13"/>
 <contactref element="R14" pad="2"/>
-<wire x1="-98.85" y1="-284.6" x2="-60.9" y2="-127.875" width="0" layer="19" extent="1-1"/>
-<wire x1="56.9" y1="27.63" x2="-60.9" y2="-127.875" width="0" layer="19" extent="1-1"/>
+<contactref element="JP1" pad="4"/>
+<wire x1="-98.85" y1="-284.6" x2="-92.01" y2="-360.4" width="0" layer="19" extent="1-1"/>
+<wire x1="-60.9" y1="-127.875" x2="-98.85" y2="-284.6" width="0" layer="19" extent="1-1"/>
+<wire x1="56.93" y1="27.6" x2="-60.9" y2="-127.875" width="0" layer="19" extent="1-1"/>
 </signal>
 <signal name="LATCH_SR">
@@
 <wire x1="59.55" y1="22.55" x2="56.9" y2="22.55" width="0.3" layer="1"/>
 <wire x1="62.4" y1="25.4" x2="59.55" y2="22.55" width="0.3" layer="1"/>
+<contactref element="JP1" pad="5"/>
+<contactref element="U$13" pad="12"/>
+<wire x1="-60.9" y1="-128.525" x2="-89.47" y2="-360.4" width="0" layer="19" extent="1-1"/>
+<wire x1="56.9" y1="22.55" x2="-60.9" y2="-128.525" width="0" layer="19" extent="1-1"/>
 </signal>
 <signal name="MOSI_SR">
@@
 <contactref element="U$13" pad="11"/>
 </signal>
-<signal name="LATCH">
-<contactref element="U$13" pad="12"/>
-<contactref element="JP1" pad="5"/>
-<wire x1="-60.9" y1="-128.525" x2="-89.47" y2="-360.4" width="0" layer="19" extent="1-1"/>
-</signal>
 <signal name="MOTOR2+">
 <contactref element="U$13" pad="2"/>
@@
 <wire x1="-75.05" y1="-193.1" x2="-66.7" y2="-129.825" width="0" layer="19" extent="1-1"/>
 </signal>
-<signal name="SHIFT2">
+<signal name="SHIFT">
 <contactref element="U$13" pad="9"/>
+<contactref element="JP2" pad="17"/>
+<wire x1="-58.95" y1="-365.8" x2="-60.9" y2="-130.475" width="0" layer="19" extent="1-1"/>
 </signal>
 <signal name="MOTOR2-">
@@
 <wire x1="41.9" y1="63.19" x2="-76.73" y2="-365.8" width="0" layer="19" extent="1-1"/>
 </signal>
-<signal name="OE">
-<contactref element="JP1" pad="4"/>
-</signal>
 <signal name="4V">
 <contactref element="PERE2" pad="1"/>
@@
 <wire x1="-76.77" y1="-360.4" x2="-68.85" y2="-183.4" width="0" layer="19" extent="1-1"/>
 </signal>
-<signal name="SHIFT_2">
-<contactref element="JP2" pad="17"/>
-</signal>
 <signal name="C0">

Commit message: распиновка разъемов плат
Parts:
- removed JP1: (no value), pinhead:1X10
- removed JP2: (no value), pinhead:1X18
- removed U$3: BOARD_SHAPE, UNKNOWN-2024:BOARD_SHAPE
- added JP3: (no value), pinhead:1X16
- added JP4: (no value), pinhead:1X12
Connections:
- net 3V3: now also JP4.3; no longer JP2.6
- net 4V: now also JP4.1; no longer JP1.10
- net 5V: now also JP4.4; no longer JP2.7
- net AUX_RADIO: now also JP4.7; no longer JP2.10
- net C0: now also JP3.13; no longer JP2.1
- net CS_LIS: now also JP3.9; no longer JP1.8
- net CS_LSM: now also JP3.10; no longer JP1.9
- net GERMO: now also JP4.6; no longer JP2.18
- net GND: now also JP4.2; no longer JP2.5
- net LATCH_SR: now also JP3.12; no longer JP1.5
- net M0_RADIO: now also JP4.9; no longer JP2.12
- net M1_RADIO: now also JP4.8; no longer JP2.11
- net MICS: now also JP3.16; no longer JP2.4
- net MISO_SENS: now also JP3.4; no longer JP1.2
- net MOSI_SENS: now also JP3.3; no longer JP1.1
- net NH3: now also JP3.15; no longer JP2.3
- net NO2: now also JP3.14; no longer JP2.2
- net OE_SR: now also JP3.11; no longer JP1.4
- net RX_GPS: now also JP4.11; no longer JP2.14
- net RX_LIDAR: now also JP3.7; no longer JP2.15
- net RX_RADIO: now also JP3.5; no longer JP1.6
- net SCK_SENS: now also JP4.12; no longer JP1.3
- net SCL: now also JP3.2; no longer JP2.9
- net SDA: now also JP3.1; no longer JP2.8
- net SHIFT: now also JP4.5; no longer JP2.17
- net TX_GPS: now also JP4.10; no longer JP2.13
- net TX_LIDAR: now also JP3.8; no longer JP2.16
- net TX_RADIO: now also JP3.6; no longer JP1.7
Other:
- outline, holes or cut-outs redrawn
