File: schematics/board/MK.brd (EAGLE design)
At the start: 76 x 76 mm, 64 parts

Commit message: jhgh
Parts:
- removed U$4: PBS_SMD_X13, UNKNOWN-2024:PBD_SMD_X13
- removed U$6: PBS_SMD_X9, UNKNOWN-2024:PBS_SMD_X9
- added SP: MOLEX-2-1.25, UNKNOWN-2024:53047-02
- moved R21 374.7 mm to (27.7, 64.5)
- moved R14 358.7 mm to (38.4, 46.4), flipped to the bottom
- moved R35 354.7 mm to (54.4, 56.5), flipped to the bottom, turned to 180 degrees
- moved R33 347.0 mm to (51.3, 56.5), flipped to the bottom, turned to 180 degrees
- moved R32 343.2 mm to (51.5, 50.0), flipped to the bottom
- moved R37 340.4 mm to (54.5, 45.1), flipped to the bottom, turned to 180 degrees
- moved U$21 336.5 mm to (46.9, 53.2), flipped to the bottom
- moved R36 332.9 mm to (38.2, 42.1), flipped to the bottom, turned to 180 degrees
- moved R34 332.3 mm to (48.0, 44.1), flipped to the bottom
- moved U$23 326.0 mm to (46.2, 46.9), flipped to the bottom
- moved U$14 316.3 mm to (21.9, 36.8), flipped to the bottom
- moved R31 312.4 mm to (53.0, 27.8), flipped to the bottom, turned to 270 degrees
- moved R30 307.1 mm to (50.9, 27.8), flipped to the bottom, turned to 270 degrees
- moved R29 301.2 mm to (53.0, 24.7), flipped to the bottom, turned to 90 degrees
- moved MOTOR_SP_V 298.5 mm to (46.1, 74.5), turned to 350 degrees
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Connections:
- removed net ADC_FOTO: U$4.4
- removed net CE_RADIO: U$6.9
- removed net CS_RADIO: U$6.8
- removed net DIR_DRIVER: U$4.12
- removed net IRQ_RADIO: U$6.7
- removed net MISO_RADIO: U$6.5
- removed net MISO_SR: U$4.6
- removed net MOSI: U$13.14
- removed net MOSI_RADIO: U$6.6
- removed net MOSI_SR: U$4.5
- removed net RX1_BLE: U$4.10
- removed net RX2_GPS: U$6.2
- removed net SCK: U$13.11
- removed net SCK_RADIO: U$6.4
- removed net SCK_SR: U$4.7
- removed net STEP_DRIVER: U$4.13
- removed net SW_AMP: U$6.1
- removed net TX1_BLE: U$4.11
- removed net TX2_GPS: U$6.3
- net 3V3: no longer U$4.1
- net 5V: no longer U$4.3
- net GND: no longer U$4.2
- net LATCH_SR: no longer U$4.9
- net MK_MOTOR1+: now also U$13.4
- net MK_MOTOR1-: now also U$13.5
- net MK_MOTOR2+: now also U$13.2
- net MK_MOTOR2-: now also U$13.3
- net MOSI_SENS: now also U$13.14
- net MOTOR1+: no longer U$13.4
- net MOTOR1-: no longer U$13.5
- net MOTOR2+: no longer U$13.2
- net MOTOR2-: no longer U$13.3
- net OE_SR: no longer U$4.8
- net SCK_SENS: now also U$13.11
- net SP+: now also SP.1
- net SP-: now also SP.2
Routing:
- net GND: track 235.2 -> 66.4 mm, vias 8 -> 3
- net 3V3: track 160.3 -> 13.8 mm, vias 3 -> 0
- net MISO_RADIO: track 102.6 -> 0.00 mm, vias 1 -> 0
- net M0_RADIO: track 0.00 -> 98.1 mm, vias 0 -> 5
- net SP-: track 0.00 -> 92.3 mm, vias 0 -> 2
- net MICS: track 0.00 -> 80.4 mm
- net SCK_RADIO: track 80.0 -> 0.00 mm
- net NH3: track 0.00 -> 78.5 mm
- net NO2: track 0.00 -> 76.5 mm
- net N$4: track 0.00 -> 70.2 mm, vias 0 -> 5
- net M1_RADIO: track 0.00 -> 63.4 mm, vias 0 -> 4
- net SP+: track 19.4 -> 74.0 mm
- net SCK_SENS: track 0.00 -> 53.7 mm, vias 0 -> 7
- net LATCH_SR: track 21.4 -> 74.7 mm, vias 1 -> 2
- net N$21: track 0.00 -> 49.7 mm, vias 0 -> 1
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Other:
- board text removed: "CE"
- board text removed: "CS"
- board text removed: "DIR"
- board text removed: "FOTO"
- board text removed: "IRQ"
- board text removed: "MISO"
- board text removed: "OE"
- board text removed: "RX1"
- board text removed: "RX2"
- board text removed: "SW"
- board text removed: "TX2"

Commit message: Плата Радио
Parts:
- moved U$1 38.1 mm to (120.4, 23.6)
Routing:
- net GND: track 66.4 -> 371.2 mm, vias 3 -> 27
- net 3V3: track 13.8 -> 271.9 mm, vias 0 -> 18
- net BUZZER: track 26.3 -> 68.6 mm, vias 2 -> 4
- net 5V: track 69.9 -> 108.7 mm
- net SDA: track 48.8 -> 85.6 mm, vias 1 -> 5
- net MOSI_SENS: track 16.5 -> 51.7 mm, vias 0 -> 4
- net SCL: track 45.7 -> 75.5 mm, vias 0 -> 3
- net 4V: track 0.00 -> 28.9 mm
- net M1_RADIO: track 63.4 -> 73.2 mm
- net MK_MOTOR2+: track 39.5 -> 36.1 mm
- net SHIFT: track 27.7 -> 29.3 mm
- net MK_MOTOR1+: track 24.8 -> 26.2 mm
- net MK_MOTOR1-: track 10.3 -> 11.5 mm
- net N$20: track 43.9 -> 44.7 mm
- net SCK_SENS: track 53.7 -> 54.4 mm

Commit message: цывуа4кеп5рн6го7л8шщ9
Routing:
- net N$24: track 18.3 -> 19.4 mm
- net PERE1: track 22.1 -> 22.7 mm
Changed lines of the file:
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@@
 <wire x1="47.8" y1="20.395" x2="47.835" y2="20.43" width="0.3" layer="16"/>
 <wire x1="47.835" y1="20.43" x2="47.835" y2="31.755025" width="0.3" layer="16"/>
-<wire x1="47.835" y1="31.755025" x2="49.7" y2="33.620025" width="0.3" layer="16"/>
-<wire x1="49.7" y1="47.35" x2="52.35" y2="50" width="0.3" layer="16"/>
-<wire x1="49.7" y1="33.620025" x2="49.7" y2="47.35" width="0.3" layer="16"/>
+<wire x1="47.835" y1="31.755025" x2="50.3" y2="34.220025" width="0.3" layer="16"/>
+<wire x1="52.35" y1="49.85" x2="52.35" y2="50" width="0.3" layer="16"/>
+<wire x1="52.35" y1="49.85" x2="50.3" y2="47.8" width="0.3" layer="16"/>
+<wire x1="50.3" y1="34.220025" x2="50.3" y2="47.8" width="0.3" layer="16"/>
 <wire x1="52.35" y1="50" x2="52.35" y2="54.6" width="0.3" layer="16"/>
 <wire x1="52.35" y1="54.6" x2="50.45" y2="56.5" width="0.3" layer="16"/>
@@
 <wire x1="45.562634375" y1="72.467196875" x2="55.2282" y2="62.80163125" width="0.3" layer="16"/>
 <wire x1="55.2282" y1="62.80163125" x2="55.2282" y2="59.29836875" width="0.3" layer="16"/>
-<wire x1="52.1" y1="48.5282" x2="48.2395" y2="48.5282" width="0.3" layer="1"/>
-<wire x1="48.2395" y1="48.5282" x2="47.8668" y2="48.9009" width="0.3" layer="1"/>
-<via x="47.8668" y="48.9009" extent="1-16" drill="0.35"/>
-<wire x1="47.8668" y1="48.9009" x2="47.8668" y2="49.6382" width="0.3" layer="16"/>
-<wire x1="47.8668" y1="49.6382" x2="47.535" y2="49.97" width="0.3" layer="16"/>
+<wire x1="52.1" y1="48.5282" x2="51.95" y2="48.3782" width="0.3" layer="1"/>
+<wire x1="51.95" y1="48.3782" x2="48.0941" y2="48.3782" width="0.3" layer="1"/>
+<wire x1="48.0668" y1="48.3509" x2="48.0941" y2="48.3782" width="0.3" layer="1"/>
+<via x="48.0668" y="48.3509" extent="1-16" drill="0.35"/>
+<wire x1="48.0668" y1="48.3509" x2="48.0668" y2="49.4382" width="0.3" layer="16"/>
+<wire x1="48.0668" y1="49.4382" x2="47.535" y2="49.97" width="0.3" layer="16"/>
 </signal>
 <signal name="PERE1">
@@
 <contactref element="R23" pad="1"/>
 <via x="31.8" y="47.9" extent="1-16" drill="0.35"/>
-<wire x1="46.52460625" y1="47.4" x2="51.55" y2="47.4" width="0.3" layer="1"/>
+<wire x1="50.85" y1="46.7" x2="47.22460625" y2="46.7" width="0.3" layer="1"/>
+<wire x1="50.85" y1="46.7" x2="51.55" y2="47.4" width="0.3" layer="1"/>
 <wire x1="31.902" y1="48.102" x2="37.8" y2="48.102" width="0.3" layer="1"/>
 <wire x1="31.902" y1="48.102" x2="31.8" y2="48" width="0.3" layer="1"/>
@@
 <wire x1="37.8" y1="48.102" x2="38.016" y2="48.318" width="0.3" layer="1"/>
 <wire x1="38.016" y1="48.318" x2="45.60660625" y2="48.318" width="0.3" layer="1"/>
-<wire x1="45.60660625" y1="48.318" x2="46.52460625" y2="47.4" width="0.3" layer="1"/>
+<wire x1="45.60660625" y1="48.318" x2="47.22460625" y2="46.7" width="0.3" layer="1"/>
 </signal>
 <signal name="PERE2">
@@
 <wire x1="47.8" y1="45.15" x2="47.8" y2="46.044975" width="0.3" layer="16"/>
 <wire x1="47.8" y1="46.044975" x2="47.15" y2="46.694975" width="0.3" layer="16"/>
-<wire x1="49.705" y1="48.13" x2="47.22" y2="48.13" width="0.3" layer="16"/>
-<wire x1="47.15" y1="48.2" x2="47.22" y2="48.13" width="0.3" layer="16"/>
+<wire x1="49.705" y1="47.38" x2="47.97" y2="47.38" width="0.3" layer="16"/>
+<wire x1="47.15" y1="48.2" x2="47.97" y2="47.38" width="0.3" layer="16"/>
 <wire x1="49.705" y1="49.07" x2="48.805" y2="49.97" width="0.3" layer="16"/>
-<wire x1="49.705" y1="49.07" x2="49.705" y2="48.13" width="0.3" layer="16"/>
+<wire x1="49.705" y1="49.07" x2="49.705" y2="47.38" width="0.3" layer="16"/>
 <wire x1="48.805" y1="49.97" x2="48.835" y2="50" width="0.3" layer="16"/>
 <wire x1="48.835" y1="50" x2="50.65" y2="50" width="0.3" layer="16"/>
@@
 <wire x1="54.45" y1="44.2" x2="55.35" y2="45.1" width="0.3" layer="16"/>
 <wire x1="45.25" y1="45.6" x2="45.214871875" y2="45.564871875" width="0.3" layer="16"/>
-<wire x1="45.25" y1="45.6" x2="45.25" y2="44.8218" width="0.3" layer="16"/>
-<wire x1="45.25" y1="44.8218" x2="45.2282" y2="44.8" width="0.3" layer="16"/>
-<via x="45.2282" y="44.8" extent="1-16" drill="0.35"/>
-<wire x1="45.2282" y1="44.8" x2="45.4282" y2="45" width="0.3" layer="1"/>
-<wire x1="45.4282" y1="45" x2="51.1" y2="45" width="0.3" layer="1"/>
+<wire x1="45.25" y1="45.6" x2="45.25" y2="44.7218" width="0.3" layer="16"/>
+<wire x1="45.25" y1="44.7218" x2="45.2282" y2="44.7" width="0.3" layer="16"/>
+<via x="45.2282" y="44.7" extent="1-16" drill="0.35"/>
+<wire x1="45.2282" y1="44.7" x2="45.5282" y2="45" width="0.3" layer="1"/>
+<wire x1="45.5282" y1="45" x2="51.1" y2="45" width="0.3" layer="1"/>
 </signal>
 <signal name="MK_MOTOR1-">
