File: schematics/board/RADIO.brd (EAGLE design)
At the start: 76 x 76 mm, 50 parts, among them J1 IPX-RADIO, J2 IPX-ANT

Commit message: iyrd
Parts:
- moved C14 105.3 mm to (100.6, 15.3), turned to 90 degrees
- moved 5V 104.1 mm to (93.0, 12.4)
- moved U$2 102.3 mm to (94.8, 17.1), turned to 270 degrees
- moved C16 98.3 mm to (90.8, 8.40), turned to 270 degrees
- moved C12 98.1 mm to (86.6, 16.2), turned to 90 degrees
- moved C13 98.0 mm to (78.7, 20.2)
- moved R11 93.3 mm to (97.5, 12.5)
- moved 3V3 92.8 mm to (75.1, 12.0), turned to 180 degrees
- moved R5 92.7 mm to (86.8, 12.3)
- moved R10 90.6 mm to (98.4, 15.3), turned to 270 degrees
- moved MP1584-5V 86.7 mm to (93.0, 12.4), turned to 270 degrees
- moved R9 84.4 mm to (98.4, 18.9), turned to 90 degrees
- moved R7 83.4 mm to (79.7, 14.5), turned to 180 degrees
- moved U$5 82.3 mm to (78.7, 17.2), turned to 270 degrees
- moved C11 81.2 mm to (89.7, 16.5), turned to 90 degrees
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
Commit message: дс дс
Parts:
- moved MP1584-3V3 45.4 mm to (37.8, 37.8)
- moved R10 45.4 mm to (60.8, 40.8)
- moved R12 45.4 mm to (38.3, 39.9)
- moved R9 45.4 mm to (60.8, 44.4)
- moved 3V3 45.4 mm to (37.5, 37.5)
- moved 5V 45.4 mm to (55.4, 37.9)
- moved C10 45.4 mm to (48.2, 35.0)
- moved C11 45.4 mm to (52.1, 42.0)
- moved C12 45.4 mm to (49.0, 41.7)
- moved C13 45.4 mm to (41.1, 45.7)
- moved C16 45.4 mm to (53.2, 33.9)
- moved C3 45.4 mm to (33.7, 37.9)
- moved C4 45.4 mm to (34.1, 41.6)
- moved C5 45.4 mm to (31.2, 41.7)
- moved C6 45.4 mm to (56.9, 39.8)
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Routing:
- net GND: track 181.9 -> 309.0 mm, vias 2 -> 12
- net BUS+: track 0.00 -> 57.5 mm
- net N$13: track 0.00 -> 56.6 mm, vias 0 -> 2
- net N$17: track 0.00 -> 43.4 mm, vias 0 -> 2
- net 5V: track 76.8 -> 108.0 mm, vias 2 -> 4
- net N$9: track 0.00 -> 30.1 mm, vias 0 -> 2
- net N$18: track 0.00 -> 24.8 mm, vias 0 -> 2
- net N$12: track 0.00 -> 24.4 mm, vias 0 -> 4
- net 3V3: track 92.3 -> 114.9 mm
- net N$15: track 0.00 -> 15.3 mm, vias 0 -> 3
- net N$14: track 0.00 -> 10.5 mm
- net N$10: track 0.00 -> 10.3 mm
- net N$16: track 0.00 -> 6.32 mm, vias 0 -> 2
- net N$19: track 0.00 -> 4.15 mm
- net N$11: track 0.00 -> 2.14 mm
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
Commit message: Платки там
Parts:
- removed C1: 100nF, rcl:C0603
- removed C2: 220uF, UNKNOWN-2024:ECAP220-CMD
- removed J1: IPX-RADIO, UNKNOWN-2024:U.FL-R-SMT-1(10)
- removed J2: IPX-ANT, UNKNOWN-2024:U.FL-R-SMT-1(10)
- removed LED1: AMP1, led:CHIPLED_0603
- removed LED2: AMP2, led:CHIPLED_0603
- removed NRF24LO1: NRF24L01_ML01SP4, UNKNOWN-2024:NRF24L01_ML01SP4
- removed R1, R2, R3, R4: 2k, rcl:R0603
- removed ROTATE1, ROTATE2, SW: CONNECT_3, UNKNOWN-2024:CONNECT_3
- removed XQ-02A: XQ-02A, UNKNOWN-2024:XQ-02A
- added JP1: (no value), pinhead:1X10
- added JP2: (no value), pinhead:1X16
Connections:
- removed net ANT_RADIO: J2.3, XQ-02A.ANT
- removed net N$1: LED1.C, R1.2
- removed net N$2: LED2.C, R2.2
- removed net N$3: LED1.A, ROTATE1.2
- removed net N$4: LED2.A, ROTATE2.2
- removed net N$5: R2.1, XQ-02A.LED2
- removed net N$6: R1.1, XQ-02A.LED1
- removed net N$7: R3.2, SW.1
- removed net N$8: R4.2, SW.3
- removed net RF-IN: J1.3, XQ-02A.RF-IN
- removed net SW: SW.2, XQ-02A.SW
- net 3V3: no longer NRF24LO1.P$1, ROTATE1.1, ROTATE2.1
- net 5V: no longer C1.2, C2.P$1, R3.1, XQ-02A.5V
- net CE_RADIO: no longer NRF24LO1.P$2
- net CS_RADIO: no longer NRF24LO1.P$3
- net GND: no longer C1.1, C2.P$2, J1.1, J1.2, J2.1, J2.2, NRF24LO1.P$8, R4.1, ROTATE1.3, ROTATE2.3, XQ-02A.GND, XQ-02A.GND1, XQ-02A.GND2, XQ-02A.GND3, XQ-02A.GND4, XQ-02A.GND5
- net IRQ_RADIO: no longer NRF24LO1.P$7
- net MISO_RADIO: no longer NRF24LO1.P$6
- net MOSI_RADIO: no longer NRF24LO1.P$5
- net SCK_RADIO: no longer NRF24LO1.P$4
Routing:
- net GND: track 309.0 -> 187.0 mm
- net 5V: track 108.0 -> 92.2 mm
- net 3V3: track 114.9 -> 100.9 mm, vias 3 -> 2
- net SW: track 11.3 -> 0.00 mm
- net N$3: track 3.75 -> 0.00 mm
- net N$4: track 3.69 -> 0.00 mm
- net IRQ_RADIO: track 13.5 -> 10.3 mm
- net N$6: track 3.16 -> 0.00 mm
- net N$5: track 2.44 -> 0.00 mm
- net ANT_RADIO: track 2.26 -> 0.00 mm
- net RF-IN: track 2.21 -> 0.00 mm
- net N$2: track 2.10 -> 0.00 mm
- net N$1: track 2.00 -> 0.00 mm
- net N$8: track 1.99 -> 0.00 mm
- net N$7: track 1.99 -> 0.00 mm
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
Commit message: ПЛАТЫ, АААААААААААААААААААААААААААА
Parts:
- added JP3: (no value), pinhead:1X18
- added R1: 10k, rcl:R0603
- added R2: 100R, rcl:R0603
- added S1: (no value), UNKNOWN-2024:SS_12D11
- added SI2302CDS: SI2302CDS, CanCubeSat:SOT23-3
- added U$10: LIS3MDL, UNKNOWN-2024:LIS3MDL
- added U$18: MOLEX-2-1.25, UNKNOWN-2024:53047-02
- added U$4: E220-400T22S, UNKNOWN-2024:E220-400T22S
- added U$9: LSM6DS3_WITHOUT, UNKNOWN-2024:LSM6DS3_WITHOUT
- added X2: AKKUM, UNKNOWN-2024:JST-2-2.5
- JP2: device pinhead:1X16 -> pinhead:1X08
- U$6: value PBS_SMD_X13 -> MOLEX-2-1.25; device UNKNOWN-2024:PBD_SMD_X13 -> UNKNOWN-2024:53047-02
- U$7: value PBS_SMD_X9 -> MOLEX-2-1.25; device UNKNOWN-2024:PBS_SMD_X9 -> UNKNOWN-2024:53047-02
- U$8: value PBS_SMD_X13 -> JST-6-2.5; device UNKNOWN-2024:PBD_SMD_X13 -> UNKNOWN-2024:JST-6-2.5
- moved U$8 142.7 mm to (8.80, -74.4), flipped to the top, turned to 0 degrees
- moved U$6 128.3 mm to (2.30, -53.7), turned to 0 degrees
- moved U$7 125.6 mm to (2.30, -61.1), turned to 0 degrees
- moved JP1 97.5 mm to (53.8, 78.6)
- moved C9 52.8 mm to (77.8, 58.0), flipped to the bottom
- moved C5 51.9 mm to (77.3, 65.5), flipped to the bottom
- moved R8 51.0 mm to (76.8, 68.9), flipped to the bottom
- moved C8 48.9 mm to (75.6, 58.0), flipped to the bottom
- moved C3 47.5 mm to (74.8, 61.7), flipped to the bottom
- moved C4 46.8 mm to (74.4, 65.4), flipped to the bottom
- moved U$1 41.5 mm to (80.4, 77.1)
- moved 3V3 41.1 mm to (71.0, 61.3), flipped to the bottom
- moved MP1584-3V3 40.6 mm to (70.7, 61.6), flipped to the bottom
- moved R12 39.8 mm to (70.2, 63.7), flipped to the bottom
- moved C7 37.0 mm to (68.4, 61.3), flipped to the bottom
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Connections:
- removed net ADC_FOTO: U$6.10, U$8.4
- removed net CE_RADIO: U$7.1
- removed net CS_RADIO: U$7.2
- removed net DIR_DRIVER: U$6.2, U$8.12
- removed net IRQ_RADIO: U$7.3
- removed net LATCH_SR: U$6.5, U$8.9
- removed net MISO_RADIO: U$7.5
- removed net MOSI_RADIO: U$7.4
- removed net OE_SR: U$6.6, U$8.8
- removed net RX1_BLE: U$6.4, U$8.10
- removed net RX2_GPS: GPS-NEO7M.P$3, U$7.8
- removed net SCK_RADIO: U$7.6
- removed net STEP_DRIVER: U$6.1, U$8.13
- removed net TX1_BLE: U$6.3, U$8.11
- removed net TX2_GPS: GPS-NEO7M.P$2, U$7.7
- new net 3V7: JP1.10
- new net AUX_RADIO: JP3.10, U$4.P$24
- new net BUS+_OUT: S1.3, X2.1
- new net C0: JP2.1, JP3.1
- new net CS_LIS: JP1.8, U$10.CS
- new net CS_LSM: JP1.9, U$9.P$6
- new net GERMO: JP3.18, R2.1
- new net LATCH: JP1.5, U$8.4
- new net M0_RADIO: JP3.12, U$4.P$20
- new net M1_RADIO: JP3.11, U$4.P$21
- new net MICS: JP2.4, JP3.4
- new net MISO_SENS: JP1.2
- new net MOSI: U$8.2
- new net MOSI_SENS: JP1.1
- new net N$2: R1.1, R2.2, SI2302CDS.1
- new net N$5: SI2302CDS.3, U$18.1, U$6.1, U$7.1
- new net NH3: JP2.3, JP3.3
- new net NO2: JP2.2, JP3.2
- new net OE: JP1.4, U$8.5
- new net RX_GPS: GPS-NEO7M.P$3, JP3.14
- new net RX_LIDAR: JP3.15
- new net RX_RADIO: JP1.6, U$4.P$23
- new net SCK: U$8.3
- new net SCK_SENS: JP1.3
- new net SCL: JP2.8, JP3.9
- new net SDA: JP2.7, JP3.8
- new net SHIFT2: U$8.6
- new net SHIFT_2: JP3.17
- new net TX_GPS: GPS-NEO7M.P$2, JP3.13
- new net TX_LIDAR: JP3.16
- new net TX_RADIO: JP1.7, U$4.P$22
- net 3V3: now also JP3.6, U$10.UCC, U$4.P$25, U$9.P$2; no longer U$6.13
- net 5V: now also JP2.6, JP3.7, U$18.2, U$6.2, U$7.2; no longer U$6.11, U$8.3
- net BUS+: now also S1.2
- net GND: now also JP2.5, JP3.5, R1.2, SI2302CDS.2, U$10.GND, U$4.P$11, U$4.P$13, U$4.P$14, U$4.P$15, U$4.P$16, U$4.P$19, U$4.P$2, U$4.P$26, U$4.P$8, U$9.P$3, X2.2; no longer U$6.12, U$8.2
- net MISO_SR: now also U$10.SDO, U$9.P$7; no longer U$6.8, U$8.6
- net MOSI_SR: now also U$10.SDA, U$9.P$5; no longer U$6.9, U$8.5
- net SCK_SR: now also U$10.SCL, U$9.P$4; no longer U$6.7, U$8.7
Routing:
- net GND: track 187.0 -> 0.00 mm, vias 12 -> 0
- net 3V3: track 100.9 -> 0.00 mm, vias 2 -> 0
- net 5V: track 92.2 -> 0.00 mm, vias 4 -> 0
- net SCK_RADIO: track 28.1 -> 0.00 mm
- net MOSI_RADIO: track 18.3 -> 0.00 mm
- net CS_RADIO: track 14.9 -> 0.00 mm
- net RX2_GPS: track 14.9 -> 0.00 mm
- net MISO_RADIO: track 14.8 -> 0.00 mm, vias 2 -> 0
- net CE_RADIO: track 13.0 -> 0.00 mm
- net TX2_GPS: track 12.6 -> 0.00 mm
- net IRQ_RADIO: track 10.3 -> 0.00 mm
- net DIR_DRIVER: track 4.10 -> 0.00 mm, vias 1 -> 0
- net OE_SR: track 4.01 -> 0.00 mm, vias 1 -> 0
- net MOSI_SR: track 4.01 -> 0.00 mm, vias 1 -> 0
- net ADC_FOTO: track 3.97 -> 0.00 mm, vias 1 -> 0
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Other:
- outline, holes or cut-outs redrawn

Commit message: схемы плат
Parts:
- LSM6DS3: value LSM6DS3_WITHOUT -> LSM6DS3
- renumbered U$18 to COMPRESS, U$4 to RADIO, U$6 to VALVE1, U$7 to VALVE2, U$9 to LSM6DS3
Changed lines of the file:
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@@
 <?xml version="1.0" encoding="utf-8"?>
 <!DOCTYPE eagle SYSTEM "eagle.dtd">
-<eagle version="9.6.2">
+<eagle version="9.4.2">
 <drawing>
 <settings>
-<setting alwaysvectorfont="no"/>
+<setting alwaysvectorfont="yes"/>
 <setting verticaltext="up"/>
 </settings>
@@
 <attribute name="VALUE" x="41.1" y="75.425" size="1.27" layer="27"/>
 </element>
-<element name="U$4" library="UNKNOWN-2024" package="E220-400T22S" value="E220-400T22S" x="62" y="35.7" smashed="yes" rot="R90">
+<element name="RADIO" library="UNKNOWN-2024" package="E220-400T22S" value="E220-400T22S" x="62" y="35.7" smashed="yes" rot="R90">
 <attribute name="NAME" x="46.5" y="32.2" size="1.27" layer="25" rot="R90"/>
 </element>
-<element name="U$9" library="UNKNOWN-2024" package="LSM6DS3_WITHOUT" value="LSM6DS3_WITHOUT" x="27.7" y="36.4" smashed="yes" rot="R270">
+<element name="LSM6DS3" library="UNKNOWN-2024" package="LSM6DS3_WITHOUT" value="LSM6DS3" x="27.7" y="36.4" smashed="yes" rot="R270">
 <attribute name="NAME" x="34.7" y="43.4" size="1.27" layer="25" rot="R270"/>
 </element>
@@
 <attribute name="VALUE" x="5.865" y="-36.505" size="1.27" layer="27"/>
 </element>
-<element name="U$18" library="UNKNOWN-2024" package="53047-02" value="MOLEX-2-1.25" x="2.3" y="-46.3" smashed="yes">
+<element name="COMPRESS" library="UNKNOWN-2024" package="53047-02" value="MOLEX-2-1.25" x="2.3" y="-46.3" smashed="yes">
 <attribute name="NAME" x="0.425" y="-44.55" size="1.27" layer="25"/>
 <attribute name="VALUE" x="0.925" y="-49.55" size="1.27" layer="27"/>
 </element>
-<element name="U$6" library="UNKNOWN-2024" package="53047-02" value="MOLEX-2-1.25" x="2.3" y="-53.7" smashed="yes">
+<element name="VALVE1" library="UNKNOWN-2024" package="53047-02" value="MOLEX-2-1.25" x="2.3" y="-53.7" smashed="yes">
 <attribute name="NAME" x="0.425" y="-51.95" size="1.27" layer="25"/>
 <attribute name="VALUE" x="0.925" y="-56.95" size="1.27" layer="27"/>
 </element>
-<element name="U$7" library="UNKNOWN-2024" package="53047-02" value="MOLEX-2-1.25" x="2.3" y="-61.1" smashed="yes">
+<element name="VALVE2" library="UNKNOWN-2024" package="53047-02" value="MOLEX-2-1.25" x="2.3" y="-61.1" smashed="yes">
 <attribute name="NAME" x="0.425" y="-59.35" size="1.27" layer="25"/>
 <attribute name="VALUE" x="0.925" y="-64.35" size="1.27" layer="27"/>
@@
 <contactref element="C16" pad="1"/>
 <contactref element="5V" pad="C"/>
-<contactref element="U$4" pad="P$26"/>
-<contactref element="U$4" pad="P$19"/>
-<contactref element="U$4" pad="P$14"/>
-<contactref element="U$4" pad="P$13"/>
-<contactref element="U$4" pad="P$16"/>
-<contactref element="U$4" pad="P$11"/>
-<contactref element="U$4" pad="P$8"/>
-<contactref element="U$4" pad="P$15"/>
-<contactref element="U$4" pad="P$2"/>
-<contactref element="U$9" pad="P$3"/>
+<contactref element="RADIO" pad="P$26"/>
+<contactref element="RADIO" pad="P$19"/>
+<contactref element="RADIO" pad="P$14"/>
+<contactref element="RADIO" pad="P$13"/>
+<contactref element="RADIO" pad="P$16"/>
+<contactref element="RADIO" pad="P$11"/>
+<contactref element="RADIO" pad="P$8"/>
+<contactref element="RADIO" pad="P$15"/>
+<contactref element="RADIO" pad="P$2"/>
+<contactref element="LSM6DS3" pad="P$3"/>
 <contactref element="U$10" pad="GND"/>
 <contactref element="X2" pad="2"/>
@@
 <contactref element="L_3.3" pad="P$1"/>
 <contactref element="R12" pad="2"/>
-<contactref element="U$4" pad="P$25"/>
-<contactref element="U$9" pad="P$2"/>
+<contactref element="RADIO" pad="P$25"/>
+<contactref element="LSM6DS3" pad="P$2"/>
 <contactref element="U$10" pad="UCC"/>
 <contactref element="JP3" pad="6"/>
@@
 <contactref element="MP1584-5V" pad="P$8"/>
 <contactref element="JP2" pad="6"/>
-<contactref element="U$7" pad="2"/>
-<contactref element="U$6" pad="2"/>
-<contactref element="U$18" pad="2"/>
+<contactref element="VALVE2" pad="2"/>
+<contactref element="VALVE1" pad="2"/>
+<contactref element="COMPRESS" pad="2"/>
 <contactref element="JP3" pad="7"/>
 <wire x1="55.3" y1="56.3" x2="57.5" y2="56.3" width="0" layer="19" extent="16-16"/>
@@
 </signal>
 <signal name="SCK_SR">
-<contactref element="U$9" pad="P$4"/>
+<contactref element="LSM6DS3" pad="P$4"/>
 <contactref element="U$10" pad="SCL"/>
 <wire x1="22.7" y1="36.4" x2="37.32" y2="39.31" width="0" layer="19" extent="1-1"/>
@@
 <signal name="MISO_SR">
 <contactref element="U$10" pad="SDO"/>
-<contactref element="U$9" pad="P$7"/>
+<contactref element="LSM6DS3" pad="P$7"/>
 <wire x1="22.7" y1="28.78" x2="37.32" y2="34.23" width="0" layer="19" extent="1-1"/>
 </signal>
 <signal name="MOSI_SR">
-<contactref element="U$9" pad="P$5"/>
+<contactref element="LSM6DS3" pad="P$5"/>
 <contactref element="U$10" pad="SDA"/>
 <wire x1="22.7" y1="33.86" x2="37.32" y2="36.77" width="0" layer="19" extent="1-1"/>
@@
 </signal>
 <signal name="AUX_RADIO">
-<contactref element="U$4" pad="P$24"/>
+<contactref element="RADIO" pad="P$24"/>
 <contactref element="JP3" pad="10"/>
 <wire x1="24.57" y1="-68.6" x2="53.54" y2="43.7" width="0" layer="19" extent="1-1"/>
 </signal>
 <signal name="RX_RADIO">
-<contactref element="U$4" pad="P$23"/>
+<contactref element="RADIO" pad="P$23"/>
 <contactref element="JP1" pad="6"/>
 <wire x1="54.81" y1="43.7" x2="55.07" y2="78.6" width="0" layer="19" extent="1-1"/>
 </signal>
 <signal name="TX_RADIO">
-<contactref element="U$4" pad="P$22"/>
+<contactref element="RADIO" pad="P$22"/>
 <contactref element="JP1" pad="7"/>
 <wire x1="56.08" y1="43.7" x2="57.61" y2="78.6" width="0" layer="19" extent="1-1"/>
 </signal>
 <signal name="M1_RADIO">
-<contactref element="U$4" pad="P$21"/>
+<contactref element="RADIO" pad="P$21"/>
 <contactref element="JP3" pad="11"/>
 <wire x1="27.11" y1="-68.6" x2="57.35" y2="43.7" width="0" layer="19" extent="1-1"/>
 </signal>
 <signal name="M0_RADIO">
-<contactref element="U$4" pad="P$20"/>
+<contactref element="RADIO" pad="P$20"/>
 <contactref element="JP3" pad="12"/>
 <wire x1="29.65" y1="-68.6" x2="58.62" y2="43.7" width="0" layer="19" extent="1-1"/>
 </signal>
 <signal name="CS_LSM">
-<contactref element="U$9" pad="P$6"/>
+<contactref element="LSM6DS3" pad="P$6"/>
 <contactref element="JP1" pad="9"/>
 <wire x1="22.7" y1="31.32" x2="62.69" y2="78.6" width="0" layer="19" extent="1-1"/>
@@
 </signal>
 <signal name="N$5">
-<contactref element="U$7" pad="1"/>
-<contactref element="U$6" pad="1"/>
-<contactref element="U$18" pad="1"/>
+<contactref element="VALVE2" pad="1"/>
+<contactref element="VALVE1" pad="1"/>
+<contactref element="COMPRESS" pad="1"/>
 <contactref element="SI2302CDS" pad="3"/>
 <wire x1="2.925" y1="-53.25" x2="2.925" y2="-60.65" width="0" layer="19" extent="1-1"/>

Commit message: подготовлены файлы для зимней сессии
Parts:
- X2: device UNKNOWN-2024:JST-2-2.5 -> UNKNOWN-2024:JST-3-2.5
Connections:
- net LATCH renamed LATCH_SR
- net OE renamed OE_SR
- removed net 3V7: JP1.10
- removed net MISO_SR: LSM6DS3.P$7, U$10.SDO
- removed net MOSI: U$8.2
- removed net MOSI_SR: LSM6DS3.P$5, U$10.SDA
- removed net SCK: U$8.3
- removed net SCK_SR: LSM6DS3.P$4, U$10.SCL
- removed net SHIFT2: U$8.6
- removed net SHIFT_2: JP3.17
- new net 4V: JP1.10, X2.3
- new net SHIFT: JP3.17, U$8.6
- net MISO_SENS: now also LSM6DS3.P$7, U$10.SDO
- net MOSI_SENS: now also LSM6DS3.P$5, U$10.SDA, U$8.2
- net SCK_SENS: now also LSM6DS3.P$4, U$10.SCL, U$8.3
Changed lines of the file:
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@@
 <attribute name="VALUE" x="73.8" y="86.556" size="1.27" layer="27" ratio="10"/>
 </element>
-<element name="X2" library="UNKNOWN-2024" package="JST-2-2.5" value="AKKUM" x="76.3" y="23.6" smashed="yes">
+<element name="X2" library="UNKNOWN-2024" package="JST-3-2.5" value="AKKUM" x="76.3" y="23.6" smashed="yes">
 <attribute name="NAME" x="79.84" y="23.6" size="1.016" layer="25" rot="R270" align="bottom-center"/>
 <attribute name="VALUE" x="77.3" y="24.87" size="1.016" layer="27" align="bottom-right"/>
@@
 <wire x1="73.6" y1="27.7" x2="73.6" y2="43.7" width="0" layer="19" extent="1-1"/>
 <wire x1="71.06" y1="27.7" x2="73.6" y2="27.7" width="0" layer="19" extent="1-1"/>
-<wire x1="75.05" y1="23.6" x2="73.6" y2="27.7" width="0" layer="19" extent="1-1"/>
+<wire x1="76.32" y1="23.6" x2="73.6" y2="27.7" width="0" layer="19" extent="1-1"/>
 <wire x1="59.89" y1="27.7" x2="71.06" y2="27.7" width="0" layer="19" extent="1-1"/>
 <wire x1="52.27" y1="27.7" x2="59.89" y2="27.7" width="0" layer="19" extent="1-1"/>
@@
 <wire x1="1.675" y1="-60.65" x2="1.675" y2="-53.25" width="0" layer="19" extent="1-1"/>
 <wire x1="16.95" y1="-68.6" x2="1.675" y2="-60.65" width="0" layer="19" extent="1-1"/>
-</signal>
-<signal name="SCK_SR">
-<contactref element="LSM6DS3" pad="P$4"/>
-<contactref element="U$10" pad="SCL"/>
-<wire x1="22.7" y1="36.4" x2="37.32" y2="39.31" width="0" layer="19" extent="1-1"/>
-</signal>
-<signal name="MISO_SR">
-<contactref element="U$10" pad="SDO"/>
-<contactref element="LSM6DS3" pad="P$7"/>
-<wire x1="22.7" y1="28.78" x2="37.32" y2="34.23" width="0" layer="19" extent="1-1"/>
-</signal>
-<signal name="MOSI_SR">
-<contactref element="LSM6DS3" pad="P$5"/>
-<contactref element="U$10" pad="SDA"/>
-<wire x1="22.7" y1="33.86" x2="37.32" y2="36.77" width="0" layer="19" extent="1-1"/>
 </signal>
 <signal name="BUS+">
@@
 <contactref element="X2" pad="1"/>
 <contactref element="S1" pad="3"/>
-<wire x1="78.5" y1="76" x2="77.55" y2="23.6" width="0" layer="19" extent="1-1"/>
+<wire x1="78.5" y1="76" x2="78.82" y2="23.6" width="0" layer="19" extent="1-1"/>
 </signal>
 <signal name="RX_GPS">
@@
 <signal name="MOSI_SENS">
 <contactref element="JP1" pad="1"/>
+<contactref element="LSM6DS3" pad="P$5"/>
+<contactref element="U$10" pad="SDA"/>
+<contactref element="U$8" pad="2"/>
+<wire x1="37.32" y1="36.77" x2="42.37" y2="78.6" width="0" layer="19" extent="1-1"/>
+<wire x1="22.7" y1="33.86" x2="37.32" y2="36.77" width="0" layer="19" extent="1-1"/>
+<wire x1="12.59" y1="-74.4" x2="22.7" y2="33.86" width="0" layer="19" extent="1-1"/>
 </signal>
 <signal name="MISO_SENS">
 <contactref element="JP1" pad="2"/>
+<contactref element="LSM6DS3" pad="P$7"/>
+<contactref element="U$10" pad="SDO"/>
+<wire x1="37.32" y1="34.23" x2="44.91" y2="78.6" width="0" layer="19" extent="1-1"/>
+<wire x1="22.7" y1="28.78" x2="37.32" y2="34.23" width="0" layer="19" extent="1-1"/>
 </signal>
 <signal name="SCK_SENS">
 <contactref element="JP1" pad="3"/>
-</signal>
-<signal name="OE">
-<contactref element="JP1" pad="4"/>
-<contactref element="U$8" pad="5"/>
-<wire x1="5.01" y1="-74.4" x2="49.99" y2="78.6" width="0" layer="19" extent="1-1"/>
-</signal>
-<signal name="LATCH">
-<contactref element="JP1" pad="5"/>
-<contactref element="U$8" pad="4"/>
-<wire x1="7.59" y1="-74.4" x2="52.53" y2="78.6" width="0" layer="19" extent="1-1"/>
-</signal>
-<signal name="3V7">
+<contactref element="LSM6DS3" pad="P$4"/>
+<contactref element="U$10" pad="SCL"/>
+<contactref element="U$8" pad="3"/>
+<wire x1="37.32" y1="39.31" x2="47.45" y2="78.6" width="0" layer="19" extent="1-1"/>
+<wire x1="22.7" y1="36.4" x2="37.32" y2="39.31" width="0" layer="19" extent="1-1"/>
+<wire x1="10.09" y1="-74.4" x2="22.7" y2="36.4" width="0" layer="19" extent="1-1"/>
+</signal>
+<signal name="4V">
 <contactref element="JP1" pad="10"/>
+<contactref element="X2" pad="3"/>
+<wire x1="73.74" y1="23.6" x2="65.23" y2="78.6" width="0" layer="19" extent="1-1"/>
 </signal>
 <signal name="SDA">
@@
 <wire x1="3.6" y1="-38.5" x2="2.925" y2="-45.85" width="0" layer="19" extent="1-1"/>
 </signal>
-<signal name="SHIFT_2">
+<signal name="SHIFT">
 <contactref element="JP3" pad="17"/>
+<contactref element="U$8" pad="6"/>
+<wire x1="42.35" y1="-68.6" x2="2.51" y2="-74.4" width="0" layer="19" extent="1-1"/>
 </signal>
 <signal name="RX_LIDAR">
@@
 <contactref element="JP3" pad="16"/>
 </signal>
-<signal name="MOSI">
-<contactref element="U$8" pad="2"/>
-</signal>
-<signal name="SCK">
-<contactref element="U$8" pad="3"/>
-</signal>
-<signal name="SHIFT2">
-<contactref element="U$8" pad="6"/>
+<signal name="OE_SR">
+<contactref element="JP1" pad="4"/>
+<contactref element="U$8" pad="5"/>
+<wire x1="5.01" y1="-74.4" x2="49.99" y2="78.6" width="0" layer="19" extent="1-1"/>
+</signal>
+<signal name="LATCH_SR">
+<contactref element="JP1" pad="5"/>
+<contactref element="U$8" pad="4"/>
+<wire x1="7.59" y1="-74.4" x2="52.53" y2="78.6" width="0" layer="19" extent="1-1"/>
 </signal>
 </signals>
