File: schematics/board/RADIO.brd (EAGLE design)
At the start: 76 x 76 mm, 47 parts, among them X2 AKKUM

Commit message: разъем в гермообъеме на 8 пинов
Connections:
- new net CO: JP2.1
- net C0: no longer JP2.1
Changed lines of the file:
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@@
 <?xml version="1.0" encoding="utf-8"?>
 <!DOCTYPE eagle SYSTEM "eagle.dtd">
-<eagle version="9.6.2">
+<eagle version="9.4.2">
 <drawing>
 <settings>
-<setting alwaysvectorfont="no"/>
+<setting alwaysvectorfont="yes"/>
 <setting verticaltext="up"/>
 </settings>
@@
 </signal>
 <signal name="C0">
-<contactref element="JP2" pad="1"/>
 <contactref element="JP4" pad="13"/>
-<wire x1="1.71" y1="-15.4" x2="80" y2="38.57" width="0" layer="19" extent="1-1"/>
 </signal>
 <signal name="NO2">
@@
 <wire x1="80" y1="41.11" x2="7.59" y2="-74.4" width="0" layer="19" extent="1-1"/>
 </signal>
+<signal name="CO">
+<contactref element="JP2" pad="1"/>
+</signal>
 </signals>

Commit message: jhgh
Parts:
- moved S1 22.1 mm to (43.0, 75.3), turned to 15.5 degrees
- moved JP5 2.00 mm to (20.0, 52.0)
Changed lines of the file:
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@@
 <?xml version="1.0" encoding="utf-8"?>
 <!DOCTYPE eagle SYSTEM "eagle.dtd">
-<eagle version="9.4.2">
+<eagle version="9.6.2">
 <drawing>
 <settings>
-<setting alwaysvectorfont="yes"/>
+<setting alwaysvectorfont="no"/>
 <setting verticaltext="up"/>
 </settings>
-<grid distance="1" unitdist="mm" unit="mm" style="lines" multiple="1" display="yes" altdistance="0.1" altunitdist="mm" altunit="mm"/>
+<grid distance="0.5" unitdist="mm" unit="mm" style="lines" multiple="1" display="no" altdistance="0.1" altunitdist="mm" altunit="mm"/>
 <layers>
 <layer number="1" name="Top" color="4" fill="1" visible="yes" active="yes"/>
@@
 <attribute name="VALUE" x="37.32" y="24.07" size="1.27" layer="27"/>
 </element>
-<element name="S1" library="UNKNOWN-2024" package="SS_12D11" value="" x="24" y="64" smashed="yes" rot="R60">
-<attribute name="NAME" x="11.61923125" y="63.66788125" size="1.27" layer="25" ratio="10" rot="R60"/>
-<attribute name="VALUE" x="14.85823125" y="69.27799375" size="1.27" layer="27" ratio="10" rot="R60"/>
+<element name="S1" library="UNKNOWN-2024" package="SS_12D11" value="" x="43" y="75.3" smashed="yes" rot="R15.5">
+<attribute name="NAME" x="33.936621875" y="83.7409125" size="1.27" layer="25" ratio="10" rot="R15.5"/>
+<attribute name="VALUE" x="40.179021875" y="85.472084375" size="1.27" layer="27" ratio="10" rot="R15.5"/>
 </element>
 <element name="X2" library="UNKNOWN-2024" package="JST-3-2.5" value="AKKUM" x="76.3" y="23.6" smashed="yes">
@@
 <attribute name="VALUE" x="76.825" y="70.32" size="1.27" layer="27" rot="R270"/>
 </element>
-<element name="JP5" library="pinhead" library_urn="urn:adsk.eagle:library:325" package="1X12" package3d_urn="urn:adsk.eagle:package:22487/2" value="" x="20" y="50" smashed="yes" rot="R270">
-<attribute name="NAME" x="21.8288" y="65.3162" size="1.27" layer="25" ratio="10" rot="R270"/>
-<attribute name="POPULARITY" value="28" x="20" y="50" size="1.778" layer="27" rot="R270" display="off"/>
-<attribute name="VALUE" x="16.825" y="65.24" size="1.27" layer="27" rot="R270"/>
+<element name="JP5" library="pinhead" library_urn="urn:adsk.eagle:library:325" package="1X12" package3d_urn="urn:adsk.eagle:package:22487/2" value="" x="20" y="52" smashed="yes" rot="R270">
+<attribute name="NAME" x="21.8288" y="67.3162" size="1.27" layer="25" ratio="10" rot="R270"/>
+<attribute name="POPULARITY" value="28" x="20" y="52" size="1.778" layer="27" rot="R270" display="off"/>
+<attribute name="VALUE" x="16.825" y="67.24" size="1.27" layer="27" rot="R270"/>
 </element>
 </elements>
@@
 <wire x1="52.27" y1="27.7" x2="59.89" y2="27.7" width="0" layer="19" extent="1-1"/>
 <wire x1="25.4" y1="65.31" x2="46.83" y2="70.95" width="0" layer="19" extent="1-1"/>
+<wire x1="20" y1="63.43" x2="25.4" y2="65.31" width="0" layer="19" extent="1-1"/>
 <wire x1="11.87" y1="-15.4" x2="22.7" y2="38.94" width="0" layer="19" extent="1-1"/>
 <wire x1="13.05" y1="-34.6" x2="11.87" y2="-15.4" width="0" layer="19" extent="1-1"/>
 <wire x1="4.55" y1="-40.5" x2="13.05" y2="-34.6" width="0" layer="19" extent="1-1"/>
-<wire x1="20" y1="61.43" x2="4.55" y2="-40.5" width="0" layer="19" extent="1-1"/>
 </signal>
 <signal name="3V3">
@@
 <wire x1="22.7" y1="41.48" x2="37.32" y2="44.39" width="0" layer="19" extent="1-1"/>
 <wire x1="25.4" y1="57.69" x2="22.7" y2="41.48" width="0" layer="19" extent="1-1"/>
+<wire x1="20" y1="60.89" x2="25.4" y2="57.69" width="0" layer="19" extent="1-1"/>
 <wire x1="15.09" y1="-74.4" x2="22.7" y2="41.48" width="0" layer="19" extent="1-1"/>
-<wire x1="20" y1="58.89" x2="15.09" y2="-74.4" width="0" layer="19" extent="1-1"/>
 </signal>
 <signal name="5V">
@@
 <wire x1="47.7" y1="63.75" x2="47.75" y2="61.8" width="0" layer="19" extent="16-16"/>
 <wire x1="45.5" y1="63.75" x2="47.7" y2="63.75" width="0" layer="19" extent="16-16"/>
-<wire x1="14.41" y1="-15.4" x2="56.83" y2="52.45" width="0" layer="19" extent="1-1"/>
+<wire x1="20" y1="58.35" x2="45.5" y2="63.75" width="0" layer="19" extent="16-16"/>
+<wire x1="14.41" y1="-15.4" x2="20" y2="58.35" width="0" layer="19" extent="1-1"/>
 <wire x1="1.675" y1="-45.85" x2="14.41" y2="-15.4" width="0" layer="19" extent="1-1"/>
 <wire x1="1.675" y1="-53.25" x2="1.675" y2="-45.85" width="0" layer="19" extent="1-1"/>
 <wire x1="1.675" y1="-60.65" x2="1.675" y2="-53.25" width="0" layer="19" extent="1-1"/>
-<wire x1="20" y1="56.35" x2="1.675" y2="-60.65" width="0" layer="19" extent="1-1"/>
 </signal>
 <signal name="BUS+">
@@
 <contactref element="S1" pad="2"/>
 <wire x1="77.11370625" y1="66" x2="77.3" y2="66.35" width="0" layer="19" extent="16-16"/>
-<wire x1="24" y1="64" x2="52.6" y2="66.725" width="0" layer="19" extent="16-16"/>
+<wire x1="43" y1="75.3" x2="52.6" y2="66.725" width="0" layer="19" extent="16-16"/>
 </signal>
 <signal name="N$9">
@@
 <contactref element="RADIO" pad="P$24"/>
 <contactref element="JP5" pad="7"/>
-<wire x1="20" y1="48.73" x2="53.54" y2="43.7" width="0" layer="19" extent="1-1"/>
+<wire x1="20" y1="50.73" x2="53.54" y2="43.7" width="0" layer="19" extent="1-1"/>
 </signal>
 <signal name="RX_RADIO">
@@
 <contactref element="RADIO" pad="P$21"/>
 <contactref element="JP5" pad="8"/>
-<wire x1="20" y1="46.19" x2="57.35" y2="43.7" width="0" layer="19" extent="1-1"/>
+<wire x1="20" y1="48.19" x2="57.35" y2="43.7" width="0" layer="19" extent="1-1"/>
 </signal>
 <signal name="M0_RADIO">
 <contactref element="RADIO" pad="P$20"/>
 <contactref element="JP5" pad="9"/>
-<wire x1="20" y1="43.65" x2="58.62" y2="43.7" width="0" layer="19" extent="1-1"/>
+<wire x1="20" y1="45.65" x2="58.62" y2="43.7" width="0" layer="19" extent="1-1"/>
 </signal>
 <signal name="CS_LSM">
@@
 <contactref element="X2" pad="1"/>
 <contactref element="S1" pad="3"/>
-<wire x1="26.35" y1="68.07031875" x2="78.82" y2="23.6" width="0" layer="19" extent="1-1"/>
+<wire x1="78.82" y1="23.6" x2="47.5290625" y2="76.55601875" width="0" layer="19" extent="1-1"/>
 </signal>
 <signal name="RX_GPS">
 <contactref element="GPS-NEO7M" pad="P$3"/>
 <contactref element="JP5" pad="11"/>
-<wire x1="20" y1="38.57" x2="25.4" y2="62.77" width="0" layer="19" extent="1-1"/>
+<wire x1="20" y1="40.57" x2="25.4" y2="62.77" width="0" layer="19" extent="1-1"/>
 </signal>
 <signal name="TX_GPS">
 <contactref element="GPS-NEO7M" pad="P$2"/>
 <contactref element="JP5" pad="10"/>
-<wire x1="20" y1="41.11" x2="25.4" y2="60.23" width="0" layer="19" extent="1-1"/>
+<wire x1="20" y1="43.11" x2="25.4" y2="60.23" width="0" layer="19" extent="1-1"/>
 </signal>
 <signal name="MOSI_SENS">
@@
 <contactref element="JP5" pad="12"/>
 <wire x1="22.7" y1="36.4" x2="37.32" y2="39.31" width="0" layer="19" extent="1-1"/>
+<wire x1="20" y1="38.03" x2="22.7" y2="36.4" width="0" layer="19" extent="1-1"/>
 <wire x1="10.09" y1="-74.4" x2="22.7" y2="36.4" width="0" layer="19" extent="1-1"/>
-<wire x1="20" y1="36.03" x2="10.09" y2="-74.4" width="0" layer="19" extent="1-1"/>
 </signal>
 <signal name="4V">
 <contactref element="X2" pad="3"/>
 <contactref element="JP5" pad="1"/>
-<wire x1="20" y1="63.97" x2="73.74" y2="23.6" width="0" layer="19" extent="1-1"/>
+<wire x1="20" y1="65.97" x2="73.74" y2="23.6" width="0" layer="19" extent="1-1"/>
 </signal>
 <signal name="SDA">
@@
 <contactref element="R2" pad="1"/>
 <contactref element="JP5" pad="6"/>
-<wire x1="5.65" y1="-34.6" x2="20" y2="51.27" width="0" layer="19" extent="1-1"/>
+<wire x1="5.65" y1="-34.6" x2="20" y2="53.27" width="0" layer="19" extent="1-1"/>
 </signal>
 <signal name="N$5">
@@
 <contactref element="U$8" pad="6"/>
 <contactref element="JP5" pad="5"/>
-<wire x1="2.51" y1="-74.4" x2="20" y2="53.81" width="0" layer="19" extent="1-1"/>
+<wire x1="20" y1="55.81" x2="2.51" y2="-74.4" width="0" layer="19" extent="1-1"/>
 </signal>
 <signal name="RX_LIDAR">

Commit message: Плата Радио
Parts:
- removed JP2: (no value), pinhead:1X08
- added JP1, JP3: (no value), pinhead:1X04
- added U$7: MOLEX-4-1.25, UNKNOWN-2024:53047-04
- U$8: value JST-6-2.5 -> MOLEX-5-1.25; device UNKNOWN-2024:JST-6-2.5 -> UNKNOWN-2024:53047-05
- moved U$8 162.1 mm to (67.9, 76.5), flipped to the bottom, turned to 214 degrees
- moved VALVE2 131.3 mm to (23.8, 68.4), flipped to the bottom, turned to 125 degrees
- moved VALVE1 129.7 mm to (28.2, 73.4), flipped to the bottom, turned to 137 degrees
- moved COMPRESS 127.6 mm to (33.5, 77.4), flipped to the bottom, turned to 149 degrees
- moved SI2302CDS 100.1 mm to (26.1, 58.0)
- moved R2 90.2 mm to (24.0, 53.9)
- moved R1 89.8 mm to (27.7, 53.9)
- moved X2 60.1 mm to (58.3, 80.9), flipped to the bottom, turned to 195 degrees
- moved C9 19.1 mm to (60.0, 51.2), turned to 0 degrees
- moved R8 17.7 mm to (70.9, 52.2), turned to 90 degrees
- moved C5 16.9 mm to (67.5, 51.7), turned to 180 degrees
- moved C8 16.3 mm to (60.0, 53.4), turned to 0 degrees
- moved C3 13.4 mm to (63.7, 54.2), turned to 90 degrees
- moved C4 12.9 mm to (67.4, 54.6), turned to 180 degrees
- moved LSM6DS3 11.9 mm to (39.4, 38.8), turned to 180 degrees
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Connections:
- net 3V3: now also U$8.5; no longer U$8.1
- net 5V: now also JP3.2, U$7.3; no longer JP2.6
- net CO: now also JP1.1; no longer JP2.1
- net GND: now also JP3.1, U$7.4; no longer JP2.5
- net LATCH_SR: now also U$8.3; no longer U$8.4
- net MICS: now also JP1.4; no longer JP2.4
- net MOSI_SENS: no longer U$8.2
- net NH3: now also JP1.3; no longer JP2.3
- net NO2: now also JP1.2; no longer JP2.2
- net OE_SR: now also U$8.2; no longer U$8.5
- net RX_LIDAR: now also U$7.2
- net SCK_SENS: now also U$8.4; no longer U$8.3
- net SCL: now also JP3.4; no longer JP2.8
- net SDA: now also JP3.3; no longer JP2.7
- net SHIFT: now also U$8.1; no longer U$8.6
- net TX_LIDAR: now also U$7.1
Routing:
- net GND: track 0.00 -> 347.1 mm, vias 0 -> 21
- net 5V: track 0.00 -> 189.8 mm, vias 0 -> 3
- net 3V3: track 0.00 -> 142.3 mm, vias 0 -> 14
- net SCK_SENS: track 0.00 -> 99.0 mm, vias 0 -> 6
- net MISO_SENS: track 0.00 -> 86.1 mm, vias 0 -> 1
- net MOSI_SENS: track 0.00 -> 84.7 mm, vias 0 -> 2
- net SDA: track 0.00 -> 82.2 mm
- net SCL: track 0.00 -> 78.6 mm, vias 0 -> 1
- net CS_LIS: track 0.00 -> 59.6 mm
- net SHIFT: track 0.00 -> 58.7 mm
- net M0_RADIO: track 0.00 -> 55.3 mm, vias 0 -> 1
- net CS_LSM: track 0.00 -> 51.5 mm, vias 0 -> 2
- net LATCH_SR: track 0.00 -> 49.4 mm
- net M1_RADIO: track 0.00 -> 45.4 mm
- net 4V: track 0.00 -> 42.7 mm
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Other:
- board text removed: "3V3"
- board text removed: "5V"
- board text removed: "CE"
- board text removed: "CS"
- board text removed: "DIR"
- board text removed: "FOTO"
- board text removed: "GND"
- board text removed: "IRQ"
- board text removed: "LATCH"
- board text removed: "MISO"
- board text removed: "MOSI"
- board text removed: "OE"
- board text removed: "RX1"
- board text removed: "RX2"
- board text removed: "SCK"
- board text removed: "STEP"
- board text removed: "SW"
- board text removed: "TX1"
- board text removed: "TX2"

Commit message: цывуа4кеп5рн6го7л8шщ9
Parts:
- moved R8 0.10 mm to (71.0, 52.2)
Routing:
- net N$5: track 18.3 -> 26.1 mm
- net N$10: track 21.0 -> 27.1 mm, vias 0 -> 4
- net BUS+: track 66.9 -> 65.1 mm
- net N$9: track 31.5 -> 30.2 mm
- net OE_SR: track 38.5 -> 39.8 mm
- net N$17: track 61.2 -> 62.2 mm
- net N$13: track 56.6 -> 57.6 mm, vias 5 -> 4
- net N$18: track 41.0 -> 41.9 mm
- net CS_LSM: track 51.5 -> 52.3 mm
- net GND: track 347.1 -> 347.9 mm
- net N$16: track 3.86 -> 4.45 mm

Commit message: Поправлены платы МК, Радио, Гермо
Parts:
- moved R12 51.8 mm to (16.1, 43.9)
- moved 3V3 50.8 mm to (14.5, 43.9), turned to 0 degrees
- moved 5V 33.9 mm to (14.5, 40.5)
- moved C13 31.7 mm to (39.4, 59.3)
- moved R6 30.3 mm to (70.0, 63.8), turned to 180 degrees
- moved R11 29.0 mm to (16.1, 40.5), turned to 90 degrees
- moved U$2 26.7 mm to (67.7, 59.3), turned to 0 degrees
- moved R8 26.5 mm to (48.9, 66.8), turned to 180 degrees
- moved U$5 26.3 mm to (42.3, 63.5), turned to 270 degrees
- moved R5 22.6 mm to (71.1, 52.7), turned to 270 degrees
- moved C11 22.4 mm to (67.1, 54.2), turned to 180 degrees
- moved C6 22.1 mm to (63.6, 62.2), turned to 180 degrees
- moved C4 21.7 mm to (47.4, 62.9), turned to 90 degrees
- moved C5 20.9 mm to (49.8, 62.9), turned to 90 degrees
- moved C12 20.5 mm to (67.1, 52.0), turned to 180 degrees
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Connections:
- removed net C0: JP4.13
- net CO: now also JP4.13
- net RX_GPS: now also JP5.10; no longer JP5.11
- net RX_LIDAR: now also JP4.8; no longer JP4.7
- net RX_RADIO: now also JP4.6; no longer JP4.5
- net TX_GPS: now also JP5.11; no longer JP5.10
- net TX_LIDAR: now also JP4.7; no longer JP4.8
- net TX_RADIO: now also JP4.5; no longer JP4.6
Routing:
- net N$17: track 62.2 -> 0.00 mm, vias 2 -> 0
- net GND: track 347.9 -> 403.8 mm, vias 21 -> 38
- net N$13: track 57.6 -> 7.00 mm, vias 4 -> 0
- net 3V3: track 142.7 -> 187.7 mm, vias 14 -> 3
- net CO: track 0.00 -> 38.4 mm
- net N$18: track 41.9 -> 7.10 mm, vias 2 -> 0
- net N$12: track 29.4 -> 0.00 mm
- net N$9: track 30.2 -> 3.69 mm, vias 2 -> 0
- net CS_LIS: track 59.6 -> 39.8 mm, vias 0 -> 1
- net AUX_RADIO: track 40.3 -> 59.4 mm
- net N$14: track 22.2 -> 3.69 mm
- net TX_RADIO: track 36.5 -> 55.0 mm, vias 1 -> 2
- net GERMO: track 3.41 -> 21.6 mm, vias 0 -> 1
- net RX_RADIO: track 39.9 -> 54.9 mm, vias 1 -> 2
- net SCK_SENS: track 99.0 -> 113.3 mm, vias 6 -> 1
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- added copper zone on layer 16, net 3V3
- added copper zone on layer 16, net 5V
- added copper zone on layer 16, net BUS+
- added copper zone on layer 16, net N$11
- added copper zone on layer 16, net N$12
- added copper zone on layer 16, net N$13
- added copper zone on layer 16, net N$16
- added copper zone on layer 16, net N$17
- added copper zone on layer 16, net N$18

Commit message: фцыувкаепнргошщз
Parts:
- moved U$1 56.9 mm to (60.9, 23.6)
- renumbered SI2302CDS to SI2302
Other:
- board text added: "3V3"
- board text added: "4V"
- board text added: "5V"
- board text added: "AUX_R"
- board text added: "CO"
- board text added: "CS_LIS"
- board text added: "CS_LSM"
- board text added: "GERMO"
- board text added: "GND"
- board text added: "LATCH"
- board text added: "M0_R"
- board text added: "M1_R"
- board text added: "MICS"
- board text added: "MISO_S"
- board text added: "MOSI_S"
- board text added: "NH3"
- board text added: "NO2"
- board text added: "OE_SR"
- board text added: "RX_G"
- board text added: "RX_L"
- board text added: "RX_R"
- board text added: "SCK_S"
- board text added: "SCL"
- board text added: "SDA"
- board text added: "SHIFT"
- board text added: "TX_G"
- board text added: "TX_L"
- board text added: "TX_R"

Commit message: проверка плат
Parts:
- JP1: device pinhead:1X04 -> pinhead:1X02
- JP4: device pinhead:1X16 -> pinhead:1X14
- moved JP1 16.0 mm to (47.5, 9.50), turned to 180 degrees
- moved C11 14.1 mm to (57.1, 44.2)
- moved C14 14.1 mm to (25.7, 52.5)
- moved C3 14.1 mm to (60.9, 48.7)
- moved C7 14.1 mm to (56.8, 55.9)
- moved U$8 14.1 mm to (57.9, 66.5)
- moved VALVE1 14.1 mm to (18.2, 63.4)
- moved VALVE2 14.1 mm to (13.8, 58.4)
- moved 3V3 14.1 mm to (4.50, 33.9)
- moved 5V 14.1 mm to (4.50, 30.5)
- moved C10 14.1 mm to (32.9, 56.7)
- moved C12 14.1 mm to (57.1, 42.0)
- moved C13 14.1 mm to (29.4, 49.3)
- moved C15 14.1 mm to (39.5, 46.8)
- moved C16 14.1 mm to (37.4, 46.8)
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Connections:
- net CO renamed FOTO1
- net NO2 renamed FOTO0
- removed net MICS: JP1.4, JP4.16
- removed net NH3: JP1.3, JP4.15
Routing:
- net NH3: track 29.2 -> 0.00 mm
- net MICS: track 23.6 -> 0.00 mm
- net FOTO1: track 38.4 -> 33.8 mm
- net SCL: track 68.4 -> 64.2 mm
- net SDA: track 71.5 -> 68.3 mm
- net LATCH_SR: track 52.3 -> 54.8 mm
- net TX_RADIO: track 55.0 -> 52.7 mm
- net MOSI_SENS: track 72.2 -> 69.9 mm
- net MISO_SENS: track 73.2 -> 70.9 mm
- net RX_RADIO: track 54.9 -> 52.6 mm
- net OE_SR: track 48.5 -> 50.7 mm
- net FOTO0: track 34.0 -> 31.8 mm
- net RX_LIDAR: track 27.4 -> 28.8 mm
- net TX_LIDAR: track 21.5 -> 22.9 mm
- net CS_LSM: track 54.0 -> 53.0 mm
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Other:
- board text added: "FOTO0"
- board text added: "FOTO1"
- board text removed: "CO"
- board text removed: "MICS"
- board text removed: "NH3"
- board text removed: "NO2"

Commit message: Платы готовы
Parts:
- U$1: value Плата радио -> Плата Радио
- renumbered S1 to POWER, U$7 to LIDAR, U$8 to MOTOR_BOARD
Routing:
- net FOTO1: track 33.8 -> 34.8 mm
Other:
- board text added: "FOT 0"
- board text added: "FOT1"
- board text added: "MOSI _S"
- board text removed: "MOSI_S"
