File: schematics/board/RADIO.sch (EAGLE design)
At the start: 49 parts, among them X2 AKKUM

Commit message: фцыувкаепнргошщз
Parts:
- renumbered SI2302CDS to SI2302
Changed lines of the file:
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@@
 <?xml version="1.0" encoding="utf-8"?>
 <!DOCTYPE eagle SYSTEM "eagle.dtd">
-<eagle version="9.4.2">
+<eagle version="9.6.2">
 <drawing>
 <settings>
-<setting alwaysvectorfont="yes"/>
+<setting alwaysvectorfont="no"/>
 <setting verticaltext="up"/>
 </settings>
@@
 <part name="S1" library="UNKNOWN-2024" deviceset="UNICS-SWITCH" device="SS_12D11"/>
 <part name="X2" library="UNKNOWN-2024" deviceset="JST-3-2.5" device="" value="AKKUM"/>
-<part name="SI2302CDS" library="CanCubeSat" deviceset="SI2302CDS" device=""/>
+<part name="SI2302" library="CanCubeSat" deviceset="SI2302CDS" device=""/>
 <part name="R1" library="rcl" library_urn="urn:adsk.eagle:library:334" deviceset="R-US_" device="R0603" package3d_urn="urn:adsk.eagle:package:23555/3" value="10k"/>
 <part name="R2" library="rcl" library_urn="urn:adsk.eagle:library:334" deviceset="R-US_" device="R0603" package3d_urn="urn:adsk.eagle:package:23555/3" value="100R"/>
@@
 <attribute name="NAME" x="-16.51" y="132.842" size="1.778" layer="95"/>
 </instance>
-<instance part="SI2302CDS" gate="G$1" x="276.86" y="134.62" smashed="yes" rot="R180"/>
+<instance part="SI2302" gate="G$1" x="276.86" y="134.62" smashed="yes" rot="R180"/>
 <instance part="R1" gate="G$1" x="287.02" y="129.54" smashed="yes" rot="R90">
 <attribute name="NAME" x="285.5214" y="125.73" size="1.778" layer="95" rot="R90"/>
@@
 </segment>
 <segment>
-<pinref part="SI2302CDS" gate="G$1" pin="S"/>
+<pinref part="SI2302" gate="G$1" pin="S"/>
 <wire x1="287.02" y1="134.62" x2="297.18" y2="134.62" width="0.1524" layer="91"/>
 <label x="292.1" y="134.62" size="1.778" layer="95"/>
@@
 <net name="N$2" class="0">
 <segment>
-<pinref part="SI2302CDS" gate="G$1" pin="G"/>
+<pinref part="SI2302" gate="G$1" pin="G"/>
 <wire x1="276.86" y1="127" x2="276.86" y2="124.46" width="0.1524" layer="91"/>
 <pinref part="R2" gate="G$1" pin="2"/>
@@
 <wire x1="259.08" y1="134.62" x2="241.3" y2="134.62" width="0.1524" layer="91"/>
 <junction x="259.08" y="116.84"/>
-<pinref part="SI2302CDS" gate="G$1" pin="D"/>
+<pinref part="SI2302" gate="G$1" pin="D"/>
 <wire x1="259.08" y1="134.62" x2="266.7" y2="134.62" width="0.1524" layer="91"/>
 <junction x="259.08" y="134.62"/>

Commit message: проверка плат
Parts:
- JP1: device pinhead:PINHD-1X4 -> pinhead:PINHD-1X2
- JP4: device pinhead:PINHD-1X16 -> pinhead:PINHD-1X14
Connections:
- net CO renamed FOTO1
- net NO2 renamed FOTO0
- removed net MICS: JP1.4, JP4.16
- removed net NH3: JP1.3, JP4.15
Changed lines of the file:
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@@
 <?xml version="1.0" encoding="utf-8"?>
 <!DOCTYPE eagle SYSTEM "eagle.dtd">
-<eagle version="9.6.2">
+<eagle version="9.4.2">
 <drawing>
 <settings>
-<setting alwaysvectorfont="no"/>
+<setting alwaysvectorfont="yes"/>
 <setting verticaltext="up"/>
 </settings>
@@
 <part name="VALVE1" library="UNKNOWN-2024" deviceset="MOLEX-2-1.25" device=""/>
 <part name="VALVE2" library="UNKNOWN-2024" deviceset="MOLEX-2-1.25" device=""/>
-<part name="JP4" library="pinhead" library_urn="urn:adsk.eagle:library:325" deviceset="PINHD-1X16" device="" package3d_urn="urn:adsk.eagle:package:22432/2"/>
+<part name="JP4" library="pinhead" library_urn="urn:adsk.eagle:library:325" deviceset="PINHD-1X14" device="" package3d_urn="urn:adsk.eagle:package:22417/2"/>
 <part name="JP5" library="pinhead" library_urn="urn:adsk.eagle:library:325" deviceset="PINHD-1X12" device="" package3d_urn="urn:adsk.eagle:package:22487/2"/>
 <part name="U$7" library="UNKNOWN-2024" deviceset="MOLEX-4-1.25" device=""/>
 <part name="U$8" library="UNKNOWN-2024" deviceset="MOLEX-5-1.25" device=""/>
-<part name="JP1" library="pinhead" library_urn="urn:adsk.eagle:library:325" deviceset="PINHD-1X4" device="" package3d_urn="urn:adsk.eagle:package:22407/2"/>
+<part name="JP1" library="pinhead" library_urn="urn:adsk.eagle:library:325" deviceset="PINHD-1X2" device="" package3d_urn="urn:adsk.eagle:package:22435/2"/>
 <part name="JP3" library="pinhead" library_urn="urn:adsk.eagle:library:325" deviceset="PINHD-1X4" device="" package3d_urn="urn:adsk.eagle:package:22407/2"/>
 </parts>
@@
 <attribute name="NAME" x="250.19" y="90.678" size="1.778" layer="95" rot="R180"/>
 </instance>
-<instance part="JP4" gate="A" x="-35.56" y="76.2" smashed="yes">
+<instance part="JP4" gate="A" x="-35.56" y="78.74" smashed="yes">
 <attribute name="NAME" x="-41.91" y="97.155" size="1.778" layer="95"/>
-<attribute name="VALUE" x="-41.91" y="50.8" size="1.778" layer="96"/>
+<attribute name="VALUE" x="-41.91" y="53.34" size="1.778" layer="96"/>
 </instance>
 <instance part="JP5" gate="G$1" x="-35.56" y="121.92" smashed="yes">
@@
 <attribute name="NAME" x="245.11" y="71.755" size="1.778" layer="95"/>
 </instance>
-<instance part="JP1" gate="A" x="-45.72" y="5.08" smashed="yes">
+<instance part="JP1" gate="G$1" x="-45.72" y="7.62" smashed="yes">
 <attribute name="NAME" x="-52.07" y="13.335" size="1.778" layer="95"/>
-<attribute name="VALUE" x="-52.07" y="-2.54" size="1.778" layer="96"/>
+<attribute name="VALUE" x="-52.07" y="0" size="1.778" layer="96"/>
 </instance>
 <instance part="JP3" gate="A" x="-45.72" y="-10.16" smashed="yes">
@@
 </segment>
 </net>
-<net name="NO2" class="0">
-<segment>
-<wire x1="-71.12" y1="60.96" x2="-38.1" y2="60.96" width="0.1524" layer="91"/>
-<label x="-71.12" y="60.96" size="1.778" layer="95"/>
-<pinref part="JP4" gate="A" pin="14"/>
-</segment>
-<segment>
-<wire x1="-68.58" y1="7.62" x2="-48.26" y2="7.62" width="0.1524" layer="91"/>
-<label x="-68.58" y="7.62" size="1.778" layer="95"/>
-<pinref part="JP1" gate="A" pin="2"/>
-</segment>
-</net>
-<net name="NH3" class="0">
-<segment>
-<wire x1="-38.1" y1="58.42" x2="-71.12" y2="58.42" width="0.1524" layer="91"/>
-<label x="-71.12" y="58.42" size="1.778" layer="95"/>
-<pinref part="JP4" gate="A" pin="15"/>
-</segment>
-<segment>
-<wire x1="-48.26" y1="5.08" x2="-68.58" y2="5.08" width="0.1524" layer="91"/>
-<label x="-68.58" y="5.08" size="1.778" layer="95"/>
-<pinref part="JP1" gate="A" pin="3"/>
-</segment>
-</net>
-<net name="MICS" class="0">
-<segment>
-<wire x1="-71.12" y1="55.88" x2="-38.1" y2="55.88" width="0.1524" layer="91"/>
-<label x="-71.12" y="55.88" size="1.778" layer="95"/>
-<pinref part="JP4" gate="A" pin="16"/>
-</segment>
-<segment>
-<wire x1="-68.58" y1="2.54" x2="-48.26" y2="2.54" width="0.1524" layer="91"/>
-<label x="-68.58" y="2.54" size="1.778" layer="95"/>
-<pinref part="JP1" gate="A" pin="4"/>
-</segment>
-</net>
 <net name="SDA" class="0">
 <segment>
@@
 </segment>
 </net>
-<net name="CO" class="0">
+<net name="FOTO1" class="0">
 <segment>
 <wire x1="-48.26" y1="10.16" x2="-68.58" y2="10.16" width="0.1524" layer="91"/>
 <label x="-68.58" y="10.16" size="1.778" layer="95"/>
-<pinref part="JP1" gate="A" pin="1"/>
+<pinref part="JP1" gate="G$1" pin="1"/>
 </segment>
 <segment>
@@
 </segment>
 </net>
+<net name="FOTO0" class="0">
+<segment>
+<wire x1="-71.12" y1="60.96" x2="-38.1" y2="60.96" width="0.1524" layer="91"/>
+<label x="-71.12" y="60.96" size="1.778" layer="95"/>
+<pinref part="JP4" gate="A" pin="14"/>
+</segment>
+<segment>
+<wire x1="-68.58" y1="7.62" x2="-48.26" y2="7.62" width="0.1524" layer="91"/>
+<label x="-68.58" y="7.62" size="1.778" layer="95"/>
+<pinref part="JP1" gate="G$1" pin="2"/>
+</segment>
+</net>

Commit message: Платы готовы
Parts:
- U$1: value Плата радио -> Плата Радио
- renumbered S1 to POWER, U$7 to LIDAR, U$8 to MOTOR_BOARD
Changed lines of the file:
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@@
 <parts>
 <part name="GPS-NEO7M" library="UNKNOWN-2024" deviceset="GPS-NEO7M" device=""/>
-<part name="U$1" library="UNKNOWN-2024" deviceset="LOGO" device="PCB-&quot;&quot;" value="Плата радио"/>
+<part name="U$1" library="UNKNOWN-2024" deviceset="LOGO" device="PCB-&quot;&quot;" value="Плата Радио"/>
 <part name="MP1584-3V3" library="UNKNOWN-2024" deviceset="MP1584-B" device=""/>
 <part name="U$2" library="UNKNOWN-2024" deviceset="MP2225" device=""/>
@@
 <part name="LSM6DS3" library="UNKNOWN-2024" deviceset="LSM6DS3_WITHOUT" device="" value="LSM6DS3"/>
 <part name="U$10" library="UNKNOWN-2024" deviceset="LIS3MDL" device=""/>
-<part name="S1" library="UNKNOWN-2024" deviceset="UNICS-SWITCH" device="SS_12D11"/>
+<part name="POWER" library="UNKNOWN-2024" deviceset="UNICS-SWITCH" device="SS_12D11"/>
 <part name="X2" library="UNKNOWN-2024" deviceset="JST-3-2.5" device="" value="AKKUM"/>
 <part name="SI2302" library="CanCubeSat" deviceset="SI2302CDS" device=""/>
@@
 <part name="JP4" library="pinhead" library_urn="urn:adsk.eagle:library:325" deviceset="PINHD-1X14" device="" package3d_urn="urn:adsk.eagle:package:22417/2"/>
 <part name="JP5" library="pinhead" library_urn="urn:adsk.eagle:library:325" deviceset="PINHD-1X12" device="" package3d_urn="urn:adsk.eagle:package:22487/2"/>
-<part name="U$7" library="UNKNOWN-2024" deviceset="MOLEX-4-1.25" device=""/>
-<part name="U$8" library="UNKNOWN-2024" deviceset="MOLEX-5-1.25" device=""/>
+<part name="LIDAR" library="UNKNOWN-2024" deviceset="MOLEX-4-1.25" device=""/>
+<part name="MOTOR_BOARD" library="UNKNOWN-2024" deviceset="MOLEX-5-1.25" device=""/>
 <part name="JP1" library="pinhead" library_urn="urn:adsk.eagle:library:325" deviceset="PINHD-1X2" device="" package3d_urn="urn:adsk.eagle:package:22435/2"/>
 <part name="JP3" library="pinhead" library_urn="urn:adsk.eagle:library:325" deviceset="PINHD-1X4" device="" package3d_urn="urn:adsk.eagle:package:22407/2"/>
@@
 <attribute name="VALUE" x="45.72" y="17.78" size="1.27" layer="96"/>
 </instance>
-<instance part="S1" gate="1" x="-5.08" y="99.06" smashed="yes" rot="R90">
+<instance part="POWER" gate="1" x="-5.08" y="99.06" smashed="yes" rot="R90">
 <attribute name="NAME" x="-3.175" y="92.71" size="1.778" layer="95" rot="R180"/>
 <attribute name="VALUE" x="-8.255" y="95.25" size="1.778" layer="96" rot="R180"/>
@@
 <attribute name="VALUE" x="-41.91" y="101.6" size="1.778" layer="96"/>
 </instance>
-<instance part="U$7" gate="G$1" x="251.46" y="40.64" smashed="yes">
+<instance part="LIDAR" gate="G$1" x="251.46" y="40.64" smashed="yes">
 <attribute name="NAME" x="245.11" y="46.355" size="1.778" layer="95"/>
 <attribute name="VALUE" x="247.65" y="30.48" size="1.778" layer="96"/>
 </instance>
-<instance part="U$8" gate="G$1" x="251.46" y="63.5" smashed="yes">
+<instance part="MOTOR_BOARD" gate="G$1" x="251.46" y="63.5" smashed="yes">
 <attribute name="NAME" x="245.11" y="71.755" size="1.778" layer="95"/>
 </instance>
@@
 <wire x1="248.92" y1="35.56" x2="233.68" y2="35.56" width="0.1524" layer="91"/>
 <label x="233.68" y="35.56" size="1.778" layer="95"/>
-<pinref part="U$7" gate="G$1" pin="4"/>
+<pinref part="LIDAR" gate="G$1" pin="4"/>
 </segment>
 <segment>
@@
 <wire x1="248.92" y1="58.42" x2="231.14" y2="58.42" width="0.1524" layer="91"/>
 <label x="231.14" y="58.42" size="1.778" layer="95"/>
-<pinref part="U$8" gate="G$1" pin="5"/>
+<pinref part="MOTOR_BOARD" gate="G$1" pin="5"/>
 </segment>
 </net>
@@
 <wire x1="248.92" y1="38.1" x2="233.68" y2="38.1" width="0.1524" layer="91"/>
 <label x="233.68" y="38.1" size="1.778" layer="95"/>
-<pinref part="U$7" gate="G$1" pin="3"/>
+<pinref part="LIDAR" gate="G$1" pin="3"/>
 </segment>
 <segment>
@@
 </segment>
 <segment>
-<pinref part="S1" gate="1" pin="P"/>
+<pinref part="POWER" gate="1" pin="P"/>
 <wire x1="0" y1="101.6" x2="10.16" y2="101.6" width="0.1524" layer="91"/>
 <label x="5.08" y="101.6" size="1.778" layer="95"/>
@@
 <wire x1="-10.16" y1="104.14" x2="-25.4" y2="104.14" width="0.1524" layer="91"/>
 <label x="-25.4" y="104.14" size="1.778" layer="95"/>
-<pinref part="S1" gate="1" pin="S"/>
+<pinref part="POWER" gate="1" pin="S"/>
 </segment>
 </net>
@@
 <wire x1="248.92" y1="60.96" x2="231.14" y2="60.96" width="0.1524" layer="91"/>
 <label x="231.14" y="60.96" size="1.778" layer="95"/>
-<pinref part="U$8" gate="G$1" pin="4"/>
+<pinref part="MOTOR_BOARD" gate="G$1" pin="4"/>
 </segment>
 </net>
@@
 <wire x1="248.92" y1="68.58" x2="231.14" y2="68.58" width="0.1524" layer="91"/>
 <label x="231.14" y="68.58" size="1.778" layer="95"/>
-<pinref part="U$8" gate="G$1" pin="1"/>
+<pinref part="MOTOR_BOARD" gate="G$1" pin="1"/>
 </segment>
 </net>
@@
 <wire x1="248.92" y1="40.64" x2="233.68" y2="40.64" width="0.1524" layer="91"/>
 <label x="233.68" y="40.64" size="1.778" layer="95"/>
-<pinref part="U$7" gate="G$1" pin="2"/>
+<pinref part="LIDAR" gate="G$1" pin="2"/>
 </segment>
 <segment>
@@
 <wire x1="248.92" y1="43.18" x2="233.68" y2="43.18" width="0.1524" layer="91"/>
 <label x="233.68" y="43.18" size="1.778" layer="95"/>
-<pinref part="U$7" gate="G$1" pin="1"/>
+<pinref part="LIDAR" gate="G$1" pin="1"/>
 </segment>
 <segment>
@@
 <wire x1="248.92" y1="66.04" x2="231.14" y2="66.04" width="0.1524" layer="91"/>
 <label x="231.14" y="66.04" size="1.778" layer="95"/>
-<pinref part="U$8" gate="G$1" pin="2"/>
+<pinref part="MOTOR_BOARD" gate="G$1" pin="2"/>
 </segment>
 </net>
@@
 <wire x1="248.92" y1="63.5" x2="231.14" y2="63.5" width="0.1524" layer="91"/>
 <label x="231.14" y="63.5" size="1.778" layer="95"/>
-<pinref part="U$8" gate="G$1" pin="3"/>
-</segment>
-</net>
+<pinref part="MOTOR_BOARD" gate="G$1" pin="3"/>
+</segment>
+</net>
