File: schematics/board/SP.brd (EAGLE design)
At the start: 30 x 46 mm, 20 parts

Commit message: Платы готовы
Parts:
- added D7: MBR0520LT, diode:SOD123
- added U$10, U$11, U$9: (no value), KNPN-2023:VIAS-CONNECT
- U$1, U$3, U$8: value SOLAR-2_1 -> SOLAR-2_INVERT0-2; device KNPN-2023:SOLAR_1-2 -> KNPN-2023:SOLAR_0-2_INVERT
- U$2, U$6: value SOLAR-2_0 -> SOLAR-2_INVERT1-2; device KNPN-2023:SOLAR_0-2 -> KNPN-2023:SOLAR_1-2_INVERT
- U$4: value SOLAR-2_0 -> SOLAR-2_INVERT0-2; device KNPN-2023:SOLAR_0-2 -> KNPN-2023:SOLAR_0-2_INVERT
- moved D5 76.3 mm to (37.6, 29.0), flipped to the bottom
- moved D6 60.3 mm to (37.6, 17.0), flipped to the bottom, turned to 180 degrees
- moved U$6 56.0 mm to (38.4, 32.5), turned to 90 degrees
- moved U$8 52.1 mm to (38.4, 13.5), turned to 270 degrees
- moved U$5 16.5 mm to (13.5, 5.50), flipped to the bottom
- moved FOTO 7.80 mm to (28.3, 2.50)
- moved JP1 7.80 mm to (22.8, 43.5)
- moved SP-OUT 7.80 mm to (22.8, 1.90)
- moved U$7 7.80 mm to (22.8, 4.20)
- moved C1 2.24 mm to (17.5, 35.7)
- moved PWR 2.24 mm to (21.1, 34.4)
- moved R1 2.06 mm to (21.1, 37.6)
- turned D1 to 0 degrees
- turned D2 to 180 degrees
- turned D3 to 180 degrees
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Connections:
- new net N$1: D7.A, JP1.2
- new net N$5: D1.C, D2.A, U$1.OUT-2, U$1.OUT-21, U$2.IN-2
- new net N$6: D3.A, D4.C, U$3.IN-2, U$4.OUT-2, U$4.OUT-21
- new net N$7: D1.A, U$1.IN-2, U$9.1
- net N$2: now also D5.A, U$11.1, U$6.IN-2; no longer D2.C, D3.A, U$2.OUT-2, U$2.OUT-21, U$3.IN-2
- net N$3: now also U$10.1; no longer D1.C, U$1.OUT
- net N$8: now also U$6.OUT; no longer U$6.OUT-2, U$6.OUT-21
- net SP+: now also D7.C, U$10.2, U$11.2, U$9.2; no longer D1.A, D2.A, D5.A, JP1.2, U$1.IN-2, U$2.IN-2, U$6.IN-2
- net SP+-: now also D2.C, U$2.OUT, U$3.OUT-2, U$3.OUT-21, U$8.OUT-2, U$8.OUT-21; no longer D4.C, U$3.OUT, U$4.OUT-2, U$4.OUT-21, U$8.OUT
Routing:
- net SP+-: track 43.5 -> 124.2 mm, vias 0 -> 2
- net N$6: track 0.00 -> 31.0 mm, vias 0 -> 1
- net N$5: track 0.00 -> 28.3 mm, vias 0 -> 1
- net SP-: track 43.1 -> 68.3 mm
- net N$8: track 0.00 -> 15.9 mm, vias 0 -> 1
- net N$2: track 23.3 -> 7.82 mm
- net N$3: track 15.1 -> 7.68 mm
- net N$7: track 0.00 -> 7.36 mm, vias 0 -> 1
- net N$1: track 0.00 -> 3.55 mm
- net SP+: track 43.5 -> 44.6 mm, vias 2 -> 0
- net N$4: track 2.78 -> 3.28 mm
Other:
- board size 30 x 46 mm -> 45.6 x 46 mm
- board text added: "0V"
- board text removed: "1.5V"
- board text removed: "2V"
