File: schematics/board/MOTOR.brd (EAGLE design)
At the start: 76 x 76 mm, 77 parts

Commit message: сч мипэхъ\
Parts:
- removed MOTOR0: (no value), pinhead:1X02
- added U$10: MOLEX-2-1.25, UNKNOWN-2024:53047-02
- U$9: value Плата МОТОРЫ -> Плата МОТОРОВ
- moved SI2302CDS10 150.9 mm to (67.6, 53.3)
- moved R16 138.5 mm to (62.3, 61.2)
- moved R15 129.6 mm to (58.4, 56.7)
- moved JP13 128.2 mm to (71.4, 32.4)
- moved JP15 127.7 mm to (58.0, 9.58), turned to 45 degrees
- moved U$6 127.2 mm to (67.1, 44.7), flipped to the bottom, turned to 257 degrees
- moved U$7 126.4 mm to (63.3, 22.2), flipped to the bottom, turned to 302 degrees
- moved JP14 124.5 mm to (69.2, 27.0)
- moved U$13 123.9 mm to (82.0, 79.0)
- moved JP16 122.2 mm to (52.1, 6.43), turned to 13 degrees
- moved R20 120.8 mm to (62.6, 17.3), flipped to the bottom, turned to 270 degrees
- moved JP18 116.9 mm to (44.9, 64.0)
- moved U$8 116.7 mm to (30.7, 66.9), flipped to the bottom, turned to 167 degrees
- moved U$5 115.1 mm to (53.8, 63.3), flipped to the bottom, turned to 212 degrees
- moved JP17 115.0 mm to (46.7, 71.4)
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Connections:
- net LATCH renamed LATCH_SR
- net SCK renamed SCK_SENS
- removed net MOSI: JP6.2, U$13.14
- removed net OE: JP6.5
- removed net SHIFT2: JP6.6, U$13.9
- new net MOSI_SENS: JP6.2
- new net SHIFT: JP6.6, U$13.14
- net N$1: now also U$10.2; no longer MOTOR0.2
- net N$6: now also U$10.1; no longer MOTOR0.1
- net OE_SR: now also JP6.5
Routing:
- net N$31: track 0.00 -> 25.7 mm
- net N$16: track 0.00 -> 19.1 mm
- net N$18: track 0.00 -> 15.3 mm
- net N$32: track 0.00 -> 13.7 mm
- net N$19: track 0.00 -> 11.1 mm
- net N$33: track 0.00 -> 10.6 mm
- net N$17: track 0.00 -> 9.30 mm
- net N$35: track 0.00 -> 4.87 mm
- net N$34: track 0.00 -> 2.53 mm
- net N$20: track 0.00 -> 1.15 mm

Commit message: Моторчики
Parts:
- removed JP6: (no value), pinhead:1X06
- added JP19: (no value), pinhead:1X05
- moved R14 104.0 mm to (27.0, 15.7)
- moved JP5 101.2 mm to (65.8, 20.9), turned to 225 degrees
- moved R1 98.3 mm to (13.4, 12.9), flipped to the bottom
- moved MOTOR4 98.2 mm to (61.2, 49.2), turned to 103 degrees
- moved SI2302CDS6 97.1 mm to (16.6, 61.8), flipped to the bottom
- moved SI2302CDS16 90.7 mm to (42.4, 66.7), flipped to the bottom, turned to 180 degrees
- moved SI2302CDS5 89.3 mm to (13.0, 61.8), flipped to the bottom
- moved SI2302CDS9 88.5 mm to (58.6, 61.0), flipped to the bottom, turned to 180 degrees
- moved SI2302CDS15 84.5 mm to (39.5, 67.7), flipped to the bottom, turned to 180 degrees
- moved MOTOR1 82.3 mm to (13.7, 46.2), turned to 238 degrees
- moved R3 81.8 mm to (10.8, 21.9), flipped to the bottom, turned to 90 degrees
- moved U$13 81.4 mm to (38.0, 10.5), turned to 180 degrees
- moved SI2302CDS12 81.3 mm to (65.8, 27.7), flipped to the bottom, turned to 180 degrees
- moved R2 81.3 mm to (13.6, 19.3), flipped to the bottom
- moved JP2 80.4 mm to (6.88, 23.7), turned to 283 degrees
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Connections:
- removed net MOSI_SENS: JP6.2
- net 3V3: now also JP19.1; no longer JP6.1
- net LATCH_SR: now also JP19.3; no longer JP6.4
- net OE_SR: now also JP19.4; no longer JP6.5
- net SCK_SENS: now also JP19.2; no longer JP6.3
- net SHIFT: now also JP19.5; no longer JP6.6
Routing:
- net GND: track 0.00 -> 283.9 mm, vias 0 -> 11
- net 16V: track 0.00 -> 248.8 mm, vias 0 -> 4
- net MOTOR7: track 0.00 -> 112.8 mm, vias 0 -> 7
- net MOTOR2: track 0.00 -> 96.7 mm, vias 0 -> 5
- net MOTOR4: track 0.00 -> 87.4 mm, vias 0 -> 3
- net MOTOR5: track 0.00 -> 59.3 mm, vias 0 -> 5
- net MOTOR1: track 0.00 -> 51.3 mm, vias 0 -> 3
- net 3V3: track 0.00 -> 30.1 mm
- net MOTOR6: track 0.00 -> 27.5 mm, vias 0 -> 5
- net MOTOR0: track 0.00 -> 25.1 mm, vias 0 -> 5
- net N$14: track 0.00 -> 23.4 mm
- net N$39: track 0.00 -> 23.1 mm
- net N$7: track 0.00 -> 22.8 mm
- net OE_SR: track 0.00 -> 20.3 mm, vias 0 -> 1
- net N$1: track 0.00 -> 19.8 mm
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
Commit message: Платы готовы
Parts:
- removed JP1, JP11, JP13, JP15, JP17, JP3, JP5, JP7, JP9, MOTOR1, MOTOR2, MOTOR3, MOTOR4, MOTOR5, MOTOR6, MOTOR7: (no value), pinhead:1X02
- removed JP10, JP12, JP14, JP16, JP18, JP2, JP4, JP8: (no value), pinhead:1X03
- removed JP19: (no value), pinhead:1X05
- removed SI2302CDS1, SI2302CDS10, SI2302CDS11, SI2302CDS12, SI2302CDS13, SI2302CDS14, SI2302CDS15, SI2302CDS16, SI2302CDS2, SI2302CDS3, SI2302CDS4, SI2302CDS5, SI2302CDS6, SI2302CDS7, SI2302CDS8, SI2302CDS9: SI2302CDS, CanCubeSat:SOT23-3
- removed U$1, U$2, U$3, U$4, U$6, U$7, U$8: CONCEVIC, CanCubeSat:CONCEVIC
- removed U$13: 74HC595, CanCubeSat:TSSOP16
- added 16V, GND: (no value), pinhead:1X02/90
- added 74HC595: 74HC595, CanCubeSat:TSSOP16
- added BUT0, BUT1, BUT2, BUT3, BUT4, BUT5, BUT6, BUT7: (no value), pinheadCS:1X02
- added END0, END1, END2, END3, END4, END5, END6, END7: CONCEVIC, CanCubeSat:CONCEVIC
- added MOT0, MOT1, MOT2, MOT3, MOT4, MOT5, MOT6, MOT7, PWR_16V: JST-2-2.5, UNKNOWN-2024:JST-2-2.5
- added RADIO: MOLEX-5-1.25, UNKNOWN-2024:53047-05
- added U$11, U$15, U$16, U$20, U$28, U$32: IRF5852, NA-2025:TSOP-6
- added U$35, U$36, U$37, U$38, U$39, U$40, U$41, U$42: CONTACT_SIDE_4MM_2PIN, UNKNOWN-2024:CONTACT_SIDE_4MM_2PIN
- U$10: value MOLEX-2-1.25 -> IRF5852; device UNKNOWN-2024:53047-02 -> NA-2025:TSOP-6
- U$5: value CONCEVIC -> IRF5852; device CanCubeSat:CONCEVIC -> NA-2025:TSOP-6
- U$9: value Плата МОТОРОВ -> Плата Моторов
- moved R23 55.8 mm to (63.2, 23.7), flipped to the top, turned to 225 degrees
- moved R11 54.4 mm to (15.1, 57.7), flipped to the top, turned to 225 degrees
- moved R24 54.0 mm to (64.7, 22.2), flipped to the top, turned to 45 degrees
- moved R10 49.8 mm to (16.6, 56.2), flipped to the top, turned to 45 degrees
- moved R12 49.3 mm to (11.6, 52.3), flipped to the top, turned to 135 degrees
- moved R6 47.1 mm to (33.5, 5.69), flipped to the top, turned to 225 degrees
- moved R25 46.9 mm to (68.5, 27.7), flipped to the top, turned to 315 degrees
- moved U$9 44.7 mm to (5.32, 45.7)
- moved R22 44.0 mm to (68.9, 51.4), flipped to the top
- moved R3 41.9 mm to (51.3, 11.2), flipped to the top
- moved U$5 41.2 mm to (13.6, 54.5), flipped to the top, turned to 45 degrees
- moved R19 40.5 mm to (52.4, 68.4), flipped to the top, turned to 45 degrees
- moved R9 36.3 mm to (11.1, 28.5), flipped to the top, turned to 180 degrees
- moved R5 34.7 mm to (28.1, 9.50), flipped to the top, turned to 315 degrees
- moved R16 33.0 mm to (28.5, 69.0), flipped to the top, turned to 90 degrees
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Connections:
- removed net 16V: JP1.2, JP10.3, JP11.2, JP12.3, JP13.2, JP14.3, JP15.2, JP16.3, JP17.2, JP18.3, JP2.3, JP3.2, JP4.3, JP5.1, JP7.2, JP8.3, JP9.2, R12.1, R16.1, R19.1, R22.1, R25.1, R3.1, R6.1, R9.1
- removed net GND: JP5.2, R11.2, R14.1, R15.2, R18.2, R2.2, R21.2, R24.2, R5.2, R8.2, SI2302CDS1.2, SI2302CDS10.2, SI2302CDS11.2, SI2302CDS12.2, SI2302CDS13.2, SI2302CDS14.2, SI2302CDS15.2, SI2302CDS16.2, SI2302CDS2.2, SI2302CDS3.2, SI2302CDS4.2, SI2302CDS5.2, SI2302CDS6.2, SI2302CDS7.2, SI2302CDS8.2, SI2302CDS9.2, U$1.P$1, U$13.8, U$2.P$1, U$3.P$1, U$4.P$1, U$5.P$1, U$6.P$1, U$7.P$1, U$8.P$1
- removed net N$33: JP16.2, MOTOR6.1
- removed net N$34: JP16.1, SI2302CDS14.3
- removed net N$35: R22.2, SI2302CDS14.1
- removed net N$36: JP17.1, MOTOR7.2, SI2302CDS15.3
- removed net N$37: R23.2, R24.1, SI2302CDS15.1, U$8.P$2
- removed net N$38: JP18.2, MOTOR7.1
- removed net N$39: JP18.1, SI2302CDS16.3
- removed net N$40: R25.2, SI2302CDS16.1
- new net 16V_IN: 16V.1, MOT0.1, MOT1.1, MOT2.1, MOT3.1, MOT4.1, MOT5.1, MOT6.1, MOT7.1, U$10.P$6, U$11.P$6, U$15.P$6, U$16.P$6, U$20.P$6, U$28.P$6, U$32.P$6, U$5.P$6
- new net 16V_OUT: 16V.2, PWR_16V.1
- new net GND_IN: END0.P$1, END1.P$1, END2.P$1, END3.P$1, END4.P$1, END5.P$1, END6.P$1, END7.P$1, GND.1, R11.2, R15.2, R18.2, R2.2, R21.2, R24.2, R5.2, R8.2, U$10.P$2, U$11.P$2, U$15.P$2, U$16.P$2, U$20.P$2, U$28.P$2, U$32.P$2, U$5.P$2
- new net GND_OUT: 74HC595.8, GND.2, PWR_16V.2, R14.1
- net 3V3: now also 74HC595.10, 74HC595.16, RADIO.1; no longer JP19.1, U$13.10, U$13.16
- net LATCH_SR: now also 74HC595.12, RADIO.3; no longer JP19.3, U$13.12
- net MOTOR0: now also 74HC595.7; no longer U$13.15
- net MOTOR1: now also 74HC595.1; no longer U$13.1
- net MOTOR2: now also 74HC595.2; no longer U$13.2
- net MOTOR3: now also 74HC595.3; no longer U$13.3
- net MOTOR4: now also 74HC595.15; no longer U$13.4
- net MOTOR5: now also 74HC595.4; no longer U$13.5
- net MOTOR6: now also 74HC595.5; no longer U$13.6
- net MOTOR7: now also 74HC595.6; no longer U$13.7
- net N$1: now also MOT0.2, R3.1, U$11.P$4, U$38.P$1; no longer JP1.1, SI2302CDS1.3, U$10.2
- net N$10: now also BUT2.2, U$16.P$5, U$36.P$2; no longer R6.2, SI2302CDS4.1
- net N$11: now also END3.P$2, R10.2, R11.1, U$5.P$3; no longer JP7.1, MOTOR2.2, SI2302CDS5.3
- net N$12: now also END2.P$2, U$16.P$3; no longer SI2302CDS5.1, U$3.P$2
- net N$13: now also BUT2.1, R9.1, U$16.P$1; no longer JP8.2, MOTOR2.1
- net N$14: now also MOT3.2, R12.2, U$37.P$1, U$5.P$4; no longer JP8.1, SI2302CDS6.3
- net N$15: now also BUT3.2, U$37.P$2, U$5.P$5; no longer R9.2, SI2302CDS6.1
- net N$16: now also BUT3.1, R12.1, U$5.P$1; no longer JP9.1, MOTOR3.2, SI2302CDS7.3
- net N$17: now also END4.P$2, R13.2, R15.1, U$15.P$3; no longer R10.2, R11.1, SI2302CDS7.1, U$4.P$2
- net N$18: now also MOT4.2, R16.2, U$15.P$4, U$39.P$1; no longer JP10.2, MOTOR3.1
- net N$19: now also BUT4.2, U$15.P$5, U$39.P$2; no longer JP10.1, SI2302CDS8.3
- net N$2: now also MOT1.2, R6.2, U$10.P$4, U$35.P$1; no longer JP3.1, MOTOR1.2, SI2302CDS3.3
- net N$20: now also BUT4.1, R16.1, U$15.P$1; no longer R12.2, SI2302CDS8.1
- net N$21: now also END5.P$2, R17.2, R18.1, U$20.P$3; no longer JP11.1, MOTOR4.2, SI2302CDS9.3
- net N$22: now also MOT5.2, R19.2, U$20.P$4, U$40.P$1; no longer R13.2, R15.1, SI2302CDS9.1, U$5.P$2
- net N$23: now also BUT5.2, U$20.P$5, U$40.P$2; no longer JP12.2, MOTOR4.1
- net N$24: now also BUT5.1, R19.1, U$20.P$1; no longer JP12.1, SI2302CDS10.3
- net N$25: now also END6.P$2, R20.2, R21.1, U$28.P$3; no longer R16.2, SI2302CDS10.1
- net N$26: now also MOT6.2, R22.2, U$28.P$4, U$41.P$1; no longer JP13.1, MOTOR5.2, SI2302CDS11.3
- net N$27: now also BUT6.2, U$28.P$5, U$41.P$2; no longer R17.2, R18.1, SI2302CDS11.1, U$6.P$2
- net N$28: now also BUT6.1, R22.1, U$28.P$1; no longer JP14.2, MOTOR5.1
- net N$29: now also END7.P$2, R23.2, R24.1, U$32.P$3; no longer JP14.1, SI2302CDS12.3
- net N$3: now also END1.P$2, U$10.P$3; no longer SI2302CDS3.1, U$2.P$2
- net N$30: now also MOT7.2, R25.2, U$32.P$4, U$42.P$1; no longer R19.2, SI2302CDS12.1
- net N$31: now also BUT7.2, U$32.P$5, U$42.P$2; no longer JP15.1, MOTOR6.2, SI2302CDS13.3
- net N$32: now also BUT7.1, R25.1, U$32.P$1; no longer R20.2, R21.1, SI2302CDS13.1, U$7.P$2
- net N$4: now also END0.P$2, U$11.P$3; no longer SI2302CDS1.1, U$1.P$2
- net N$5: now also BUT1.2, U$10.P$5, U$35.P$2; no longer JP4.2, MOTOR1.1
- net N$6: now also BUT0.1, R3.2, U$11.P$1; no longer JP2.2, U$10.1
- net N$7: now also BUT1.1, R6.1, U$10.P$1; no longer JP4.1, SI2302CDS4.3
- net N$8: now also BUT0.2, U$11.P$5, U$38.P$2; no longer JP2.1, SI2302CDS2.3
- net N$9: now also MOT2.2, R9.2, U$16.P$4, U$36.P$1; no longer R3.2, SI2302CDS2.1
- net OE_SR: now also 74HC595.13, RADIO.4; no longer JP19.4, U$13.13
- net SCK_SENS: now also 74HC595.11, RADIO.2; no longer JP19.2, U$13.11
- net SHIFT: now also 74HC595.14, RADIO.5; no longer JP19.5, U$13.14
Routing:
- net GND: track 283.9 -> 0.00 mm, vias 11 -> 0
- net 16V: track 248.8 -> 0.00 mm, vias 4 -> 0
- net 16V_IN: track 0.00 -> 240.4 mm
- net GND_IN: track 0.00 -> 237.3 mm, vias 0 -> 39
- net GND_OUT: track 0.00 -> 87.3 mm, vias 0 -> 2
- net MOTOR7: track 112.8 -> 40.7 mm, vias 7 -> 0
- net MOTOR2: track 96.7 -> 28.4 mm, vias 5 -> 0
- net MOTOR3: track 4.48 -> 49.9 mm, vias 1 -> 0
- net MOTOR1: track 51.3 -> 6.82 mm, vias 3 -> 0
- net MOTOR6: track 27.5 -> 70.0 mm, vias 5 -> 0
- net MOTOR5: track 59.3 -> 92.1 mm, vias 5 -> 0
- net N$10: track 1.53 -> 26.6 mm
- net N$39: track 23.1 -> 0.00 mm
- net N$20: track 1.15 -> 22.2 mm, vias 0 -> 1
- net N$30: track 2.93 -> 21.8 mm
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- added copper zone on layer 1, net GND_IN
- added copper zone on layer 16, net GND_IN
Other:
- outline, holes or cut-outs redrawn
- board text added: "PWR_16V"
