File: schematics/board/MK.sch (EAGLE design)
At the start: 57 parts

Commit message: фцыувкаепнргошщз
Parts:
- renumbered PERE1 to PERE_L, PERE2 to PERE_SP, SI2302CDS to SI2302
Changed lines of the file:
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@@
 <?xml version="1.0" encoding="utf-8"?>
 <!DOCTYPE eagle SYSTEM "eagle.dtd">
-<eagle version="9.4.2">
+<eagle version="9.6.2">
 <drawing>
 <settings>
-<setting alwaysvectorfont="yes"/>
+<setting alwaysvectorfont="no"/>
 <setting verticaltext="up"/>
 </settings>
@@
 <part name="MICRO_SD" library="UNKNOWN-2024" deviceset="SD" device=""/>
 <part name="BUZZER" library="CanCubeSat" deviceset="BUZZER" device="S8R6"/>
-<part name="SI2302CDS" library="CanCubeSat" deviceset="SI2302CDS" device=""/>
+<part name="SI2302" library="CanCubeSat" deviceset="SI2302CDS" device=""/>
 <part name="R9" library="rcl" library_urn="urn:adsk.eagle:library:334" deviceset="R-US_" device="R0603" package3d_urn="urn:adsk.eagle:package:23555/3" value="10k"/>
 <part name="R10" library="rcl" library_urn="urn:adsk.eagle:library:334" deviceset="R-US_" device="R0603" package3d_urn="urn:adsk.eagle:package:23555/3" value="100R"/>
@@
 <part name="R20" library="rcl" library_urn="urn:adsk.eagle:library:334" deviceset="R-US_" device="R2512" package3d_urn="urn:adsk.eagle:package:23545/2" value="R05"/>
 <part name="U$17" library="UNKNOWN-2024" deviceset="IRF7905PBF" device=""/>
-<part name="PERE1" library="UNKNOWN-2024" deviceset="JST-2-2.5" device=""/>
+<part name="PERE_L" library="UNKNOWN-2024" deviceset="JST-2-2.5" device=""/>
 <part name="R22" library="rcl" library_urn="urn:adsk.eagle:library:334" deviceset="R-US_" device="R0603" package3d_urn="urn:adsk.eagle:package:23555/3" value="5k1"/>
 <part name="R23" library="rcl" library_urn="urn:adsk.eagle:library:334" deviceset="R-US_" device="R0603" package3d_urn="urn:adsk.eagle:package:23555/3" value="5k1"/>
-<part name="PERE2" library="UNKNOWN-2024" deviceset="JST-2-2.5" device=""/>
+<part name="PERE_SP" library="UNKNOWN-2024" deviceset="JST-2-2.5" device=""/>
 <part name="R24" library="rcl" library_urn="urn:adsk.eagle:library:334" deviceset="R-US_" device="R0603" package3d_urn="urn:adsk.eagle:package:23555/3" value="5k1"/>
 <part name="R25" library="rcl" library_urn="urn:adsk.eagle:library:334" deviceset="R-US_" device="R0603" package3d_urn="urn:adsk.eagle:package:23555/3" value="5k1"/>
@@
 <attribute name="NAME" x="68.58" y="-48.26" size="2.54" layer="95"/>
 </instance>
-<instance part="SI2302CDS" gate="G$1" x="109.22" y="-53.34" smashed="yes" rot="R180"/>
+<instance part="SI2302" gate="G$1" x="109.22" y="-53.34" smashed="yes" rot="R180"/>
 <instance part="R9" gate="G$1" x="119.38" y="-58.42" smashed="yes" rot="R90">
 <attribute name="NAME" x="117.8814" y="-62.23" size="1.778" layer="95" rot="R90"/>
@@
 <attribute name="NAME" x="106.68" y="1.27" size="1.778" layer="95" rot="R270"/>
 </instance>
-<instance part="PERE1" gate="G$1" x="62.23" y="-21.59" smashed="yes">
+<instance part="PERE_L" gate="G$1" x="62.23" y="-21.59" smashed="yes">
 <attribute name="VALUE" x="60.96" y="-29.21" size="1.778" layer="96"/>
 <attribute name="NAME" x="60.96" y="-18.288" size="1.778" layer="95"/>
@@
 <attribute name="VALUE" x="89.662" y="6.35" size="1.778" layer="96" rot="R90"/>
 </instance>
-<instance part="PERE2" gate="G$1" x="104.14" y="-21.59" smashed="yes">
+<instance part="PERE_SP" gate="G$1" x="104.14" y="-21.59" smashed="yes">
 <attribute name="VALUE" x="102.87" y="-29.21" size="1.778" layer="96"/>
 <attribute name="NAME" x="102.87" y="-18.288" size="1.778" layer="95"/>
@@
 <net name="GND" class="0">
 <segment>
-<pinref part="SI2302CDS" gate="G$1" pin="S"/>
+<pinref part="SI2302" gate="G$1" pin="S"/>
 <wire x1="119.38" y1="-53.34" x2="129.54" y2="-53.34" width="0.1524" layer="91"/>
 <label x="124.46" y="-53.34" size="1.778" layer="95"/>
@@
 <net name="N$13" class="0">
 <segment>
-<pinref part="SI2302CDS" gate="G$1" pin="D"/>
+<pinref part="SI2302" gate="G$1" pin="D"/>
 <wire x1="99.06" y1="-53.34" x2="88.9" y2="-53.34" width="0.1524" layer="91"/>
 <pinref part="BUZZER" gate="G$1" pin="GND"/>
@@
 <net name="N$14" class="0">
 <segment>
-<pinref part="SI2302CDS" gate="G$1" pin="G"/>
+<pinref part="SI2302" gate="G$1" pin="G"/>
 <wire x1="109.22" y1="-60.96" x2="109.22" y2="-63.5" width="0.1524" layer="91"/>
 <pinref part="R10" gate="G$1" pin="2"/>
@@
 <wire x1="93.98" y1="-12.7" x2="93.98" y2="-21.59" width="0.1524" layer="91"/>
 <wire x1="93.98" y1="-21.59" x2="69.85" y2="-21.59" width="0.1524" layer="91"/>
-<pinref part="PERE1" gate="G$1" pin="2"/>
+<pinref part="PERE_L" gate="G$1" pin="2"/>
 </segment>
 </net>
@@
 <segment>
 <pinref part="U$17" gate="G$1" pin="D1"/>
-<pinref part="PERE2" gate="G$1" pin="2"/>
+<pinref part="PERE_SP" gate="G$1" pin="2"/>
 <wire x1="111.76" y1="-12.7" x2="111.76" y2="-21.59" width="0.1524" layer="91"/>
 </segment>
@@
 <net name="4V" class="0">
 <segment>
-<pinref part="PERE2" gate="G$1" pin="1"/>
+<pinref part="PERE_SP" gate="G$1" pin="1"/>
 <wire x1="111.76" y1="-24.13" x2="121.92" y2="-24.13" width="0.1524" layer="91"/>
 <label x="118.11" y="-24.13" size="1.778" layer="95"/>
 </segment>
 <segment>
-<pinref part="PERE1" gate="G$1" pin="1"/>
+<pinref part="PERE_L" gate="G$1" pin="1"/>
 <wire x1="69.85" y1="-24.13" x2="80.01" y2="-24.13" width="0.1524" layer="91"/>
 <label x="76.2" y="-24.13" size="1.778" layer="95"/>

Commit message: проверка плат
Parts:
- removed R1: 2k, rcl:R-US_R0603
- R18, R19: value 5k1 -> 10R
- R22, R24, R26, R27, R28, R29, R32, R33, R34, R35: value 5k1 -> 10k
- R23, R25, R30, R31, R36, R37: value 5k1 -> 100R
Connections:
- removed net N$1: R1.1, U$2.S
- net GND: now also R28.1, R29.1, R34.1, R35.1, U$2.S; no longer R1.2
- net N$24: no longer R34.1
- net N$25: no longer R28.1
- net N$26: no longer R29.1
- net N$27: no longer R35.1

Commit message: Платы готовы
Parts:
- AP9930_: value MOSFET_2P+2N_AP9930GM -> AP9930GM
- R21: value (none) -> 100R
- renumbered U$13 to 74HC595, U$15 to AP9930_, U$16 to INA, U$17 to IRF7905, U$21 to AP9930, U$22 to NDC7002_, U$23 to NDC7002

Commit message: СД в центре лепестка. Платы версия 2
Parts:
- removed AP9930: MOSFET_2P+2N_AP9930GM, UNKNOWN-2024:MOSFET_2P+2N_AP9930GM
- removed AP9930_: AP9930GM, UNKNOWN-2024:MOSFET_2P+2N_AP9930GM
- added U$3, U$4, U$5, U$6: FDC6420C, KNPN-2023:FDC6420C
Connections:
- net 5V: now also U$3.PS, U$4.PS, U$5.PS, U$6.PS; no longer AP9930.P1P2S, AP9930_.P1P2S
- net GND: now also U$3.NS, U$4.NS, U$5.NS, U$6.NS; no longer AP9930.N1N2S, AP9930_.N1N2S
- net MOTOR1+: now also U$6.ND, U$6.PD; no longer AP9930.P2N2D
- net MOTOR1-: now also U$5.ND, U$5.PD; no longer AP9930.P1N1D
- net MOTOR2+: now also U$4.ND, U$4.PD; no longer AP9930_.P2N2D
- net MOTOR2-: now also U$3.ND, U$3.PD; no longer AP9930_.P1N1D
- net N$24: now also U$5.NG, U$5.PG; no longer AP9930.N1G, AP9930.P1G
- net N$25: now also U$3.NG, U$3.PG; no longer AP9930_.N1G, AP9930_.P1G
- net N$26: now also U$4.NG, U$4.PG; no longer AP9930_.N2G, AP9930_.P2G
- net N$27: now also U$6.NG, U$6.PG; no longer AP9930.N2G, AP9930.P2G
Other:
- moved on the sheet: NDC7002, NDC7002_, R26, R27, R28, R29, R30, R31, R32, R33, R34, R35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
