File: schematics/board/old/GERMO.brd (EAGLE design)
At the start: 72.1 x 32 mm, 35 parts

Commit message: Поправлены платы МК, Радио, Гермо
Parts:
- removed C2, C3, C4: 100nF, rcl:C0603
- removed JP2: (no value), pinhead:1X02
- removed R16, R2: 5k1, rcl:R0603
- removed U$14: AD5593, UNKNOWN-2024:AD5593
- added JP3: (no value), pinhead:1X04
- moved U$2 24.3 mm to (32.7, 45.0)
- moved R17 9.00 mm to (25.9, 24.6)
- moved U$6 5.52 mm to (58.6, 27.6)
- moved R40 5.50 mm to (59.5, 30.4), turned to 0 degrees
- moved U$5 5.14 mm to (57.5, 25.1)
- moved R39 5.01 mm to (56.7, 27.8)
- moved R44 4.84 mm to (53.5, 30.5), turned to 0 degrees
- moved R8 4.60 mm to (57.5, 22.8), turned to 270 degrees
- moved R46 4.04 mm to (36.4, 28.0), turned to 0 degrees
- moved R42 2.57 mm to (49.4, 30.4), turned to 0 degrees
- moved U$10 1.72 mm to (54.7, 27.5)
- moved R43 1.71 mm to (52.5, 27.9)
- moved U$9 1.60 mm to (53.5, 25.1)
- moved R12 1.60 mm to (53.5, 22.8)
- moved U$12 1.03 mm to (37.7, 25.2)
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Connections:
- removed net FOTO0: JP2.2, U$14.P$5
- removed net FOTO1: JP2.1, U$14.P$4
- removed net N$18: C2.1, U$14.P$8
- removed net N$19: R16.1, U$14.P$2
- removed net N$20: R2.1, U$14.P$1
- net 3V3: no longer C3.1, C4.1, R2.2, U$14.P$3, U$14.P$9
- net CO: now also JP3.1; no longer U$14.P$7
- net GND: no longer C2.2, C3.2, C4.2, R16.2, U$14.P$14
- net MICS: now also JP3.4; no longer U$14.P$11
- net NH3: now also JP3.3; no longer U$14.P$6
- net NO2: now also JP3.2; no longer U$14.P$10
- net SCL: no longer U$14.P$16
- net SDA: no longer U$14.P$15
Routing:
- net GND: track 130.2 -> 67.9 mm
- net 3V3: track 118.0 -> 60.9 mm
- net NO2: track 9.75 -> 41.6 mm
- net SCL: track 70.8 -> 49.3 mm
- net NH3: track 7.71 -> 24.4 mm
- net FOTO0: track 13.1 -> 0.00 mm
- net EN: track 2.50 -> 14.2 mm
- net FOTO1: track 10.2 -> 0.00 mm
- net MICS: track 16.4 -> 24.9 mm
- net SDA: track 55.5 -> 49.8 mm
- net CO: track 13.8 -> 17.6 mm
- net 5V: track 87.2 -> 90.2 mm
- net N$19: track 2.64 -> 0.00 mm
- net N$18: track 2.48 -> 0.00 mm
- net N$20: track 1.55 -> 0.00 mm
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- removed copper zone on layer 1, net GND
- removed copper zone on layer 16, net GND
