File: schematics/board/old/GERMO.sch (EAGLE design)
At the start: 35 parts

Commit message: Поправлены платы МК, Радио, Гермо
Parts:
- removed C2, C3, C4: 100nF, rcl:C-EUC0603
- removed JP2: (no value), pinhead:PINHD-1X2
- removed R16, R2: 5k1, rcl:R-US_R0603
- removed U$14: AD5593, UNKNOWN-2024:AD5593
- added JP3: (no value), pinhead:PINHD-1X4
Connections:
- removed net FOTO0: JP2.2, U$14.IO1
- removed net FOTO1: JP2.1, U$14.IO0
- removed net N$18: C2.1, U$14.VREF
- removed net N$19: R16.1, U$14.AO
- removed net N$20: R2.1, U$14.RESET
- net 3V3: no longer C3.1, C4.1, R2.2, U$14.VDD, U$14.VDDL
- net CO: now also JP3.1; no longer U$14.IO3
- net GND: no longer C2.2, C3.2, C4.2, R16.2, U$14.GND
- net MICS: now also JP3.4; no longer U$14.IO5
- net NH3: now also JP3.3; no longer U$14.IO2
- net NO2: now also JP3.2; no longer U$14.IO4
- net SCL: no longer U$14.SCL
- net SDA: no longer U$14.SDA
