File: schematics/board/old/MK.sch (EAGLE design)
At the start: 57 parts

Commit message: Поправлены платы МК, Радио, Гермо
Parts:
- added C2, C3, C4: 100nF, rcl:C-EUC0603
- added R16, R17: 5k1, rcl:R-US_R0603
- added U$14: AD5593, UNKNOWN-2024:AD5593
- JP3: device pinhead:PINHD-1X14 -> pinhead:PINHD-1X16
Connections:
- removed net FOTO1: JP3.13, R0.2, U$0.1
- new net C0: JP3.13
- new net CO: U$14.IO2
- new net MICS: JP3.16, U$14.IO5
- new net N$11: C2.1, U$14.VREF
- new net N$16: C3.1, C4.1, U$14.VDD, U$14.VDDL
- new net N$17: R16.1, U$14.AO
- new net N$19: R17.1, U$14.RESET
- new net N$4: R0.2, U$0.1, U$14.IO0
- new net NH3: JP3.15, U$14.IO4
- new net NO2: JP3.14, U$14.IO3
- net 3V3: now also R17.2, U$16.SCL; no longer U$16.VS
- net FOTO0: now also U$14.IO1; no longer JP3.14
- net GND: now also C2.2, C3.2, C4.2, R16.2, U$14.GND, U$16.IN+, U$16.IN-, U$16.SDA; no longer U$16.A0, U$16.A1, U$16.GND
- net MK_MOTOR2+: now also U$13.Q2; no longer U$13.Q6
- net MK_MOTOR2-: now also U$13.Q3; no longer U$13.Q7
- net N$15: now also U$16.A0; no longer U$16.IN-
- net N$18: now also U$16.A1; no longer U$16.IN+
- net PERE1: now also U$13.Q6; no longer U$13.Q3
- net PERE2: now also U$13.Q7; no longer U$13.Q2
- net SCL: now also U$14.SCL, U$16.VS; no longer U$16.SCL
- net SDA: now also U$14.SDA, U$16.GND; no longer U$16.SDA
Other:
- moved on the sheet: FOTO0
