File: schematics/board/old/RADIO.brd (EAGLE design)
At the start: 76 x 76 mm, 49 parts, among them X2 AKKUM

Commit message: Поправлены платы МК, Радио, Гермо
Parts:
- moved JP3 3.61 mm to (40.0, 19.5)
- moved JP1 3.35 mm to (60.0, 19.5)
- moved R8 0.10 mm to (71.0, 52.2)
Connections:
- removed net C0: JP4.13
- net CO: now also JP4.13
Routing:
- net N$5: track 18.3 -> 26.1 mm
- net N$10: track 21.0 -> 27.1 mm, vias 0 -> 4
- net NO2: track 30.9 -> 27.7 mm
- net NH3: track 29.8 -> 26.7 mm
- net MICS: track 25.3 -> 22.2 mm
- net SDA: track 82.2 -> 79.4 mm
- net 5V: track 189.8 -> 192.0 mm
- net BUS+: track 66.9 -> 65.1 mm
- net N$9: track 31.5 -> 30.2 mm
- net OE_SR: track 38.5 -> 39.8 mm
- net N$17: track 61.2 -> 62.2 mm
- net N$13: track 56.6 -> 57.6 mm, vias 5 -> 4
- net N$18: track 41.0 -> 41.9 mm
- net CS_LSM: track 51.5 -> 52.3 mm
- net GND: track 347.1 -> 347.8 mm
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