File: schematics/board/old/RADIO.sch (EAGLE design)
At the start: 48 parts, among them X2 AKKUM

Commit message: Поправлены платы МК, Радио, Гермо
Parts:
- removed JP2: (no value), pinhead:PINHD-1X8
- added JP1, JP3: (no value), pinhead:PINHD-1X4
Connections:
- removed net C0: JP4.13
- net 5V: now also JP3.2; no longer JP2.6
- net CO: now also JP1.1, JP4.13; no longer JP2.1
- net GND: now also JP3.1; no longer JP2.5
- net MICS: now also JP1.4; no longer JP2.4
- net NH3: now also JP1.3; no longer JP2.3
- net NO2: now also JP1.2; no longer JP2.2
- net SCL: now also JP3.4; no longer JP2.8
- net SDA: now also JP3.3; no longer JP2.7
Changed lines of the file:
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@@
 <?xml version="1.0" encoding="utf-8"?>
 <!DOCTYPE eagle SYSTEM "eagle.dtd">
-<eagle version="9.6.2">
+<eagle version="9.4.2">
 <drawing>
 <settings>
-<setting alwaysvectorfont="no"/>
+<setting alwaysvectorfont="yes"/>
 <setting verticaltext="up"/>
 </settings>
@@
 <part name="S1" library="UNKNOWN-2024" deviceset="UNICS-SWITCH" device="SS_12D11"/>
 <part name="X2" library="UNKNOWN-2024" deviceset="JST-3-2.5" device="" value="AKKUM"/>
-<part name="JP2" library="pinhead" library_urn="urn:adsk.eagle:library:325" deviceset="PINHD-1X8" device="" package3d_urn="urn:adsk.eagle:package:22409/2"/>
 <part name="SI2302CDS" library="CanCubeSat" deviceset="SI2302CDS" device=""/>
 <part name="R1" library="rcl" library_urn="urn:adsk.eagle:library:334" deviceset="R-US_" device="R0603" package3d_urn="urn:adsk.eagle:package:23555/3" value="10k"/>
@@
 <part name="U$7" library="UNKNOWN-2024" deviceset="MOLEX-4-1.25" device=""/>
 <part name="U$8" library="UNKNOWN-2024" deviceset="MOLEX-5-1.25" device=""/>
+<part name="JP1" library="pinhead" library_urn="urn:adsk.eagle:library:325" deviceset="PINHD-1X4" device="" package3d_urn="urn:adsk.eagle:package:22407/2"/>
+<part name="JP3" library="pinhead" library_urn="urn:adsk.eagle:library:325" deviceset="PINHD-1X4" device="" package3d_urn="urn:adsk.eagle:package:22407/2"/>
 </parts>
 <sheets>
@@
 <attribute name="NAME" x="-16.51" y="132.842" size="1.778" layer="95"/>
 </instance>
-<instance part="JP2" gate="A" x="-45.72" y="25.4" smashed="yes">
-<attribute name="NAME" x="-52.07" y="38.735" size="1.778" layer="95"/>
-<attribute name="VALUE" x="-52.07" y="12.7" size="1.778" layer="96"/>
-</instance>
 <instance part="SI2302CDS" gate="G$1" x="276.86" y="134.62" smashed="yes" rot="R180"/>
 <instance part="R1" gate="G$1" x="287.02" y="129.54" smashed="yes" rot="R90">
@@
 <instance part="U$8" gate="G$1" x="251.46" y="63.5" smashed="yes">
 <attribute name="NAME" x="245.11" y="71.755" size="1.778" layer="95"/>
+</instance>
+<instance part="JP1" gate="A" x="-45.72" y="5.08" smashed="yes">
+<attribute name="NAME" x="-52.07" y="13.335" size="1.778" layer="95"/>
+<attribute name="VALUE" x="-52.07" y="-2.54" size="1.778" layer="96"/>
+</instance>
+<instance part="JP3" gate="A" x="-45.72" y="-10.16" smashed="yes">
+<attribute name="NAME" x="-52.07" y="-1.905" size="1.778" layer="95"/>
+<attribute name="VALUE" x="-52.07" y="-17.78" size="1.778" layer="96"/>
 </instance>
 </instances>
@@
 </segment>
 <segment>
-<wire x1="-48.26" y1="25.4" x2="-68.58" y2="25.4" width="0.1524" layer="91"/>
-<label x="-68.58" y="25.4" size="1.778" layer="95"/>
-<pinref part="JP2" gate="A" pin="5"/>
-</segment>
-<segment>
 <pinref part="SI2302CDS" gate="G$1" pin="S"/>
 <wire x1="287.02" y1="134.62" x2="297.18" y2="134.62" width="0.1524" layer="91"/>
@@
 <label x="233.68" y="35.56" size="1.778" layer="95"/>
 <pinref part="U$7" gate="G$1" pin="4"/>
+</segment>
+<segment>
+<wire x1="-48.26" y1="-5.08" x2="-68.58" y2="-5.08" width="0.1524" layer="91"/>
+<label x="-68.58" y="-5.08" size="1.778" layer="95"/>
+<pinref part="JP3" gate="A" pin="1"/>
 </segment>
 </net>
@@
 </segment>
 <segment>
-<wire x1="-48.26" y1="22.86" x2="-68.58" y2="22.86" width="0.1524" layer="91"/>
-<label x="-68.58" y="22.86" size="1.778" layer="95"/>
-<pinref part="JP2" gate="A" pin="6"/>
-</segment>
-<segment>
 <wire x1="231.14" y1="134.62" x2="223.52" y2="134.62" width="0.1524" layer="91"/>
 <label x="223.52" y="134.62" size="1.778" layer="95"/>
@@
 <pinref part="U$7" gate="G$1" pin="3"/>
 </segment>
+<segment>
+<wire x1="-48.26" y1="-7.62" x2="-68.58" y2="-7.62" width="0.1524" layer="91"/>
+<label x="-68.58" y="-7.62" size="1.778" layer="95"/>
+<pinref part="JP3" gate="A" pin="2"/>
+</segment>
 </net>
 <net name="BUS+" class="0">
@@
 </segment>
 </net>
-<net name="C0" class="0">
-<segment>
-<wire x1="-38.1" y1="63.5" x2="-71.12" y2="63.5" width="0.1524" layer="91"/>
-<label x="-71.12" y="63.5" size="1.778" layer="95"/>
-<pinref part="JP4" gate="A" pin="13"/>
-</segment>
-</net>
 <net name="NO2" class="0">
-<segment>
-<wire x1="-68.58" y1="33.02" x2="-48.26" y2="33.02" width="0.1524" layer="91"/>
-<label x="-68.58" y="33.02" size="1.778" layer="95"/>
-<pinref part="JP2" gate="A" pin="2"/>
-</segment>
 <segment>
 <wire x1="-71.12" y1="60.96" x2="-38.1" y2="60.96" width="0.1524" layer="91"/>
@@
 <pinref part="JP4" gate="A" pin="14"/>
 </segment>
+<segment>
+<wire x1="-68.58" y1="7.62" x2="-48.26" y2="7.62" width="0.1524" layer="91"/>
+<label x="-68.58" y="7.62" size="1.778" layer="95"/>
+<pinref part="JP1" gate="A" pin="2"/>
+</segment>
 </net>
 <net name="NH3" class="0">
-<segment>
-<wire x1="-48.26" y1="30.48" x2="-68.58" y2="30.48" width="0.1524" layer="91"/>
-<label x="-68.58" y="30.48" size="1.778" layer="95"/>
-<pinref part="JP2" gate="A" pin="3"/>
-</segment>
 <segment>
 <wire x1="-38.1" y1="58.42" x2="-71.12" y2="58.42" width="0.1524" layer="91"/>
@@
 <pinref part="JP4" gate="A" pin="15"/>
 </segment>
+<segment>
+<wire x1="-48.26" y1="5.08" x2="-68.58" y2="5.08" width="0.1524" layer="91"/>
+<label x="-68.58" y="5.08" size="1.778" layer="95"/>
+<pinref part="JP1" gate="A" pin="3"/>
+</segment>
 </net>
 <net name="MICS" class="0">
-<segment>
-<wire x1="-68.58" y1="27.94" x2="-48.26" y2="27.94" width="0.1524" layer="91"/>
-<label x="-68.58" y="27.94" size="1.778" layer="95"/>
-<pinref part="JP2" gate="A" pin="4"/>
-</segment>
 <segment>
 <wire x1="-71.12" y1="55.88" x2="-38.1" y2="55.88" width="0.1524" layer="91"/>
@@
 <pinref part="JP4" gate="A" pin="16"/>
 </segment>
+<segment>
+<wire x1="-68.58" y1="2.54" x2="-48.26" y2="2.54" width="0.1524" layer="91"/>
+<label x="-68.58" y="2.54" size="1.778" layer="95"/>
+<pinref part="JP1" gate="A" pin="4"/>
+</segment>
 </net>
 <net name="SDA" class="0">
-<segment>
-<wire x1="-48.26" y1="20.32" x2="-68.58" y2="20.32" width="0.1524" layer="91"/>
-<label x="-68.58" y="20.32" size="1.778" layer="95"/>
-<pinref part="JP2" gate="A" pin="7"/>
-</segment>
 <segment>
 <wire x1="-38.1" y1="93.98" x2="-71.12" y2="93.98" width="0.1524" layer="91"/>
@@
 <pinref part="JP4" gate="A" pin="1"/>
 </segment>
+<segment>
+<wire x1="-48.26" y1="-10.16" x2="-68.58" y2="-10.16" width="0.1524" layer="91"/>
+<label x="-68.58" y="-10.16" size="1.778" layer="95"/>
+<pinref part="JP3" gate="A" pin="3"/>
+</segment>
 </net>
 <net name="SCL" class="0">
-<segment>
-<wire x1="-48.26" y1="17.78" x2="-68.58" y2="17.78" width="0.1524" layer="91"/>
-<label x="-68.58" y="17.78" size="1.778" layer="95"/>
-<pinref part="JP2" gate="A" pin="8"/>
-</segment>
 <segment>
 <wire x1="-38.1" y1="91.44" x2="-71.12" y2="91.44" width="0.1524" layer="91"/>
 <label x="-71.12" y="91.44" size="1.778" layer="95"/>
 <pinref part="JP4" gate="A" pin="2"/>
+</segment>
+<segment>
+<wire x1="-48.26" y1="-12.7" x2="-68.58" y2="-12.7" width="0.1524" layer="91"/>
+<label x="-68.58" y="-12.7" size="1.778" layer="95"/>
+<pinref part="JP3" gate="A" pin="4"/>
 </segment>
 </net>
@@
 <net name="CO" class="0">
 <segment>
-<wire x1="-48.26" y1="35.56" x2="-68.58" y2="35.56" width="0.1524" layer="91"/>
-<label x="-68.58" y="35.56" size="1.778" layer="95"/>
-<pinref part="JP2" gate="A" pin="1"/>
-</segment>
-</net>
+<wire x1="-48.26" y1="10.16" x2="-68.58" y2="10.16" width="0.1524" layer="91"/>
+<label x="-68.58" y="10.16" size="1.778" layer="95"/>
+<pinref part="JP1" gate="A" pin="1"/>
+</segment>
+<segment>
+<wire x1="-38.1" y1="63.5" x2="-71.12" y2="63.5" width="0.1524" layer="91"/>
+<label x="-71.12" y="63.5" size="1.778" layer="95"/>
+<pinref part="JP4" gate="A" pin="13"/>
+</segment>
+</net>
