File: schematics/board/old/MOTOR.sch (EAGLE design)
At the start: 71 parts

Commit message: Платы готовы
Parts:
- removed BUT0, BUT1, BUT2, BUT3, BUT4, BUT5, BUT6, BUT7: (no value), pinheadCS:PINHD-1X2
- removed MOT0, MOT1, MOT2, MOT3, MOT4, MOT5, MOT6, MOT7: JST-2-2.5, UNKNOWN-2024:JST-2-2.5
- removed U$11, U$15, U$16, U$20, U$28, U$32: IRF5852, NA-2025:IRF5852
- removed U$19, U$27, U$31: CONCEVIC, CanCubeSat:CONCEVIC
- removed U$35, U$36, U$37, U$38, U$39, U$40, U$41, U$42: CONTACT_SIDE_4MM_2PIN, UNKNOWN-2024:CONTACT_SIDE_4MM_2PIN
- added JP10, JP12, JP14, JP16, JP18, JP4, JP8: (no value), pinhead:PINHD-1X3
- added JP11, JP13, JP15, JP17, JP3, JP7, JP9, MOTOR1, MOTOR2, MOTOR3, MOTOR4, MOTOR5, MOTOR6, MOTOR7: (no value), pinhead:PINHD-1X2
- added SI2302CDS1, SI2302CDS10, SI2302CDS11, SI2302CDS12, SI2302CDS13, SI2302CDS14, SI2302CDS15, SI2302CDS16, SI2302CDS2, SI2302CDS3, SI2302CDS4, SI2302CDS5, SI2302CDS6, SI2302CDS7, SI2302CDS8, SI2302CDS9: SI2302CDS, CanCubeSat:SI2302CDS
- added U$6, U$7: CONCEVIC, CanCubeSat:CONCEVIC
- JP1: device pinhead:PINHD-1X2/90 -> pinhead:PINHD-1X2
- JP19: value MOLEX-5-1.25 -> (none); device UNKNOWN-2024:MOLEX-5-1.25 -> pinhead:PINHD-1X5
- JP2: device pinhead:PINHD-1X2/90 -> pinhead:PINHD-1X3
- JP5: value JST-2-2.5 -> (none); device UNKNOWN-2024:JST-2-2.5 -> pinhead:PINHD-1X2
- U$10: value IRF5852 -> MOLEX-2-1.25; device NA-2025:IRF5852 -> UNKNOWN-2024:MOLEX-2-1.25
- U$5: value IRF5852 -> CONCEVIC; device NA-2025:IRF5852 -> CanCubeSat:CONCEVIC
Connections:
- removed net 16V_IN: JP2.1, MOT0.1, MOT1.1, MOT2.1, MOT3.1, MOT4.1, MOT5.1, MOT6.1, MOT7.1, U$10G$1.D1, U$11G$1.D1, U$15G$1.D1, U$16G$1.D1, U$20G$1.D1, U$28G$1.D1, U$32G$1.D1, U$5G$1.D1
- removed net 16V_OUT: JP2.2, JP5.1
- removed net GND_IN: JP1.1, R11.2, R15.2, R18.2, R2.2, R21.2, R24.2, R5.2, R8.2, U$1.P, U$10G$2.S1, U$11G$2.S1, U$15G$2.S1, U$16G$2.S1, U$19.P, U$2.P, U$20G$2.S1, U$27.P, U$28G$2.S1, U$3.P, U$31.P, U$32G$2.S1, U$4.P, U$5G$2.S1, U$8.P
- removed net GND_OUT: JP1.2, JP5.2, R14.1, U$13.GND
- new net 16V: JP1.2, JP10.3, JP11.2, JP12.3, JP13.2, JP14.3, JP15.2, JP16.3, JP17.2, JP18.3, JP2.3, JP3.2, JP4.3, JP5.1, JP7.2, JP8.3, JP9.2, R12.1, R16.1, R19.1, R22.1, R25.1, R3.1, R6.1, R9.1
- new net GND: JP5.2, R11.2, R14.1, R15.2, R18.2, R2.2, R21.2, R24.2, R5.2, R8.2, SI2302CDS1.S, SI2302CDS10.S, SI2302CDS11.S, SI2302CDS12.S, SI2302CDS13.S, SI2302CDS14.S, SI2302CDS15.S, SI2302CDS16.S, SI2302CDS2.S, SI2302CDS3.S, SI2302CDS4.S, SI2302CDS5.S, SI2302CDS6.S, SI2302CDS7.S, SI2302CDS8.S, SI2302CDS9.S, U$1.P, U$13.GND, U$2.P, U$3.P, U$4.P, U$5.P, U$6.P, U$7.P, U$8.P
- new net N$33: JP16.2, MOTOR6.1
- new net N$34: JP16.1, SI2302CDS14.D
- new net N$35: R22.2, SI2302CDS14.G
- new net N$36: JP17.1, MOTOR7.2, SI2302CDS15.D
- new net N$37: R23.2, R24.1, SI2302CDS15.G, U$8.S
- new net N$38: JP18.2, MOTOR7.1
- new net N$39: JP18.1, SI2302CDS16.D
- new net N$40: R25.2, SI2302CDS16.G
- net MOTOR0: now also U$13.Q0; no longer U$13.Q7
- net MOTOR4: now also U$13.Q4; no longer U$13.Q0
- net MOTOR5: now also U$13.Q5; no longer U$13.Q4
- net MOTOR6: now also U$13.Q6; no longer U$13.Q5
- net MOTOR7: now also U$13.Q7; no longer U$13.Q6
- net N$1: now also JP1.1, SI2302CDS1.D, U$10.2; no longer MOT0.2, R3.1, U$11G$2.D1, U$38.P$1
- net N$10: now also R6.2, SI2302CDS4.G; no longer BUT2.2, U$16G$1.S1, U$36.P$2
- net N$11: now also JP7.1, MOTOR2.2, SI2302CDS5.D; no longer R10.2, R11.1, U$4.S, U$5G$2.G1
- net N$12: now also SI2302CDS5.G; no longer U$16G$2.G1
- net N$13: now also JP8.2, MOTOR2.1; no longer BUT2.1, R9.1, U$16G$1.G1
- net N$14: now also JP8.1, SI2302CDS6.D; no longer MOT3.2, R12.2, U$37.P$1, U$5G$2.D1
- net N$15: now also R9.2, SI2302CDS6.G; no longer BUT3.2, U$37.P$2, U$5G$1.S1
- net N$16: now also JP9.1, MOTOR3.2, SI2302CDS7.D; no longer BUT3.1, R12.1, U$5G$1.G1
- net N$17: now also R10.2, R11.1, SI2302CDS7.G, U$4.S; no longer R13.2, R15.1, U$15G$2.G1, U$8.S
- net N$18: now also JP10.2, MOTOR3.1; no longer MOT4.2, R16.2, U$15G$2.D1, U$39.P$1
- net N$19: now also JP10.1, SI2302CDS8.D; no longer BUT4.2, U$15G$1.S1, U$39.P$2
- net N$2: now also JP3.1, MOTOR1.2, SI2302CDS3.D; no longer MOT1.2, R6.2, U$10G$2.D1, U$35.P$1
- net N$20: now also R12.2, SI2302CDS8.G; no longer BUT4.1, R16.1, U$15G$1.G1
- net N$21: now also JP11.1, MOTOR4.2, SI2302CDS9.D; no longer R17.2, R18.1, U$19.S, U$20G$2.G1
- net N$22: now also R13.2, R15.1, SI2302CDS9.G, U$5.S; no longer MOT5.2, R19.2, U$20G$2.D1, U$40.P$1
- net N$23: now also JP12.2, MOTOR4.1; no longer BUT5.2, U$20G$1.S1, U$40.P$2
- net N$24: now also JP12.1, SI2302CDS10.D; no longer BUT5.1, R19.1, U$20G$1.G1
- net N$25: now also R16.2, SI2302CDS10.G; no longer R20.2, R21.1, U$27.S, U$28G$2.G1
- net N$26: now also JP13.1, MOTOR5.2, SI2302CDS11.D; no longer MOT6.2, R22.2, U$28G$2.D1, U$41.P$1
- net N$27: now also R17.2, R18.1, SI2302CDS11.G, U$6.S; no longer BUT6.2, U$28G$1.S1, U$41.P$2
- net N$28: now also JP14.2, MOTOR5.1; no longer BUT6.1, R22.1, U$28G$1.G1
- net N$29: now also JP14.1, SI2302CDS12.D; no longer R23.2, R24.1, U$31.S, U$32G$2.G1
- net N$3: now also SI2302CDS3.G; no longer U$10G$2.G1
- net N$30: now also R19.2, SI2302CDS12.G; no longer MOT7.2, R25.2, U$32G$2.D1, U$42.P$1
- net N$31: now also JP15.1, MOTOR6.2, SI2302CDS13.D; no longer BUT7.2, U$32G$1.S1, U$42.P$2
- net N$32: now also R20.2, R21.1, SI2302CDS13.G, U$7.S; no longer BUT7.1, R25.1, U$32G$1.G1
- net N$4: now also SI2302CDS1.G; no longer U$11G$2.G1
- net N$5: now also JP4.2, MOTOR1.1; no longer BUT1.2, U$10G$1.S1, U$35.P$2
- net N$6: now also JP2.2, U$10.1; no longer BUT0.1, R3.2, U$11G$1.G1
- net N$7: now also JP4.1, SI2302CDS4.D; no longer BUT1.1, R6.1, U$10G$1.G1
- net N$8: now also JP2.1, SI2302CDS2.D; no longer BUT0.2, U$11G$1.S1, U$38.P$2
- net N$9: now also R3.2, SI2302CDS2.G; no longer MOT2.2, R9.2, U$16G$2.D1, U$36.P$1
Other:
- moved on the sheet: JP1, JP5, R1, R10, R11, R12, R13, R15, R16, R17, R18, R19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
