File: schematics/board/old/SP.brd (EAGLE design)
At the start: 45.6 x 46 mm, 24 parts

Commit message: Платы готовы
Parts:
- removed D7: MBR0520LT, diode:SOD123
- removed U$10, U$11, U$9: (no value), KNPN-2023:VIAS-CONNECT
- U$1, U$3, U$8: value SOLAR-2_INVERT0-2 -> SOLAR-2_1; device KNPN-2023:SOLAR_0-2_INVERT -> KNPN-2023:SOLAR_1-2
- U$2, U$6: value SOLAR-2_INVERT1-2 -> SOLAR-2_0; device KNPN-2023:SOLAR_1-2_INVERT -> KNPN-2023:SOLAR_0-2
- U$4: value SOLAR-2_INVERT0-2 -> SOLAR-2_0; device KNPN-2023:SOLAR_0-2_INVERT -> KNPN-2023:SOLAR_0-2
- moved D5 76.3 mm to (2.00, -38.5), flipped to the top
- moved D6 60.3 mm to (14.0, -38.5), flipped to the top, turned to 0 degrees
- moved U$6 56.0 mm to (8.00, -14.5), turned to 0 degrees
- moved U$8 52.1 mm to (7.50, -28.5), turned to 0 degrees
- moved U$5 20.4 mm to (0.00, -4.00), flipped to the top
- moved FOTO 7.80 mm to (20.5, 2.50)
- moved JP1 7.80 mm to (15.0, 43.5)
- moved SP-OUT 7.80 mm to (15.0, 1.90)
- moved U$7 7.80 mm to (15.0, 4.20)
- moved C1 2.24 mm to (15.5, 36.7)
- moved PWR 2.24 mm to (19.1, 35.4)
- moved R1 2.06 mm to (19.1, 38.1)
- turned D1 to 180 degrees
- turned D2 to 0 degrees
- turned D3 to 0 degrees
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Connections:
- removed net N$1: D7.A, JP1.2
- removed net N$5: D1.C, D2.A, U$1.OUT-2, U$1.OUT-21, U$2.IN-2
- removed net N$6: D3.A, D4.C, U$3.IN-2, U$4.OUT-2, U$4.OUT-21
- removed net N$7: D1.A, U$1.IN-2, U$9.1
- net N$2: now also D2.C, D3.A, U$2.OUT-2, U$2.OUT-21, U$3.IN-2; no longer D5.A, U$11.1, U$6.IN-2
- net N$3: now also D1.C, U$1.OUT; no longer U$10.1
- net N$8: now also U$6.OUT-2, U$6.OUT-21; no longer U$6.OUT
- net SP+: now also D1.A, D2.A, D5.A, JP1.2, U$1.IN-2, U$2.IN-2, U$6.IN-2; no longer D7.C, U$10.2, U$11.2, U$9.2
- net SP+-: now also D4.C, U$3.OUT, U$4.OUT-2, U$4.OUT-21, U$8.OUT; no longer D2.C, U$2.OUT, U$3.OUT-2, U$3.OUT-21, U$8.OUT-2, U$8.OUT-21
Routing:
- net SP+-: track 124.2 -> 43.5 mm, vias 2 -> 0
- net N$6: track 31.0 -> 0.00 mm, vias 1 -> 0
- net N$5: track 28.3 -> 0.00 mm, vias 1 -> 0
- net SP-: track 68.3 -> 43.1 mm
- net N$8: track 15.9 -> 0.00 mm, vias 1 -> 0
- net N$2: track 7.82 -> 23.3 mm
- net N$3: track 7.68 -> 15.1 mm
- net N$7: track 7.36 -> 0.00 mm, vias 1 -> 0
- net N$1: track 3.55 -> 0.00 mm
- net SP+: track 44.6 -> 43.5 mm, vias 0 -> 2
- net N$4: track 3.28 -> 2.78 mm
Other:
- board size 45.6 x 46 mm -> 30 x 46 mm
- board text added: "1.5V"
- board text added: "2V"
- board text removed: "0V"
