File: schematics/MOTOR.sch (EAGLE design)
At the start: 79 parts

Commit message: фцыувкаепнргошщз
Parts:
- BUT1, BUT2, BUT3, BUT4, BUT5, BUT6, BUT7: device pinhead:PINHD-1X2 -> pinheadCS:PINHD-1X2
- MOT1, MOT2, MOT3, MOT4, MOT5, MOT6, MOT7: value (none) -> JST-2-2.5; device pinhead:PINHD-1X2 -> UNKNOWN-2024:JST-2-2.5
Other:
- moved on the sheet: MOT1, MOT2, MOT3, MOT4, MOT5, MOT6, MOT7

Commit message: Плата MOTOR разведена, но не сделана шелкография
Parts:
- removed U$12, U$17, U$21, U$23, U$25, U$29, U$33, U$6: -, NA-2025:VIAS
- removed U$14, U$18, U$22, U$24, U$26, U$30, U$34, U$7: +, NA-2025:VIAS
- added U$35, U$36, U$37, U$38, U$39, U$40, U$41, U$42: CONTACT_SIDE_4MM_2PIN, UNKNOWN-2024:CONTACT_SIDE_4MM_2PIN
- JP19: value (none) -> MOLEX-5-1.25; device pinhead:PINHD-1X5 -> UNKNOWN-2024:MOLEX-5-1.25
- JP5: value (none) -> JST-2-2.5; device pinhead:PINHD-1X2 -> UNKNOWN-2024:JST-2-2.5
Connections:
- net MOTOR0: now also U$13.Q7; no longer U$13.Q0
- net MOTOR4: now also U$13.Q0; no longer U$13.Q4
- net MOTOR5: now also U$13.Q4; no longer U$13.Q5
- net MOTOR6: now also U$13.Q5; no longer U$13.Q6
- net MOTOR7: now also U$13.Q6; no longer U$13.Q7
- net N$1: now also U$38.P$1; no longer U$14.1
- net N$10: now also U$36.P$2; no longer U$23.1
- net N$14: now also U$37.P$1; no longer U$7.1
- net N$15: now also U$37.P$2; no longer U$6.1
- net N$18: now also U$39.P$1; no longer U$18.1
- net N$19: now also U$39.P$2; no longer U$17.1
- net N$2: now also U$35.P$1; no longer U$22.1
- net N$22: now also U$40.P$1; no longer U$26.1
- net N$23: now also U$40.P$2; no longer U$25.1
- net N$26: now also U$41.P$1; no longer U$30.1
- net N$27: now also U$41.P$2; no longer U$29.1
- net N$30: now also U$42.P$1; no longer U$34.1
- net N$31: now also U$42.P$2; no longer U$33.1
- net N$5: now also U$35.P$2; no longer U$21.1
- net N$8: now also U$38.P$2; no longer U$12.1
- net N$9: now also U$36.P$1; no longer U$24.1
Other:
- moved on the sheet: JP5
