File: schematics/shema.brd (EAGLE design)
At the start: 37.5 x 20 mm, 18 parts

Commit message: заказ плат
Parts:
- moved R3 1.00 mm to (21.6, 11.1)
- moved R1 0.50 mm to (24.8, 10.2)
- moved C1 0.20 mm to (29.1, 9.17)
Routing:
- net C: track 32.6 -> 35.2 mm
- net N$9: track 5.25 -> 7.16 mm, vias 0 -> 1
- net N$1: track 12.2 -> 13.2 mm, vias 1 -> 2
