File: schematics/Cansat-2025-1.brd (EAGLE design)
At the start: 102.5 x 79.5 mm, 75 parts, among them X1 JST-5, X2 JST-2-1.25, X3 JST-2-K-S, X4 JST-2-K-S

Commit message: заказ плат
Parts:
- added 3V3, 5V: (no value), led:CHIP-LED0603
- added AD8572: AD8572, grib:AD8572
- added C10, C16, C17, C9: 22u, rcl:C1206
- added C11, C14, C3, C7: 0,1u, rcl:C0603
- added C12, C4: 0,1u, rcl:C1206
- added C13, C6: 22u, rcl:C0603
- added C15, C8: 33p, rcl:C0603
- added C18, C22: 0.1uF, rcl:C0603
- added C19, C20, C21: 10uF, rcl:153CLV-0405
- added C23, C24: 1uF, rcl:153CLV-0405
- added COMPRESS, VALVE1, VALVE2: MOLEX-2-1.25, UNKNOWN-2024:53047-02
- added GPS-NEO7M: GPS-NEO7M, UNKNOWN-2024:GPS-NEO7M
- added JP1: (no value), pinhead:1X14
- added JP2, JP9: (no value), pinhead:1X02
- added JP5: (no value), pinhead:1X12
- added JP6: (no value), pinhead:1X04
- added JP7, JP8: (no value), pinhead:1X03
- added LIDAR: MOLEX-4-1.25, UNKNOWN-2024:53047-04
- added LSM6DS3: LSM6DS3, UNKNOWN-2024:LSM6DS3_WITHOUT
- added L_3.3, U$8: L_3.3MKH, CanCubeSat:L_SPM5020
- added MAX600: MAX660, grib:MAX660
- added MCP1700: MCP1700, grib:MCP1700
- added ME2-O2_OXYGEN_SENSOR: ME2-O2_OXYGEN_SENSOR, grib:ME2-O2_OXYGEN_SENSOR
- added MOTOR_BOARD: MOLEX-5-1.25, UNKNOWN-2024:53047-05
- added MP1584-3V3: MP1584-B, UNKNOWN-2024:MP1584-B
- added MP1584-5V: MP1584, UNKNOWN-2024:MP1584-B
- added POWER: (no value), UNKNOWN-2024:SS_12D11
- added R40, R43: 100k, rcl:R0603
- added R41, R44, R48: 10k, rcl:R0603
- added R42: 31k6, rcl:R0603
- added R45: 53k6, rcl:R0603
- added R46, R47: 2k, rcl:R0603
- added R49, R58: 100R, rcl:R0603
- added R50, RT1: 5K, rcl:R0603
- added R51: 68K, rcl:R0603
- added R52, R53, R56, R57: 10K, rcl:R0603
- added R54: 47R, rcl:R0603
- added R55: 5.1K, rcl:R0603
- added RADIO: E220-400T22S, UNKNOWN-2024:E220-400T22S
- added SI1, SI2300A: SI2302CDS, CanCubeSat:SOT23-3
- added U$10: LIS3MDL, UNKNOWN-2024:LIS3MDL
- added U$5: Плата Радио, UNKNOWN-2024:LOGO
- added U$6, U$7: MP2225, UNKNOWN-2024:TSOT23-8
- added X5: AKKUM, UNKNOWN-2024:JST-3-2.5
- moved C5 102.0 mm to (22.3, 157.3)
- moved PERE_L 102.0 mm to (29.0, 173.8)
- moved PERE_SP 102.0 mm to (20.5, 170.3)
- moved R0 102.0 mm to (55.9, 168.3)
- moved 74HC595 102.0 mm to (23.2, 134.6)
- moved AP1 102.0 mm to (48.1, 148.6)
- moved AP9930_ 102.0 mm to (47.8, 122.0)
- moved BME280 102.0 mm to (27.3, 155.5)
- moved BUZZER 102.0 mm to (15.8, 146.5)
- moved C2 102.0 mm to (24.7, 126.2)
- moved FOTO0 102.0 mm to (26.0, 107.1)
- moved INA 102.0 mm to (25.2, 157.9)
- moved IRF7905 102.0 mm to (33.4, 168.4)
- moved JP3 102.0 mm to (68.0, 140.0)
- moved JP4 102.0 mm to (8.00, 142.0)
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Connections:
- new net -3V: AD8572.P4, C20.-, MAX600.P5
- new net 3.3-5.5V: C23.+, JP7.3, MCP1700.P3
- new net 3V: AD8572.P8, C22.1, C24.+, MAX600.P8, MCP1700.P2
- new net 3V2: C10.2, C8.1, C9.2, GPS-NEO7M.P$1, JP5.3, LSM6DS3.P$2, L_3.3.P$1, MOTOR_BOARD.5, MP1584-3V3.P$7, MP1584-3V3.P$8, R42.2, R47.2, RADIO.P$25, U$10.UCC
- new net 4V1: JP5.1, X5.3
- new net 5V2: C15.1, C16.2, C17.2, COMPRESS.2, JP5.4, JP6.2, LIDAR.3, MP1584-5V.P$7, MP1584-5V.P$8, R45.2, R46.2, U$8.P$1, VALVE1.2, VALVE2.2
- new net AUX_RADIO1: JP5.7, RADIO.P$24
- new net BUS+: C12.2, C13.2, C4.2, C6.2, MP1584-3V3.P$1, MP1584-3V3.P$2, MP1584-5V.P$1, MP1584-5V.P$2, POWER.2, R40.1, R43.1, U$6.P$2, U$7.P$2
- new net BUS+_OUT: POWER.3, X5.1
- new net C: AD8572.P2, C19.-, ME2-O2_OXYGEN_SENSOR.C, R51.1, R52.2
- new net CS_LIS1: JP1.9, U$10.CS
- new net CS_LSM1: JP1.10, LSM6DS3.P$6
- new net D: ME2-O2_OXYGEN_SENSOR.D, R54.2
- new net D1: JP9.2, SI2300A.3
- new net FOTO2: JP1.13, JP2.1
- new net FOTO3: JP1.14, JP2.2
- new net G: JP9.1, R57.2, R58.1, R58.2, SI2300A.1
- new net GERMO1: JP5.6, R49.1
- new net GND2: 3V3.C, 5V.C, C10.1, C11.1, C12.1, C13.1, C16.1, C17.1, C3.1, C4.1, C6.1, C9.1, GPS-NEO7M.P$4, JP5.2, JP6.1, LIDAR.4, LSM6DS3.P$3, MP1584-3V3.P$3, MP1584-3V3.P$4, MP1584-3V3.P$5, MP1584-3V3.P$6, MP1584-5V.P$3, MP1584-5V.P$4, MP1584-5V.P$5, MP1584-5V.P$6, R41.2, R44.2, R48.2, RADIO.P$11, RADIO.P$13, RADIO.P$14, RADIO.P$15, RADIO.P$16, RADIO.P$19, RADIO.P$2, RADIO.P$26, RADIO.P$8, SI1.2, U$10.GND, U$6.P$1, U$6.P$4, U$7.P$1, U$7.P$4, X5.2
- new net GND3: AD8572.P3, C18.2, C20.+, C22.2, C23.-, C24.-, JP7.2, MAX600.P3, MCP1700.P1, R52.1, R54.1
- new net GND4: JP8.3, R56.2, R57.1, SI2300A.2
- new net IN: JP8.2, R55.1
- new net LATCH_SR1: JP1.12, MOTOR_BOARD.3
- new net M0_RADIO1: JP5.9, RADIO.P$20
- new net M1_RADIO1: JP5.8, RADIO.P$21
- new net MISO_SENS1: JP1.4, LSM6DS3.P$7, U$10.SDO
- new net MOSI_SENS1: JP1.3, LSM6DS3.P$5, U$10.SDA
- new net N$10: R40.2, U$6.P$6
- new net N$11: C7.2, U$6.P$5
- new net N$12: C7.1, L_3.3.P$2, U$6.P$3
- new net N$16: C14.2, U$7.P$5
- new net N$17: C14.1, U$7.P$3, U$8.P$2
- new net N$19: 5V.A, R46.1
- new net N$3: C8.2, R41.1, R42.1, U$6.P$8
- new net N$30: 3V3.A, R47.1
- new net N$31: R48.1, R49.2, SI1.1
- new net N$33: COMPRESS.1, SI1.3, VALVE1.1, VALVE2.1
- new net N$34: AD8572.P1, C19.+, R50.1, R53.2, RT1.1
- new net N$36: R50.2, R51.2, RT1.2
- new net N$37: C21.+, MAX600.P2
- new net N$38: C21.-, MAX600.P4
- new net N$6: C11.2, U$7.P$7
- new net N$7: R43.2, U$7.P$6
- new net N$8: C15.2, R44.1, R45.1, U$7.P$8
- new net N$9: C3.2, U$6.P$7
- new net OE_SR1: JP1.11, MOTOR_BOARD.2
- new net OUT: JP8.1, R55.2, R56.1
- new net RX_GPS1: GPS-NEO7M.P$3, JP5.10
- new net RX_LIDAR1: JP1.8, LIDAR.2
- new net RX_RADIO1: JP1.6, RADIO.P$23
- new net SCK_SENS1: JP5.12, LSM6DS3.P$4, MOTOR_BOARD.4, U$10.SCL
- new net SCL2: JP1.2, JP6.4
- new net SDA2: JP1.1, JP6.3
- new net SHIFT1: JP5.5, MOTOR_BOARD.1
- new net SOUT: C18.1, JP7.1, R53.1
- new net TX_GPS1: GPS-NEO7M.P$2, JP5.11
- new net TX_LIDAR1: JP1.7, LIDAR.1
- new net TX_RADIO1: JP1.5, RADIO.P$22
Routing:
- net GND2: track 0.00 -> 403.8 mm, vias 0 -> 38
- net 3V2: track 0.00 -> 187.7 mm, vias 0 -> 3
- net 5V2: track 0.00 -> 186.5 mm, vias 0 -> 2
- net SCK_SENS1: track 0.00 -> 113.3 mm, vias 0 -> 1
- net BUS+: track 0.00 -> 78.4 mm
- net MISO_SENS1: track 0.00 -> 70.9 mm, vias 0 -> 1
- net MOSI_SENS1: track 0.00 -> 69.9 mm
- net SHIFT1: track 0.00 -> 69.8 mm
- net SDA2: track 0.00 -> 68.3 mm
- net SCL2: track 0.00 -> 64.2 mm
- net GND3: track 0.00 -> 61.9 mm, vias 0 -> 1
- net AUX_RADIO1: track 0.00 -> 59.4 mm
- net LATCH_SR1: track 0.00 -> 54.8 mm
- net CS_LSM1: track 0.00 -> 53.0 mm, vias 0 -> 2
- net TX_RADIO1: track 0.00 -> 52.7 mm, vias 0 -> 2
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- added copper zone on layer 16, net 3V2
- added copper zone on layer 16, net 5V2
- added copper zone on layer 16, net BUS+
- added copper zone on layer 1, net GND2
- added copper zone on layer 16, net GND2
- added copper zone on layer 16, net GND3
- added copper zone on layer 1, net GND4
- added copper zone on layer 16, net GND4
- added copper zone on layer 16, net N$11
- added copper zone on layer 16, net N$12
- added copper zone on layer 16, net N$16
- added copper zone on layer 16, net N$17
- added copper zone on layer 16, net N$3
- added copper zone on layer 16, net N$8
Other:
- board size 102.5 x 79.5 mm -> 76 x 178 mm
- board text added: "D"
- board text added: "FOT 0"
- board text added: "FOT1"
- board text added: "G"
- board text added: "IN"
- board text added: "MOSI _S"
- board text added: "OUT"
- board text added: "RX_G"
- board text added: "TX_G"

Commit message: СД в центре лепестка. Платы версия 2
Parts:
- removed AD8572: AD8572, grib:AD8572
- removed ADS1115: ADS1115, NA-2025:MSOP10
- removed AP1: MOSFET_2P+2N_AP9930GM, UNKNOWN-2024:SO8
- removed AP9930: MOSFET_2P+2N_AP9930GM, NA-2025:SO8
- removed AP9930_: AP9930GM, UNKNOWN-2024:SO8
- removed C18, C22: 0.1uF, rcl:C0603
- removed C19, C20, C21: 10uF, rcl:153CLV-0405
- removed C23, C24: 1uF, rcl:153CLV-0405
- removed JP7: (no value), pinhead:1X03
- removed MAX600: MAX660, grib:MAX660
- removed MCP1700: MCP1700, grib:MCP1700
- removed ME2-O2_OXYGEN_SENSOR: ME2-O2_OXYGEN_SENSOR, grib:ME2-O2_OXYGEN_SENSOR
- removed R10, R2, R52, R53, R9: 10K, rcl:R0603
- removed R50, RT1: 5K, rcl:R0603
- removed R51: 68K, rcl:R0603
- removed R54: 47R, rcl:R0603
- removed R7, R8: 5K1, rcl:R0603
- removed U$2: IRF5852, NA-2025:TSOP-6
- removed U$3: VT93N1, KNPN-2023:VT93N1
- removed X1: JST-5, NA-2025:MOLEX-5-1.25
- removed X2: JST-2-1.25, NA-2025:MOLEX-2-1.25
- removed X3, X4: JST-2-K-S, NA-2025:B2B-PH-K-S
- added AD1: AD8572, grib:AD8572
- added ADS1: ADS1115, NA-2025:MSOP10
- added C25, C29: 0.1uF, rcl:C0603
- added C26, C27, C28: 10uF, rcl:153CLV-0405
- added C30, C31: 1uF, rcl:153CLV-0405
- added JP10: (no value), pinhead:1X03
- added MAX1: MAX660, grib:MAX660
- added MCP1: MCP1700, grib:MCP1700
- added ME2-O2_OXYGEN_SENSOR1: ME2-O2_OXYGEN_SENSOR, grib:ME2-O2_OXYGEN_SENSOR
- added R59, R60, R66, R68: 10K, rcl:R0603
- added R61, R62: 2k, rcl:R0603
- added R63, R64: 5K1, rcl:R0603
- added R65, R67: 100R, rcl:R0603
- added RT2: 5K, rcl:R0603
- added U$11: IRF5852, NA-2025:TSOP-6
- added U$12, U$13, U$19, U$20, U$21, U$22: FDC6420C, KNPN-2023:TSOP-6
- added U$9: VT93N1, KNPN-2023:VT93N1
- added X6: JST-5, NA-2025:MOLEX-5-1.25
- added X7: JST-2-1.25, NA-2025:MOLEX-2-1.25
- added X8, X9: JST-2-K-S, NA-2025:B2B-PH-K-S
- R1: value 10K -> 5K
- R3: value 2k -> 68K
- R4: value 2k -> 10K
- R5: value 100R -> 10K
- R6: value 100R -> 47R
- moved R3 58.7 mm to (14.0, 89.3), flipped to the bottom, turned to 180 degrees
- moved R1 53.9 mm to (14.0, 87.2), flipped to the bottom, turned to 0 degrees
- moved C1 53.0 mm to (14.0, 80.9), flipped to the bottom, turned to 180 degrees
- moved R6 50.0 mm to (14.0, 93.5), flipped to the bottom, turned to 0 degrees
- moved R5 49.8 mm to (14.0, 83.0), flipped to the bottom, turned to 180 degrees
- moved R4 49.0 mm to (14.0, 91.4), flipped to the bottom, turned to 0 degrees
- moved U$4 26.9 mm to (12.2, 128.1), turned to 0 degrees
- moved SP 19.3 mm to (7.10, 123.6), turned to 298 degrees
- moved FOTO0 19.3 mm to (10.4, 118.4), turned to 308 degrees
- moved R18 16.8 mm to (12.9, 121.3), turned to 218 degrees
- moved MICRO_SD 10.8 mm to (24.2, 104.3), turned to 147.5 degrees
- moved C2 5.33 mm to (28.8, 122.8), turned to 147.5 degrees
- moved R16 5.08 mm to (31.3, 123.8), turned to 327.5 degrees
- moved R17 4.95 mm to (28.5, 125.6), turned to 147.5 degrees
- moved R32 4.54 mm to (50.8, 150.6), turned to 0 degrees
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Connections:
- removed net -3V: AD8572.P4, C20.-, MAX600.P5
- removed net 3.3-5.5V: C23.+, JP7.3, MCP1700.P3
- removed net 3V: AD8572.P8, C22.1, C24.+, MAX600.P8, MCP1700.P2
- removed net 5V: AP9930.7, R1.2, R2.1, X3.1
- removed net C: AD8572.P2, C19.-, ME2-O2_OXYGEN_SENSOR.C, R51.1, R52.2
- removed net D: ME2-O2_OXYGEN_SENSOR.D, R54.2
- removed net GND3: AD8572.P3, C18.2, C20.+, C22.2, C23.-, C24.-, JP7.2, MAX600.P3, MCP1700.P1, R52.1, R54.1
- removed net M1: AP9930.2, X4.1
- removed net M2: AP9930.6, X4.2
- removed net N$34: AD8572.P1, C19.+, R50.1, R53.2, RT1.1
- removed net N$36: R50.2, R51.2, RT1.2
- removed net N$37: C21.+, MAX600.P2
- removed net N$38: C21.-, MAX600.P4
- removed net PHOTO: ADS1115.5, R4.2, X2.P$1
- removed net SCL: ADS1115.9, R7.1, X1.P$3
- removed net SDA: ADS1115.10, R8.1, X1.P$2
- removed net SOUT: C18.1, JP7.1, R53.1
- removed net UM1: R5.1, X1.P$4
- removed net UM1_MOSFET: AP9930.1, AP9930.8, R1.1, U$2.P$6
- removed net UM2: R6.2, X1.P$5
- removed net UM2_MOSFET: AP9930.4, AP9930.5, R2.2, U$2.P$4
- new net -3V1: AD1.P4, C27.-, MAX1.P5
- new net 3.3-5.5V1: C30.+, JP10.3, MCP1.P3
- new net 3V4: ADS1.8, C25.2, R61.1, R62.1, R63.2, R64.2, X6.P$1
- new net 5V3: R59.2, R60.1, U$12.P$2, U$13.P$2, X8.1
- new net C1: AD1.P2, C26.-, ME2-O2_OXYGEN_SENSOR1.C, R3.1, R4.2
- new net D2: ME2-O2_OXYGEN_SENSOR1.D, R6.2
- new net GND5: ADS1.3, C25.1, R66.1, R68.1, U$11.P$2, U$11.P$5, U$12.P$5, U$13.P$5, U$9.P$2, X7.P$2, X8.2
- new net M3: U$12.P$4, U$12.P$6, X9.2
- new net M4: U$13.P$4, U$13.P$6, X9.1
- new net N$39: ADS1.4, R61.2, U$9.P$1
- new net N$40: R65.1, R66.2, U$11.P$1
- new net N$41: R67.2, R68.2, U$11.P$3
- new net N$42: C28.-, MAX1.P4
- new net PHOTO1: ADS1.5, R62.2, X7.P$1
- new net SCL3: ADS1.9, R63.1, X6.P$3
- new net SDA3: ADS1.10, R64.1, X6.P$2
- new net SOUT1: C1.1, JP10.1, R5.1
- new net UM1_MOSFET1: R59.1, U$11.P$6, U$13.P$1, U$13.P$3
- new net UM2_MOSFET1: R60.2, U$11.P$4, U$12.P$1, U$12.P$3
- new net UM3: R67.1, X6.P$4
- new net UM4: R65.2, X6.P$5
- net 3V3: now also AD1.P8, C29.1, C31.+, MAX1.P8, MCP1.P2; no longer ADS1115.8, C1.2, R3.1, R4.1, R7.2, R8.2, X1.P$1
- net 5V1: now also U$19.P$2, U$20.P$2, U$21.P$2, U$22.P$2; no longer AP1.7, AP9930_.7
- net GND: now also AD1.P3, C1.2, C27.+, C29.2, C30.-, C31.-, JP10.2, MAX1.P3, MCP1.P1, R4.1, R6.1; no longer ADS1115.3, AP9930.3, C1.1, R10.1, R9.1, U$2.P$2, U$2.P$5, U$3.P$2, X2.P$2, X3.2
- net GND1: now also U$19.P$5, U$20.P$5, U$21.P$5, U$22.P$5; no longer AP1.3, AP9930_.3
- net MOTOR1+: now also U$22.P$4, U$22.P$6; no longer AP1.6
- net MOTOR1-: now also U$21.P$4, U$21.P$6; no longer AP1.2
- net MOTOR2+: now also U$20.P$4, U$20.P$6; no longer AP9930_.6
- net MOTOR2-: now also U$19.P$4, U$19.P$6; no longer AP9930_.2
- net N$1: now also AD1.P1, C26.+, R1.1, RT2.1; no longer R9.2, U$2.P$3
- net N$24: now also U$21.P$1, U$21.P$3; no longer AP1.1, AP1.8
- net N$25: now also U$19.P$1, U$19.P$3; no longer AP9930_.1, AP9930_.8
- net N$26: now also U$20.P$1, U$20.P$3; no longer AP9930_.4, AP9930_.5
- net N$27: now also U$22.P$1, U$22.P$3; no longer AP1.4, AP1.5
- net N$4: now also R1.2, RT2.2; no longer ADS1115.4, U$3.P$1
- net N$5: now also C28.+, MAX1.P2; no longer R10.2, R6.1, U$2.P$1
Routing:
- net GND5: track 0.00 -> 71.3 mm, vias 0 -> 6
- net GND3: track 61.9 -> 0.00 mm, vias 1 -> 0
- net 3V: track 49.5 -> 0.00 mm, vias 1 -> 0
- net SOUT: track 38.7 -> 0.00 mm, vias 1 -> 0
- net C: track 35.2 -> 0.00 mm, vias 1 -> 0
- net 3.3-5.5V1: track 0.00 -> 34.6 mm, vias 0 -> 1
- net 3.3-5.5V: track 32.5 -> 0.00 mm, vias 1 -> 0
- net 5V3: track 0.00 -> 32.1 mm, vias 0 -> 2
- net -3V: track 31.0 -> 0.00 mm, vias 2 -> 0
- net M4: track 0.00 -> 27.3 mm, vias 0 -> 2
- net GND: track 71.3 -> 97.4 mm, vias 7 -> 3
- net M2: track 25.8 -> 0.00 mm, vias 1 -> 0
- net C1: track 0.00 -> 23.4 mm, vias 0 -> 1
- net 3V4: track 0.00 -> 22.7 mm
- net SCL3: track 0.00 -> 21.7 mm
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- added copper zone on layer 1, net GND5
- added copper zone on layer 16, net GND5
- removed copper zone on layer 16, net GND3
Other:
- outline, holes or cut-outs redrawn
- board text added: "3V3 5V5"
- board text added: "FDC6 420C"
- board text added: "SOUT"
