File: schematics/RADIO.brd (EAGLE design)
At the start: 76 x 76 mm, 49 parts, among them X2 AKKUM

Commit message: Поправлены платы МК, Радио, Гермо
Parts:
- moved R12 51.8 mm to (16.1, 43.9)
- moved 3V3 50.8 mm to (14.5, 43.9), turned to 0 degrees
- moved 5V 33.9 mm to (14.5, 40.5)
- moved C13 32.2 mm to (39.4, 59.3)
- moved R6 30.3 mm to (70.0, 63.8), turned to 180 degrees
- moved R11 29.0 mm to (16.1, 40.5), turned to 90 degrees
- moved U$2 26.7 mm to (67.7, 59.3), turned to 0 degrees
- moved R8 26.4 mm to (48.9, 66.8), turned to 180 degrees
- moved U$5 26.3 mm to (42.3, 63.5), turned to 270 degrees
- moved R5 22.6 mm to (71.1, 52.7), turned to 270 degrees
- moved C11 22.4 mm to (67.1, 54.2), turned to 180 degrees
- moved C6 22.1 mm to (63.6, 62.2), turned to 180 degrees
- moved C4 21.7 mm to (47.4, 62.9), turned to 90 degrees
- moved C5 20.9 mm to (49.8, 62.9), turned to 90 degrees
- moved C12 20.5 mm to (67.1, 52.0), turned to 180 degrees
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Connections:
- removed net C0: JP4.13
- net CO: now also JP4.13
- net RX_GPS: now also JP5.10; no longer JP5.11
- net RX_LIDAR: now also JP4.8; no longer JP4.7
- net RX_RADIO: now also JP4.6; no longer JP4.5
- net TX_GPS: now also JP5.11; no longer JP5.10
- net TX_LIDAR: now also JP4.7; no longer JP4.8
- net TX_RADIO: now also JP4.5; no longer JP4.6
Routing:
- net GND: track 0.00 -> 403.8 mm, vias 0 -> 38
- net 3V3: track 0.00 -> 187.7 mm, vias 0 -> 3
- net 5V: track 0.00 -> 186.5 mm, vias 0 -> 2
- net SCK_SENS: track 0.00 -> 113.3 mm, vias 0 -> 1
- net MISO_SENS: track 0.00 -> 73.2 mm, vias 0 -> 1
- net MOSI_SENS: track 0.00 -> 72.2 mm
- net SDA: track 0.00 -> 71.5 mm
- net SHIFT: track 0.00 -> 69.8 mm
- net SCL: track 0.00 -> 68.4 mm
- net AUX_RADIO: track 0.00 -> 59.4 mm
- net TX_RADIO: track 0.00 -> 55.0 mm, vias 0 -> 2
- net RX_RADIO: track 0.00 -> 54.9 mm, vias 0 -> 2
- net CS_LSM: track 0.00 -> 54.0 mm, vias 0 -> 2
- net LATCH_SR: track 0.00 -> 52.3 mm
- net M1_RADIO: track 0.00 -> 52.2 mm
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- added copper zone on layer 16, net 3V3
- added copper zone on layer 16, net 5V
- added copper zone on layer 16, net BUS+
- added copper zone on layer 16, net N$11
- added copper zone on layer 16, net N$12
- added copper zone on layer 16, net N$13
- added copper zone on layer 16, net N$16
- added copper zone on layer 16, net N$17
- added copper zone on layer 16, net N$18
